File: Electrical_Group/VCU_CM5/5v_buck.kicad_sch (KiCad schematic)
At the start: 17 parts, among them U2 TPS5430DDA

Commit message: [VCU_CM5] update to V1.0
still needs many modifications
Parts:
- removed C13: 10u 50V, Capacitor_SMD:C_1206_3216Metric, symbol Device:C_Small
- F3: renamed from F2; footprint Fuse:Fuse_1206_3216Metric -> Fuse:Fuse_1206_3216Metric_Pad1.42x1.75mm_HandSolder
- U3: renamed from U2; footprint Package_SO:TI_SO-PowerPAD-8_ThermalVias -> Package_SO:TI_SO-PowerPAD-8
- renumbered C14 to C10, C15 to C11, C16 to C12, C17 to C13, C18 to C14, C19 to C15, C20 to C16, C21 to C17, C12 to C9, D2 to D4, D3 to D5, L3 to L2, R8 to R13, R9 to R14
Other:
- company: (none) -> NTURacing Team
- title: (none) -> VCU_CM5
