File: Electrical_Group/VCU_CM5/CAN.kicad_sch (KiCad schematic)
At the start: 9 parts, among them J5 CAN, U3 TCAN1042VDRQ1

Commit message: [VCU_CM5] update to V1.0
still needs many modifications
Parts:
- removed J5: CAN, Connector_JST:JST_PH_B2B-PH-K_1x02_P2.00mm_Vertical, symbol Connector_Generic:Conn_01x02
- D6: renamed from D4; now fitted
- FL2: footprint SamacSys_Parts_EP6:EXCX4CE900U -> nturt_kicad_lib_EP7:EXCX4CE900U
- renumbered C22 to C18, C23 to C19, R10 to R15, R11 to R16, R12 to R17, U3 to U4
Connections:
- net +5V renamed +5V_CM
- net CAN+ renamed CAN_H
- net CAN_H: now also D6.2 (K); no longer D6.1 (K)
- net CAN- renamed CAN_L
- net CAN_L: now also D6.1 (K); no longer D6.2 (K)
Other:
- company: (none) -> NTURacing Team
- title: (none) -> VCU_CM5
- moved on the sheet: C18, C19
