File: Electrical_Group/VCU_CM5/VCU_CM5.kicad_pcb (KiCad board)
At the start: 6 copper layers, 102 x 85 mm, 386 parts, among them J1 USB3_A, J10 MSD-4-A, J11 Conn_01x30_Socket, J12 Conn_02x16_Odd_Even, J13 USART6, J14 MSD-4-A, J15 buzzer, J16 CAN, J18 CAN, J19 CAN, J2 LVBattery, J3 24V_raw, J4 5Vout, J5 CAN, J6 S_SWD, J7 MIPI_CAM_22P, J8 JST_SH, J9 MIPI_DISP_15P, Q1 AO3400A, Q2 MMBT3904, Q3 2N7002, Q4 2N7002, SW1 POWER_BTN, SW2 RESET, SW3 BOOT0, U1 LM66100DCK, U10 SN74LVC4245APWR, U11 STM32H743ZITx, U12 TPS5430DDA, U13 TCAN1042VDRQ1, U14 USB2514B_Bi, U17 TCAN1042VDRQ1, U18 TCAN1042VDRQ1, U19 MCP2515-xST, U2 TPS5430DDA, U3 TCAN1042VDRQ1, U4 LSM6DSOX, U5 STM32F103CBT6, U6 TLV75733PDRV, U7 TLV75733PDRV, U8 TLV75733PDRV, U9 MCP2515-xST, Y1 8MHz X50328MSB2GI, Y2 12MHz 830105420809, Y3 8MHz X50328MSB2GI, Y4 32.768kHz Q13FC13500004, Y5 24MHz, Y6 12MHz 830105420809

Commit message: [VCU_CM5] update to V1.0
still needs many modifications
Parts:
- removed the C1 at (288.6, 142.0)
- removed the C10 at (210.0, 102.6)
- removed the C110 at (266.4, 134.8)
- removed the C122 at (281.1, 83.9)
- removed the C13 at (263.2, 139.6)
- removed the C2 at (288.6, 139.7)
- removed the C3 at (283.6, 145.4)
- removed the C30 at (152.0, 166.4)
- removed the C31 at (172.3, 72.3)
- removed the C32 at (250.4, 186.8)
- removed the C4 at (276.5, 136.4)
- removed the C54 at (274.0, 98.0)
- removed the D29 at (257.8, 167.7)
- removed the D30 at (209.8, 43.8)
- removed the D31 at (209.8, 46.4)
- removed the D32 at (209.8, 49.0)
- removed the D33 at (209.8, 51.6)
- removed the D5 at (172.9, 86.0)
- removed the D6 at (172.9, 78.0)
- removed J12: Conn_02x16_Odd_Even, Connector_PinSocket_2.00mm:PinSocket_2x16_P2.00mm_Vertical
- removed J13: USART6, Connector_JST:JST_PH_B3B-PH-K_1x03_P2.00mm_Vertical
- removed J15: buzzer, Connector_JST:JST_XH_B2B-XH-A_1x02_P2.50mm_Vertical
- removed J16, J18, J19: CAN, Connector_JST:JST_PH_B2B-PH-K_1x02_P2.00mm_Vertical
- removed the J3 at (297.0, 140.5)
- removed the J4 at (297.0, 132.9)
- removed the J7 at (215.5, 90.5)
- removed the L1 at (283.6, 141.4)
- removed the Q3 at (253.5, 165.8)
- removed the R105 at (96.6, 69.5)
- removed the R107 at (96.6, 73.5)
- removed the R109 at (99.5, 63.5)
- removed the R111 at (99.5, 67.5)
- removed the R113 at (99.5, 71.5)
- removed the R115 at (99.5, 75.5)
- removed the R119 at (203.4, 46.9)
- removed the R121 at (203.4, 50.9)
- removed the R13 at (218.7, 177.0)
- removed the R14 at (218.7, 179.0)
- removed the R15 at (218.7, 181.0)
- removed the R150 at (275.6, 119.2)
- removed the R16 at (218.7, 183.0)
- removed the R17 at (169.4, 85.7)
- removed the R28 at (169.4, 65.7)
- removed the R30 at (149.1, 165.8)
- removed the R31 at (149.1, 167.8)
- removed the R32 at (169.4, 69.7)
- removed the R33 at (169.4, 71.7)
- removed the R34 at (169.4, 73.7)
- removed the R35 at (247.5, 184.2)
- removed the R36 at (247.5, 186.2)
- removed the R37 at (247.5, 188.2)
- removed the U19 at (276.0, 115.2)
- removed the U4 at (222.5, 178.1)
- removed the Y2 at (276.6, 98.0)
- removed the Y5 at (277.5, 83.9)
- added C123: Xp, Capacitor_SMD:C_0402_1005Metric, F.Cu at (226.0, 87.3)
- added C20: 1u, Capacitor_SMD:C_0402_1005Metric, F.Cu at (210.4, 147.8)
- added C21: 10u, Capacitor_SMD:C_0402_1005Metric, F.Cu at (217.9, 147.3)
- added C22: 1u, Capacitor_SMD:C_0402_1005Metric, F.Cu at (210.4, 149.8)
- added C23: 10u, Capacitor_SMD:C_0402_1005Metric, F.Cu at (217.9, 149.3)
- added C51: 30p, Capacitor_SMD:C_0402_1005Metric, F.Cu at (270.6, 97.3)
- added C7: 1u, Capacitor_SMD:C_0402_1005Metric, F.Cu at (269.6, 132.1)
- added C8: 1u, Capacitor_SMD:C_0402_1005Metric, F.Cu at (267.8, 129.8)
- added C84: 22u, Capacitor_SMD:C_0805_2012Metric, B.Cu at (233.4, 142.9)
- added C85: 22u, Capacitor_SMD:C_0805_2012Metric, B.Cu at (231.4, 142.9)
- added D16: RED_LED, LED_SMD:LED_0603_1608Metric, B.Cu at (199.9, 102.3)
- added D17: SMBJ5.0A, Diode_SMD:D_SMB, F.Cu at (224.9, 113.4)
- added D2: WHITE, LED_SMD:LED_0603_1608Metric, B.Cu at (277.2, 135.8)
- added D3: zener 3.6V, Diode_SMD:D_SOD-123, F.Cu at (265.3, 130.6)
- added F1: 0.5A, Fuse:Fuse_1206_3216Metric_Pad1.42x1.75mm_HandSolder, B.Cu at (283.7, 90.4)
- added F10: 30mA, Fuse:Fuse_0805_2012Metric_Pad1.15x1.40mm_HandSolder, B.Cu at (212.5, 136.0)
- added F11: 30mA, Fuse:Fuse_0805_2012Metric_Pad1.15x1.40mm_HandSolder, B.Cu at (212.5, 137.9)
- added F12: 30mA, Fuse:Fuse_0805_2012Metric_Pad1.15x1.40mm_HandSolder, B.Cu at (212.5, 139.8)
- added F13: 30mA, Fuse:Fuse_0805_2012Metric_Pad1.15x1.40mm_HandSolder, B.Cu at (212.5, 141.7)
- added F14: 30mA, Fuse:Fuse_0805_2012Metric_Pad1.15x1.40mm_HandSolder, B.Cu at (212.5, 143.6)
- added F15: 30mA, Fuse:Fuse_0805_2012Metric_Pad1.15x1.40mm_HandSolder, B.Cu at (212.5, 145.5)
- added F16: 30mA, Fuse:Fuse_0805_2012Metric_Pad1.15x1.40mm_HandSolder, B.Cu at (212.5, 147.4)
- added F17: 30mA, Fuse:Fuse_0805_2012Metric_Pad1.15x1.40mm_HandSolder, B.Cu at (212.5, 149.3)
- added F18: 30mA, Fuse:Fuse_0805_2012Metric_Pad1.15x1.40mm_HandSolder, B.Cu at (212.5, 151.2)
- added F19: 30mA, Fuse:Fuse_0805_2012Metric_Pad1.15x1.40mm_HandSolder, B.Cu at (212.5, 153.1)
- added F20: 30mA, Fuse:Fuse_0805_2012Metric_Pad1.15x1.40mm_HandSolder, B.Cu at (212.5, 155.0)
- added F21: 30mA, Fuse:Fuse_0805_2012Metric_Pad1.15x1.40mm_HandSolder, B.Cu at (212.5, 122.7)
- added F22: 30mA, Fuse:Fuse_0805_2012Metric_Pad1.15x1.40mm_HandSolder, B.Cu at (212.5, 124.6)
- added F23: 30mA, Fuse:Fuse_0805_2012Metric_Pad1.15x1.40mm_HandSolder, B.Cu at (212.5, 126.5)
- added F24: 30mA, Fuse:Fuse_0805_2012Metric_Pad1.15x1.40mm_HandSolder, B.Cu at (212.5, 128.4)
- added F4: RPI_FUSE_5A, Fuse:Fuse_1206_3216Metric_Pad1.42x1.75mm_HandSolder, B.Cu at (226.9, 113.5)
- added F5: 30mA, Fuse:Fuse_0805_2012Metric_Pad1.15x1.40mm_HandSolder, B.Cu at (212.5, 118.9)
- added F6: 30mA, Fuse:Fuse_0805_2012Metric_Pad1.15x1.40mm_HandSolder, B.Cu at (212.5, 120.8)
- added F7: 30mA, Fuse:Fuse_0805_2012Metric_Pad1.15x1.40mm_HandSolder, B.Cu at (212.5, 130.3)
- added F8: 30mA, Fuse:Fuse_0805_2012Metric_Pad1.15x1.40mm_HandSolder, B.Cu at (212.5, 132.2)
- added F9: 30mA, Fuse:Fuse_0805_2012Metric_Pad1.15x1.40mm_HandSolder, B.Cu at (212.5, 134.1)
- added J11: STDC14, nturt_kicad_lib_EP7:box_header_14P_pitch1.27_smd, B.Cu at (249.0, 154.3)
- added J9: Conn_02x15_Odd_Even, Connector_PinHeader_2.00mm:PinHeader_2x15_P2.00mm_Vertical_SMD, F.Cu at (249.0, 156.0)
- added NT1: NetTie, NetTie:NetTie-2_SMD_Pad0.5mm, B.Cu at (226.7, 104.0)
- added R1: 0R, Resistor_SMD:R_0603_1608Metric_Pad0.98x0.95mm_HandSolder, B.Cu at (296.0, 101.4)
- added R100: 75R, Resistor_SMD:R_0603_1608Metric, F.Cu at (204.9, 150.9)
- added R102: 100R, Resistor_SMD:R_0603_1608Metric, F.Cu at (212.5, 119.6)
- added R104: 100R, Resistor_SMD:R_0603_1608Metric, F.Cu at (212.5, 121.6)
- added R11: 100k, Resistor_SMD:R_0402_1005Metric, F.Cu at (267.7, 133.6)
- added R110: 100R, Resistor_SMD:R_0603_1608Metric, F.Cu at (212.5, 127.6)
- added R118: 100R, Resistor_SMD:R_0603_1608Metric, F.Cu at (212.5, 135.6)
- added R12: 100k, Resistor_SMD:R_0402_1005Metric, F.Cu at (272.5, 137.5)
- added R124: 100R, Resistor_SMD:R_0603_1608Metric, F.Cu at (212.5, 141.6)
- added R126: 100R, Resistor_SMD:R_0603_1608Metric, F.Cu at (212.5, 143.6)
- added R128: 10k, Resistor_SMD:R_0603_1608Metric_Pad0.98x0.95mm_HandSolder, B.Cu at (231.8, 145.4)
- added R131: 0R, Resistor_SMD:R_0402_1005Metric_Pad0.72x0.64mm_HandSolder, F.Cu at (231.3, 95.5)
- added R132: 0R, Resistor_SMD:R_0402_1005Metric_Pad0.72x0.64mm_HandSolder, F.Cu at (232.3, 95.5)
- added R133: 100R, Resistor_SMD:R_0603_1608Metric, B.Cu at (244.3, 149.2)
- added R134: 0R, Resistor_SMD:R_0603_1608Metric, B.Cu at (258.0, 154.3)
- added R141: 100R, Resistor_SMD:R_0603_1608Metric, F.Cu at (212.5, 145.6)
- added R2: 0R, Resistor_SMD:R_0603_1608Metric_Pad0.98x0.95mm_HandSolder, B.Cu at (294.5, 101.4)
- added R3: 0R, Resistor_SMD:R_0603_1608Metric_Pad0.98x0.95mm_HandSolder, B.Cu at (294.3, 105.9)
- added R42: 100R, Resistor_SMD:R_0603_1608Metric_Pad0.98x0.95mm_HandSolder, B.Cu at (238.4, 125.8)
- added R49: 680R, Resistor_SMD:R_0402_1005Metric, B.Cu at (201.6, 102.3)
- added R61: 75R, Resistor_SMD:R_0603_1608Metric_Pad0.98x0.95mm_HandSolder, B.Cu at (208.8, 122.7)
- added R62: 75R, Resistor_SMD:R_0603_1608Metric_Pad0.98x0.95mm_HandSolder, B.Cu at (208.8, 124.2)
- added R63: 75R, Resistor_SMD:R_0603_1608Metric_Pad0.98x0.95mm_HandSolder, B.Cu at (208.8, 125.7)
- added R65: 75R, Resistor_SMD:R_0603_1608Metric_Pad0.98x0.95mm_HandSolder, B.Cu at (208.8, 128.7)
- added R66: 75R, Resistor_SMD:R_0603_1608Metric_Pad0.98x0.95mm_HandSolder, B.Cu at (208.8, 130.2)
- added R67: 75R, Resistor_SMD:R_0603_1608Metric_Pad0.98x0.95mm_HandSolder, B.Cu at (208.8, 131.7)
- added R68: 75R, Resistor_SMD:R_0603_1608Metric_Pad0.98x0.95mm_HandSolder, B.Cu at (208.8, 133.2)
- added R84: 75R, Resistor_SMD:R_0603_1608Metric, F.Cu at (204.9, 126.9)
- added R85: 75R, Resistor_SMD:R_0603_1608Metric, F.Cu at (204.9, 128.4)
- added R86: 75R, Resistor_SMD:R_0603_1608Metric, F.Cu at (204.9, 129.9)
- added R87: 75R, Resistor_SMD:R_0603_1608Metric, F.Cu at (204.9, 131.4)
- added R88: 75R, Resistor_SMD:R_0603_1608Metric, F.Cu at (204.9, 132.9)
- added R89: 75R, Resistor_SMD:R_0603_1608Metric, F.Cu at (204.9, 134.4)
- added R90: 75R, Resistor_SMD:R_0603_1608Metric, F.Cu at (204.9, 135.9)
- added R91: 75R, Resistor_SMD:R_0603_1608Metric, F.Cu at (204.9, 137.4)
- added R92: 75R, Resistor_SMD:R_0603_1608Metric, F.Cu at (204.9, 138.9)
- added R93: 75R, Resistor_SMD:R_0603_1608Metric, F.Cu at (204.9, 140.4)
- added R94: 75R, Resistor_SMD:R_0603_1608Metric, F.Cu at (204.9, 141.9)
- added R95: 75R, Resistor_SMD:R_0603_1608Metric, F.Cu at (204.9, 143.4)
- added R96: 75R, Resistor_SMD:R_0603_1608Metric, F.Cu at (204.9, 144.9)
- added TP1: RPI_CAN0_H, nturt_kicad_lib_EP7:edge_pad_1.4mm_0.7mm, F.Cu at (298.0, 98.0)
- added TP10: GND, nturt_kicad_lib_EP7:edge_pad_1.4mm_0.7mm, F.Cu at (298.0, 114.0)
- added TP11: 24V_in, nturt_kicad_lib_EP7:edge_pad_1.4mm_0.7mm, F.Cu at (298.0, 150.0)
- added TP12: +5V, nturt_kicad_lib_EP7:edge_pad_1.4mm_0.7mm, F.Cu at (298.0, 116.0)
- added TP13: BUZZER_P, nturt_kicad_lib_EP7:edge_pad_1.4mm_0.7mm, F.Cu at (298.1, 122.0)
- added TP14: BUZZER_N, nturt_kicad_lib_EP7:edge_pad_1.4mm_0.7mm, F.Cu at (298.1, 120.0)
- added TP2: RPI_CAN0_L, nturt_kicad_lib_EP7:edge_pad_1.4mm_0.7mm, F.Cu at (298.0, 100.0)
- added TP3: RPI_CAN1_H, nturt_kicad_lib_EP7:edge_pad_1.4mm_0.7mm, F.Cu at (298.0, 102.0)
- added TP4: RPI_CAN1_L, nturt_kicad_lib_EP7:edge_pad_1.4mm_0.7mm, F.Cu at (298.0, 104.0)
- added TP5: STM32_CAN1_H, nturt_kicad_lib_EP7:edge_pad_1.4mm_0.7mm, F.Cu at (298.0, 106.0)
- added TP6: STM32_CAN1_L, nturt_kicad_lib_EP7:edge_pad_1.4mm_0.7mm, F.Cu at (298.0, 108.0)
- added TP7: STM32_CAN2_H, nturt_kicad_lib_EP7:edge_pad_1.4mm_0.7mm, F.Cu at (298.0, 110.0)
- added TP8: STM32_CAN2_L, nturt_kicad_lib_EP7:edge_pad_1.4mm_0.7mm, F.Cu at (298.0, 112.0)
- added TP9: GND_in, nturt_kicad_lib_EP7:edge_pad_1.4mm_0.7mm, F.Cu at (298.0, 146.0)
- added U11: REF3133AIDBZR, Package_TO_SOT_SMD:SOT-23, B.Cu at (237.7, 142.9)
- added U2: TLV75733PDRV, Package_SON:WSON-6-1EP_2x2mm_P0.65mm_EP1x1.6mm, F.Cu at (267.8, 131.6)
- added Y4: 40Mhz XTM32040000DT00351001, Crystal:Crystal_SMD_3225-4Pin_3.2x2.5mm, F.Cu at (227.6, 140.4)
- added Y6: 24Mhz X322524MOB4SI, Crystal:Crystal_SMD_3225-4Pin_3.2x2.5mm, F.Cu at (226.0, 89.9)
- C1: renamed from C5; footprint Capacitor_THT:CP_Radial_D8.0mm_P3.80mm -> Capacitor_SMD:CP_Elec_6.3x5.2
- C109: renamed from C107; value 1n -> 1u
- C2: renamed from C6; moved to B.Cu
- C24: value 0u1 -> 1u
- C25: value 0u1 -> 10u
- C26, C28: value 330p -> 1u
- C27, C29: value 330p -> 10u
- C3: renamed from C7; moved to B.Cu
- C30: renamed from C33; value 1n -> 1u
- C4: renamed from C8; moved to B.Cu
- C42: renamed from C45; moved to B.Cu
- C5: renamed from C9; footprint Capacitor_THT:CP_Radial_D8.0mm_P3.80mm -> Capacitor_SMD:CP_Elec_6.3x5.2
- C56, C58, C60, C62, C64, C66, C68, C70, C72, C74, C76, C78, C80: value 1n -> 1u
- C82, C83: value 0u1 -> 470n; footprint Capacitor_SMD:C_0402_1005Metric -> Capacitor_SMD:C_0603_1608Metric; moved to B.Cu
- D10, D11, D7, D8, D9: value WHITE Button -> zener 3.6V; footprint LED_SMD:LED_0603_1608Metric -> Diode_SMD:D_SOD-323
- D12: footprint Diode_SMD:D_SOD-523 -> Diode_SMD:D_SOD-323
- D13, D14, FL1, Module1, SW2, SW3: moved to B.Cu
- D15: value RED -> GREEN_LED; moved to B.Cu
- D18: renamed from D16; footprint Diode_SMD:D_SOD-523 -> Diode_SMD:D_SOD-323
- D19: renamed from D17; footprint Diode_SMD:D_SOD-523 -> Diode_SMD:D_SOD-323
- D20: renamed from D18; footprint Diode_SMD:D_SOD-523 -> Diode_SMD:D_SOD-323
- D21: renamed from D19; footprint Diode_SMD:D_SOD-523 -> Diode_SMD:D_SOD-323
- D22: renamed from D20; footprint Diode_SMD:D_SOD-523 -> Diode_SMD:D_SOD-323
- D23: renamed from D21; footprint Diode_SMD:D_SOD-523 -> Diode_SMD:D_SOD-323
- D24: renamed from D22; footprint Diode_SMD:D_SOD-523 -> Diode_SMD:D_SOD-323
- D25: renamed from D23; footprint Diode_SMD:D_SOD-523 -> Diode_SMD:D_SOD-323
- D26: renamed from D24; footprint Diode_SMD:D_SOD-523 -> Diode_SMD:D_SOD-323
- D27: renamed from D25; footprint Diode_SMD:D_SOD-523 -> Diode_SMD:D_SOD-323
- D28: renamed from D26; footprint Diode_SMD:D_SOD-523 -> Diode_SMD:D_SOD-323
- D29: renamed from D27; footprint Diode_SMD:D_SOD-523 -> Diode_SMD:D_SOD-323
- D30: renamed from D28; footprint Diode_SMD:D_SOD-523 -> Diode_SMD:D_SOD-323
- D31: renamed from D34; footprint Diode_SMD:D_SOD-523 -> Diode_SMD:D_SOD-323
- D32: renamed from D35; moved to B.Cu
- D35: renamed from D38; moved to F.Cu
- D36: renamed from D40; moved to F.Cu
- D38: renamed from D41; moved to F.Cu
- D6: renamed from D4; moved to F.Cu
- F2: renamed from F1; moved to B.Cu
- F25: renamed from F3; footprint Fuse:Fuse_1206_3216Metric -> Fuse:Fuse_1206_3216Metric_Pad1.42x1.75mm_HandSolder; moved to B.Cu
- F3: renamed from F2; footprint Fuse:Fuse_1206_3216Metric -> Fuse:Fuse_1206_3216Metric_Pad1.42x1.75mm_HandSolder; moved to B.Cu
- FL2, FL3, FL4, FL5: footprint SamacSys_Parts_EP6:EXCX4CE900U -> nturt_kicad_lib_EP7:EXCX4CE900U
- J10: renamed from J14; footprint SamacSys_Parts_EP6:MSD4A -> nturt_kicad_lib_EP7:MSD4A
- J2: value LVBattery -> UPS_CAP; footprint Connector_JST:JST_XH_B2B-XH-A_1x02_P2.50mm_Vertical -> Connector_PinHeader_2.00mm:PinHeader_1x02_P2.00mm_Horizontal; moved to B.Cu
- J3: renamed from J6; footprint Connector_PinHeader_2.54mm:PinHeader_1x03_P2.54mm_Vertical -> Connector_PinHeader_2.00mm:PinHeader_1x03_P2.00mm_Vertical; moved to B.Cu
- J4: renamed from J8; footprint Connector_JST:JST_SH_BM04B-SRSS-TB_1x04-1MP_P1.00mm_Vertical -> Connector_JST:JST_SH_SM04B-SRSS-TB_1x04-1MP_P1.00mm_Horizontal
- J5: value CAN -> MIPI_CAM_22P; footprint Connector_JST:JST_PH_B2B-PH-K_1x02_P2.00mm_Vertical -> Connector_FFC-FPC:Hirose_FH12-22S-0.5SH_1x22-1MP_P0.50mm_Horizontal; moved to B.Cu
- J6: renamed from J9; moved to B.Cu
- J7: renamed from J10; footprint SamacSys_Parts_EP6:MSD4A -> nturt_kicad_lib_EP7:MSD4A; moved to F.Cu
- J8: renamed from J11; footprint Connector_FFC-FPC:Amphenol_F32Q-1A7x1-11030_1x30-1MP_P0.5mm_Horizontal -> Connector_FFC-FPC:Amphenol_F32Q-1A7x1-11040_1x40-1MP_P0.5mm_Horizontal; moved to B.Cu
- JP1: value BTN1_AS_RST -> stlink NRST; moved to B.Cu
- L1: renamed from L2; moved to B.Cu
- R106, R108, R112, R114, R116: value 0R -> 100R; footprint Resistor_SMD:R_0402_1005Metric -> Resistor_SMD:R_0603_1608Metric
- R120, R122, R23, R29: value 1k -> 100R; footprint Resistor_SMD:R_0402_1005Metric -> Resistor_SMD:R_0603_1608Metric
- R18, R22, R24: value 10k -> 150R 1%; footprint Resistor_SMD:R_0402_1005Metric -> Resistor_SMD:R_0603_1608Metric
- R19, R21, R25, R27: value 10k -> 100R; footprint Resistor_SMD:R_0402_1005Metric -> Resistor_SMD:R_0603_1608Metric
- R20, R26: value 1k -> 150R 1%; footprint Resistor_SMD:R_0402_1005Metric -> Resistor_SMD:R_0603_1608Metric
- R38: renamed from R47; footprint Resistor_SMD:R_0402_1005Metric -> Resistor_SMD:R_0603_1608Metric_Pad0.98x0.95mm_HandSolder; moved to B.Cu
- R39: renamed from R48; footprint Resistor_SMD:R_0402_1005Metric -> Resistor_SMD:R_0603_1608Metric_Pad0.98x0.95mm_HandSolder; moved to B.Cu
- R4: value 20k -> 0R; footprint Resistor_SMD:R_0402_1005Metric -> Resistor_SMD:R_0603_1608Metric_Pad0.98x0.95mm_HandSolder; moved to B.Cu
- R40: renamed from R49; footprint Resistor_SMD:R_0402_1005Metric -> Resistor_SMD:R_0603_1608Metric_Pad0.98x0.95mm_HandSolder; moved to B.Cu
- R41: renamed from R50; footprint Resistor_SMD:R_0402_1005Metric -> Resistor_SMD:R_0603_1608Metric_Pad0.98x0.95mm_HandSolder; moved to B.Cu
- R46: renamed from R54; footprint Resistor_SMD:R_0402_1005Metric -> Resistor_SMD:R_0402_1005Metric_Pad0.72x0.64mm_HandSolder
- R47: renamed from R55; footprint Resistor_SMD:R_0402_1005Metric -> Resistor_SMD:R_0402_1005Metric_Pad0.72x0.64mm_HandSolder
- R48: renamed from R56; moved to B.Cu
- R64: value 10k -> 75R; footprint Resistor_SMD:R_0402_1005Metric -> Resistor_SMD:R_0603_1608Metric_Pad0.98x0.95mm_HandSolder; moved to B.Cu
- R69, R70, R71, R72, R73, R74, R75, R76, R77, R78, R79, R80: value 10R -> 75R; footprint Resistor_SMD:R_0603_1608Metric -> Resistor_SMD:R_0603_1608Metric_Pad0.98x0.95mm_HandSolder; moved to B.Cu
- R81, R82, R83: value 10R -> 75R
- R97: value 1k -> 75R; footprint Resistor_SMD:R_0402_1005Metric -> Resistor_SMD:R_0603_1608Metric
- R98: value 100 -> 75R; footprint Resistor_SMD:R_0402_1005Metric -> Resistor_SMD:R_0603_1608Metric
- R99: value 100k -> 75R; footprint Resistor_SMD:R_0402_1005Metric -> Resistor_SMD:R_0603_1608Metric
- SW1: value POWER_BTN -> RPI_PWR; footprint Button_Switch_SMD:SW_SPST_PTS810 -> Button_Switch_SMD:SW_Tactile_SPST_NO_Straight_CK_PTS636Sx25SMTRLFS; moved to B.Cu
- U10: value SN74LVC4245APWR -> MCP2518FD; footprint Package_SO:TSSOP-24_4.4x7.8mm_P0.65mm -> Package_SO:SOIC-14_3.9x8.7mm_P1.27mm
- U13: renamed from U12; footprint Package_SO:TI_SO-PowerPAD-8_ThermalVias -> Package_SO:TI_SO-PowerPAD-8
- U3: renamed from U2; footprint Package_SO:TI_SO-PowerPAD-8_ThermalVias -> Package_SO:TI_SO-PowerPAD-8
- U9: value MCP2515-xST -> MCP2518FD; footprint Package_SO:TSSOP-20_4.4x6.5mm_P0.65mm -> Package_SO:SOIC-14_3.9x8.7mm_P1.27mm
- Y2: renamed from Y6; value 12MHz 830105420809 -> 40Mhz XTM32040000DT00351001
- Y3: value 8MHz X50328MSB2GI -> 40Mhz XTM32040000DT00351001; footprint Crystal:Crystal_SMD_5032-2Pin_5.0x3.2mm -> Crystal:Crystal_SMD_3225-4Pin_3.2x2.5mm
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- renumbered C14 to C10, C98 to C100, C99 to C101, C100 to C102, C101 to C103, C102 to C104, C103 to C105, C104 to C106, C105 to C107, C106 to C108, C15 to C11, C108 to C110, C109 to C111, C111 to C112, C112 to C113, C113 to C114, C114 to C115, C115 to C116, C116 to C117, C117 to C118, C118 to C119, C16 to C12, C119 to C120, C120 to C121, C121 to C122, C123 to C124, C124 to C125, C125 to C126, C126 to C127, C127 to C128, C128 to C129, C17 to C13, C129 to C130, C130 to C131, C140 to C136, C141 to C137, C18 to C14, C142 to C143, C143 to C144, C19 to C15, C20 to C16, C21 to C17, C22 to C18, C23 to C19, C34 to C31, C35 to C32, C36 to C33, C37 to C34, C38 to C35, C39 to C36, C40 to C37, C41 to C38, C42 to C39, C43 to C40, C44 to C41, C46 to C43, C47 to C44, C48 to C45, C49 to C46, C50 to C47, C51 to C48, C52 to C49, C144 to C50, C145 to C52, C146 to C54, C11 to C6, C84 to C86, C85 to C87, C86 to C88, C87 to C89, C12 to C9, C88 to C90, C89 to C91, C90 to C92, C91 to C93, C92 to C94, C93 to C95, C94 to C96, C95 to C97, C96 to C98, C97 to C99, D36 to D33, D37 to D34, D2 to D4, D3 to D5, L3 to L2, L4 to L3, Q4 to Q3, R7 to R10, R84 to R101, R85 to R103, R86 to R105, R87 to R107, R88 to R109, R89 to R111, R90 to R113, R91 to R115, R92 to R117, R93 to R119, R94 to R121, R95 to R123, R96 to R125, R110 to R127, R117 to R129, R8 to R13, R118 to R130, R123 to R135, R124 to R136, R125 to R137, R126 to R138, R127 to R139, R9 to R14, R128 to R140, R129 to R142, R130 to R143, R131 to R144, R132 to R145, R133 to R146, R134 to R147, R135 to R148, R136 to R149, R10 to R15, R137 to R150, R138 to R151, R139 to R152, R144 to R155, R145 to R156, R146 to R158, R11 to R16, R147 to R160, R148 to R161, R149 to R162, R12 to R17, R38 to R28, R39 to R30, R40 to R31, R41 to R32, R42 to R33, R43 to R34, R44 to R35, R45 to R36, R46 to R37, R51 to R43, R52 to R44, R53 to R45, R1 to R5, R57 to R50, R58 to R51, R59 to R52, R60 to R53, R61 to R54, R62 to R55, R63 to R56, R65 to R57, R66 to R58, R67 to R59, R2 to R6, R68 to R60, R3 to R7, R5 to R8, R6 to R9, U11 to U12, U13 to U14, U14 to U15, U18 to U19, U3 to U4, Y4 to Y5
Connections:
- net /computer/compute module/USB_D+ renamed /computer/compute module/USB.D+
- net /computer/compute module/USB_D- renamed /computer/compute module/USB.D-
- net /stlink/VCP_MCU.RX renamed /stlink/VCP_MCU_UART.RX
- net /stlink/VCP_MCU.TX renamed /stlink/VCP_MCU_UART.TX
- C10 pad 2: /power/5v buck mcu/24V_IN -> +24V
- C109 pad 1: /vcu mcu/current loop sensors/CL_CH15 -> /vcu mcu/current loop sensors/current loop 15/CL_LOOP
- C110 pad 1: /vcu mcu/current loop sensors/CL_CH15 -> /vcu mcu/CL_CH15
- C111 pad 1: /power/5v buck mcu/24V_IN -> +24V
- C112 pad 2: /power/5v buck mcu/24V_IN -> +24V
- C120 pad 1: +5V -> +5V_CM
- C124 pad 1: /computer/3V3_CAM -> +3V3_CMOUT
- C125 pad 1: /computer/3V3_CAM -> +3V3_CMOUT
- C126 pad 1: /computer/3V3_CAM -> +3V3_CMOUT
- C127 pad 1: /computer/3V3_CAM -> +3V3_CMOUT
- C128 pad 1: /computer/3V3_CAM -> +3V3_CMOUT
- C129 pad 1: /computer/3V3_CAM -> +3V3_CMOUT
- C130 pad 1: /computer/3V3_CAM -> +3V3_CMOUT
- C131 pad 1: /computer/3V3_CAM -> +3V3_CMOUT
- C136 pad 1: +5V -> +5V_CM
- C143 pad 1: +5V -> +5V_CM
- C18 pad 1: +5V -> +5V_CM
- C24 pad 1: GND -> /vcu mcu/current loop sensors/current loop 18/CL_LOOP
- C24 pad 2: +3V3 -> GND
- C25 pad 1: GND -> /vcu mcu/CL_CH18
- C25 pad 2: +3V3 -> GND
- C26 pad 1: /vcu mcu/button3 -> /vcu mcu/current loop sensors/current loop 19/CL_LOOP
- C27 pad 1: /vcu mcu/button1 -> /vcu mcu/CL_CH19
- C28 pad 1: /vcu mcu/button2 -> /vcu mcu/current loop sensors/current loop 20/CL_LOOP
- C29 pad 1: /vcu mcu/button5 -> /vcu mcu/CL_CH20
- C30 pad 1: /vcu mcu/current loop sensors/CL_CH1 -> /vcu mcu/current loop sensors/current loop 1/CL_LOOP
- C31 pad 1: /vcu mcu/current loop sensors/CL_CH1 -> /vcu mcu/CL_CH1
- C43 pad 1: +5V_RPI -> +5V_CM
- C44 pad 1: +5V_RPI -> +5V_CM
- C45 pad 1: +5V_RPI -> +5V_CM
- C50 pad 1: Net-(U19-OSC2) -> Net-(U9-OSC2)
- C52 pad 1: Net-(U19-OSC1) -> Net-(U9-OSC1)
- C53 pad 1: Net-(U9-OSC2) -> Net-(U10-OSC1)
- C56 pad 1: /vcu mcu/current loop sensors/CL_CH2 -> /vcu mcu/current loop sensors/current loop 2/CL_LOOP
- C57 pad 1: /vcu mcu/current loop sensors/CL_CH2 -> /vcu mcu/CL_CH2
- C58 pad 1: /vcu mcu/current loop sensors/CL_CH3 -> /vcu mcu/current loop sensors/current loop 3/CL_LOOP
- C59 pad 1: /vcu mcu/current loop sensors/CL_CH3 -> /vcu mcu/CL_CH3
- C60 pad 1: /vcu mcu/current loop sensors/CL_CH4 -> /vcu mcu/current loop sensors/current loop 4/CL_LOOP
- C61 pad 1: /vcu mcu/current loop sensors/CL_CH4 -> /vcu mcu/CL_CH4
- C62 pad 1: /vcu mcu/current loop sensors/CL_CH5 -> /vcu mcu/current loop sensors/current loop 5/CL_LOOP
- C63 pad 1: /vcu mcu/current loop sensors/CL_CH5 -> /vcu mcu/CL_CH5
- C64 pad 1: /vcu mcu/current loop sensors/CL_CH6 -> /vcu mcu/current loop sensors/current loop 6/CL_LOOP
- C65 pad 1: /vcu mcu/current loop sensors/CL_CH6 -> /vcu mcu/CL_CH6
- C66 pad 1: /vcu mcu/current loop sensors/CL_CH7 -> /vcu mcu/current loop sensors/current loop 7/CL_LOOP
- C67 pad 1: /vcu mcu/current loop sensors/CL_CH7 -> /vcu mcu/CL_CH7
- C68 pad 1: /vcu mcu/current loop sensors/CL_CH8 -> /vcu mcu/current loop sensors/current loop 8/CL_LOOP
- C69 pad 1: /vcu mcu/current loop sensors/CL_CH8 -> /vcu mcu/CL_CH8
- C70 pad 1: /vcu mcu/current loop sensors/CL_CH9 -> /vcu mcu/current loop sensors/current loop 9/CL_LOOP
- C71 pad 1: /vcu mcu/current loop sensors/CL_CH9 -> /vcu mcu/CL_CH9
- C72 pad 1: /vcu mcu/current loop sensors/CL_CH10 -> /vcu mcu/current loop sensors/current loop 10/CL_LOOP
- C73 pad 1: /vcu mcu/current loop sensors/CL_CH10 -> /vcu mcu/CL_CH10
- C74 pad 1: /vcu mcu/current loop sensors/CL_CH11 -> /vcu mcu/current loop sensors/current loop 11/CL_LOOP
- C75 pad 1: /vcu mcu/current loop sensors/CL_CH11 -> /vcu mcu/CL_CH11
- C76 pad 1: /vcu mcu/current loop sensors/CL_CH12 -> /vcu mcu/current loop sensors/current loop 12/CL_LOOP
- C77 pad 1: /vcu mcu/current loop sensors/CL_CH12 -> /vcu mcu/CL_CH12
- C78 pad 1: /vcu mcu/current loop sensors/CL_CH13 -> /vcu mcu/current loop sensors/current loop 13/CL_LOOP
- C79 pad 1: /vcu mcu/current loop sensors/CL_CH13 -> /vcu mcu/CL_CH13
- C80 pad 1: /vcu mcu/current loop sensors/CL_CH14 -> /vcu mcu/current loop sensors/current loop 14/CL_LOOP
- C81 pad 1: /vcu mcu/current loop sensors/CL_CH14 -> /vcu mcu/CL_CH14
- C82 pad 1: +3V3 -> +5V
- C83 pad 1: +5V -> Net-(U11-OUT)
- C9 pad 1: /power/5v buck mcu/24V_IN -> +24V
- D10 pad 1: Net-(D10-K) -> /vcu mcu/CL_CH19
- D10 pad 2: +3V3 -> GND
- D11 pad 1: Net-(D11-K) -> /vcu mcu/CL_CH20
- D11 pad 2: +3V3 -> GND
- D12 pad 1: /vcu mcu/current loop sensors/CL_CH1 -> /vcu mcu/CL_CH1
- D15 pad 1: /computer/compute module/nACT_LED -> Net-(D15-K)
- D15 pad 2: Net-(D15-A) -> +3V3_CMOUT
- D18 pad 1: /vcu mcu/current loop sensors/CL_CH2 -> /vcu mcu/CL_CH2
- D19 pad 1: /vcu mcu/current loop sensors/CL_CH3 -> /vcu mcu/CL_CH3
- D20 pad 1: /vcu mcu/current loop sensors/CL_CH4 -> /vcu mcu/CL_CH4
- D21 pad 1: /vcu mcu/current loop sensors/CL_CH5 -> /vcu mcu/CL_CH5
- D22 pad 1: /vcu mcu/current loop sensors/CL_CH6 -> /vcu mcu/CL_CH6
- D23 pad 1: /vcu mcu/current loop sensors/CL_CH7 -> /vcu mcu/CL_CH7
- D24 pad 1: /vcu mcu/current loop sensors/CL_CH8 -> /vcu mcu/CL_CH8
- D25 pad 1: /vcu mcu/current loop sensors/CL_CH9 -> /vcu mcu/CL_CH9
- D26 pad 1: /vcu mcu/current loop sensors/CL_CH10 -> /vcu mcu/CL_CH10
- D27 pad 1: /vcu mcu/current loop sensors/CL_CH11 -> /vcu mcu/CL_CH11
- D28 pad 1: /vcu mcu/current loop sensors/CL_CH12 -> /vcu mcu/CL_CH12
- D29 pad 1: /vcu mcu/current loop sensors/CL_CH13 -> /vcu mcu/CL_CH13
- D30 pad 1: /vcu mcu/current loop sensors/CL_CH14 -> /vcu mcu/CL_CH14
- D31 pad 1: /vcu mcu/current loop sensors/CL_CH15 -> /vcu mcu/CL_CH15
- D35 pad 1: /CAN 2/CAN+ -> /CAN 2/CAN_L
- D35 pad 2: /CAN 2/CAN- -> /CAN 2/CAN_H
- D36 pad 1: /CAN 1/CAN+ -> /CAN 1/CAN_L
- D36 pad 2: /CAN 1/CAN- -> /CAN 1/CAN_H
- D38 pad 1: /CAN 3/CAN+ -> /CAN 3/CAN_L
- D38 pad 2: /CAN 3/CAN- -> /CAN 3/CAN_H
- D5 pad 1: +5V_RPI -> +5V_CM
- D6 pad 1: /CAN 4/CAN+ -> /CAN 4/CAN_L
- D6 pad 2: /CAN 4/CAN- -> /CAN 4/CAN_H
- D7 pad 1: Net-(D7-K) -> /vcu mcu/CL_CH16
- D7 pad 2: +3V3 -> GND
- D8 pad 1: Net-(D8-K) -> /vcu mcu/CL_CH17
- D8 pad 2: +3V3 -> GND
- D9 pad 1: Net-(D9-K) -> /vcu mcu/CL_CH18
- D9 pad 2: +3V3 -> GND
- F3 pad 2: +5V_RPI -> +5V_CM
- FL1 pad 1: Net-(J2-Pin_1) -> Net-(FL1-Pad1)
- FL1 pad 2: Net-(J2-Pin_2) -> Net-(FL1-Pad2)
- FL2 pad 3: /CAN 4/CAN- -> /CAN 4/CAN_L
- FL2 pad 4: /CAN 4/CAN+ -> /CAN 4/CAN_H
- FL3 pad 3: /CAN 2/CAN- -> /CAN 2/CAN_L
- FL3 pad 4: /CAN 2/CAN+ -> /CAN 2/CAN_H
- FL4 pad 3: /CAN 1/CAN- -> /CAN 1/CAN_L
- FL4 pad 4: /CAN 1/CAN+ -> /CAN 1/CAN_H
- FL5 pad 3: /CAN 3/CAN- -> /CAN 3/CAN_L
- FL5 pad 4: /CAN 3/CAN+ -> /CAN 3/CAN_H
- J1 pad 1: +5V_RPI -> Net-(J1-VBUS)
- J1 pad 4: unconnected-(J1-GND-Pad4) -> GND
- J10 pad G1: GND -> unconnected-(J10-GND_1-PadG1)
- J10 pad G2: GND -> unconnected-(J10-GND_2-PadG2)
- J10 pad G3: GND -> unconnected-(J10-GND_3-PadG3)
- J10 pad G4: GND -> unconnected-(J10-GND_4-PadG4)
- J2 pad 1: Net-(J2-Pin_1) -> GND
- J2 pad 2: Net-(J2-Pin_2) -> /power/5V_proUPS
- J4 pad MP: GND -> unconnected-(J4-MountPin-PadMP)_1
- J5 pad 1: /CAN 4/CAN- -> /computer/3V3_CAM
- J5 pad 2: /CAN 4/CAN+ -> /computer/MIPI0.SDA
- J6 pad MP: GND -> unconnected-(J6-MountPin-PadMP)_1
- J7 pad G1: GND -> unconnected-(J7-GND_1-PadG1)
- J7 pad G2: GND -> unconnected-(J7-GND_2-PadG2)
- J7 pad G3: GND -> unconnected-(J7-GND_3-PadG3)
- J7 pad G4: GND -> unconnected-(J7-GND_4-PadG4)
- J8 pad 1: Net-(J11-Pin_1) -> Net-(J8-Pin_1)
- J8 pad 10: /vcu mcu/current loop sensors/CL_CH5 -> Net-(J8-Pin_10)
- J8 pad 11: Net-(J11-Pin_11) -> Net-(J8-Pin_11)
- J8 pad 12: /vcu mcu/current loop sensors/CL_CH6 -> Net-(J8-Pin_12)
- J8 pad 13: Net-(J11-Pin_13) -> Net-(J8-Pin_13)
- J8 pad 14: /vcu mcu/current loop sensors/CL_CH7 -> Net-(J8-Pin_14)
- J8 pad 15: Net-(J11-Pin_15) -> Net-(J8-Pin_15)
- J8 pad 16: /vcu mcu/current loop sensors/CL_CH8 -> Net-(J8-Pin_16)
- J8 pad 17: Net-(J11-Pin_17) -> Net-(J8-Pin_17)
- J8 pad 18: /vcu mcu/current loop sensors/CL_CH9 -> Net-(J8-Pin_18)
- J8 pad 19: Net-(J11-Pin_19) -> Net-(J8-Pin_19)
- J8 pad 2: /vcu mcu/current loop sensors/CL_CH1 -> Net-(J8-Pin_2)
- J8 pad 20: /vcu mcu/current loop sensors/CL_CH10 -> Net-(J8-Pin_20)
- J8 pad 21: Net-(J11-Pin_21) -> Net-(J8-Pin_21)
- J8 pad 22: /vcu mcu/current loop sensors/CL_CH11 -> Net-(J8-Pin_22)
- J8 pad 23: Net-(J11-Pin_23) -> Net-(J8-Pin_23)
- J8 pad 24: /vcu mcu/current loop sensors/CL_CH12 -> Net-(J8-Pin_24)
- J8 pad 25: Net-(J11-Pin_25) -> Net-(J8-Pin_25)
- J8 pad 26: /vcu mcu/current loop sensors/CL_CH13 -> Net-(J8-Pin_26)
- J8 pad 27: Net-(J11-Pin_27) -> Net-(J8-Pin_27)
- J8 pad 28: /vcu mcu/current loop sensors/CL_CH14 -> Net-(J8-Pin_28)
- J8 pad 29: Net-(J11-Pin_29) -> Net-(J8-Pin_29)
- J8 pad 3: Net-(J11-Pin_3) -> Net-(J8-Pin_3)
- J8 pad 30: /vcu mcu/current loop sensors/CL_CH15 -> Net-(J8-Pin_30)
- J8 pad 4: /vcu mcu/current loop sensors/CL_CH2 -> Net-(J8-Pin_4)
- J8 pad 5: Net-(J11-Pin_5) -> Net-(J8-Pin_5)
- J8 pad 6: /vcu mcu/current loop sensors/CL_CH3 -> Net-(J8-Pin_6)
- J8 pad 7: Net-(J11-Pin_7) -> Net-(J8-Pin_7)
- J8 pad 8: /vcu mcu/current loop sensors/CL_CH4 -> Net-(J8-Pin_8)
- J8 pad 9: Net-(J11-Pin_9) -> Net-(J8-Pin_9)
- J8 pad MP: (no net) -> unconnected-(J8-MountPin-PadMP)_1
- JP1 pad 1: /vcu mcu/NRST -> Net-(JP1-A)
- JP1 pad 2: /vcu mcu/button_raw1 -> GND
- Module1 pad 101: GND -> /computer/compute module/USB.OTG
- Module1 pad 77: +5V_CM -> /computer/compute module/RPI_5V_in
- Module1 pad 78: +3V3_CMOUT -> Net-(Module1A-GPIO_VREF(1.8v/3.3v_Input))
- Module1 pad 79: +5V_CM -> /computer/compute module/RPI_5V_in
- Module1 pad 81: +5V_CM -> /computer/compute module/RPI_5V_in
- Module1 pad 83: +5V_CM -> /computer/compute module/RPI_5V_in
- Module1 pad 85: +5V_CM -> /computer/compute module/RPI_5V_in
- Module1 pad 87: +5V_CM -> /computer/compute module/RPI_5V_in
- Q1 pad 3: Net-(Q1-D) -> /vcu mcu/EXTI7
- R101 pad 1: /vcu mcu/current loop sensors/CL_CH2 -> /vcu mcu/current loop sensors/current loop 2/CL_LOOP
- R103 pad 1: /vcu mcu/current loop sensors/CL_CH3 -> /vcu mcu/current loop sensors/current loop 3/CL_LOOP
- R105 pad 1: /vcu mcu/current loop sensors/CL_CH4 -> /vcu mcu/current loop sensors/current loop 4/CL_LOOP
- R106 pad 1: /vcu mcu/LCD_SCK -> /vcu mcu/current loop sensors/current loop 4/CL_LOOP
- R106 pad 2: unconnected-(R106-Pad2) -> /vcu mcu/CL_CH4
- R107 pad 1: /vcu mcu/current loop sensors/CL_CH5 -> /vcu mcu/current loop sensors/current loop 5/CL_LOOP
- R108 pad 1: /vcu mcu/TP_CS -> /vcu mcu/current loop sensors/current loop 5/CL_LOOP
- R108 pad 2: unconnected-(R108-Pad2) -> /vcu mcu/CL_CH5
- R109 pad 1: /vcu mcu/current loop sensors/CL_CH6 -> /vcu mcu/current loop sensors/current loop 6/CL_LOOP
- R111 pad 1: /vcu mcu/current loop sensors/CL_CH7 -> /vcu mcu/current loop sensors/current loop 7/CL_LOOP
- R112 pad 1: unconnected-(R112-Pad1) -> /vcu mcu/current loop sensors/current loop 7/CL_LOOP
- R112 pad 2: /vcu mcu/TP_MOSI -> /vcu mcu/CL_CH7
- R113 pad 1: /vcu mcu/current loop sensors/CL_CH8 -> /vcu mcu/current loop sensors/current loop 8/CL_LOOP
- R114 pad 1: unconnected-(R114-Pad1) -> /vcu mcu/current loop sensors/current loop 8/CL_LOOP
- R114 pad 2: /vcu mcu/TP_SCK -> /vcu mcu/CL_CH8
- R115 pad 1: /vcu mcu/current loop sensors/CL_CH9 -> /vcu mcu/current loop sensors/current loop 9/CL_LOOP
- R116 pad 1: unconnected-(R116-Pad1) -> /vcu mcu/current loop sensors/current loop 9/CL_LOOP
- R116 pad 2: /vcu mcu/LCD_MOSI -> /vcu mcu/CL_CH9
- R117 pad 1: /vcu mcu/current loop sensors/CL_CH10 -> /vcu mcu/current loop sensors/current loop 10/CL_LOOP
- R119 pad 1: /vcu mcu/current loop sensors/CL_CH11 -> /vcu mcu/current loop sensors/current loop 11/CL_LOOP
- R120 pad 1: /vcu mcu/LED_B11 -> /vcu mcu/current loop sensors/current loop 11/CL_LOOP
- R120 pad 2: Net-(D31-K) -> /vcu mcu/CL_CH11
- R121 pad 1: /vcu mcu/current loop sensors/CL_CH12 -> /vcu mcu/current loop sensors/current loop 12/CL_LOOP
- R122 pad 1: /vcu mcu/LED_B13 -> /vcu mcu/current loop sensors/current loop 12/CL_LOOP
- R122 pad 2: Net-(D33-K) (its old number) -> /vcu mcu/CL_CH12
- R123 pad 1: /vcu mcu/current loop sensors/CL_CH13 -> /vcu mcu/current loop sensors/current loop 13/CL_LOOP
- R125 pad 1: /vcu mcu/current loop sensors/CL_CH14 -> /vcu mcu/current loop sensors/current loop 14/CL_LOOP
- R127 pad 2: /vcu mcu/NRST -> /stlink/DEBUG.RST
- R140 pad 1: /vcu mcu/current loop sensors/CL_CH15 -> /vcu mcu/current loop sensors/current loop 15/CL_LOOP
- R18 pad 1: /vcu mcu/button_raw3 -> /vcu mcu/current loop sensors/current loop 16/CL_LOOP
- R18 pad 2: +3V3 -> GND
- R19 pad 1: /vcu mcu/button3 -> /vcu mcu/current loop sensors/current loop 16/CL_LOOP
- R19 pad 2: /vcu mcu/button_raw3 -> /vcu mcu/CL_CH16
- R20 pad 1: Net-(D6-K) -> /vcu mcu/current loop sensors/current loop 17/CL_LOOP
- R20 pad 2: /vcu mcu/button_raw1 -> GND
- R21 pad 1: /vcu mcu/button_raw1 -> /vcu mcu/current loop sensors/current loop 17/CL_LOOP
- R21 pad 2: +3V3 -> /vcu mcu/CL_CH17
- R22 pad 1: /vcu mcu/button1 -> /vcu mcu/current loop sensors/current loop 18/CL_LOOP
- R22 pad 2: /vcu mcu/button_raw1 -> GND
- R23 pad 1: Net-(D7-K) -> /vcu mcu/current loop sensors/current loop 18/CL_LOOP
- R23 pad 2: /vcu mcu/button_raw2 -> /vcu mcu/CL_CH18
- R24 pad 1: /vcu mcu/button_raw2 -> /vcu mcu/current loop sensors/current loop 19/CL_LOOP
- R24 pad 2: +3V3 -> GND
- R25 pad 1: /vcu mcu/button2 -> /vcu mcu/current loop sensors/current loop 19/CL_LOOP
- R25 pad 2: /vcu mcu/button_raw2 -> /vcu mcu/CL_CH19
- R26 pad 1: Net-(D8-K) -> /vcu mcu/current loop sensors/current loop 20/CL_LOOP
- R26 pad 2: /vcu mcu/button_raw5 -> GND
- R27 pad 1: /vcu mcu/button_raw5 -> /vcu mcu/current loop sensors/current loop 20/CL_LOOP
- R27 pad 2: +3V3 -> /vcu mcu/CL_CH20
- R28 pad 1: /vcu mcu/current loop sensors/CL_CH1 -> /vcu mcu/current loop sensors/current loop 1/CL_LOOP
- R29 pad 1: Net-(D9-K) -> /vcu mcu/current loop sensors/current loop 1/CL_LOOP
- R29 pad 2: /vcu mcu/button_raw4 -> /vcu mcu/CL_CH1
- R34 pad 2: Net-(U5-NRST) -> Net-(JP1-A)
- R4 pad 1: /power/PWR_LOSS -> /CAN 4/CAN_L
- R4 pad 2: Net-(Q1-D) -> /CAN 2/CAN_L
- R46 pad 1: /DFP0.D+ -> /DFP3.D+
- R47 pad 2: /DFP0.D- -> /DFP3.D-
- R48 pad 1: +3V3_CMOUT -> Net-(D15-K)
- R48 pad 2: Net-(D15-A) -> /computer/compute module/nPWR_LED
- R64 pad 1: Net-(U9-~{RESET}) -> Net-(J8-Pin_34)
- R64 pad 2: +3V3 -> Net-(F22-Pad2)
- R69 pad 1: Net-(J11-Pin_1) -> Net-(J8-Pin_24)
- R69 pad 2: +24V -> Net-(F9-Pad2)
- R7 pad 1: +5V -> +3V3
- R7 pad 2: /power/PWR_LOSS -> /vcu mcu/EXTI7
- R70 pad 1: Net-(J11-Pin_3) -> Net-(J8-Pin_22)
- R70 pad 2: +24V -> Net-(F10-Pad2)
- R71 pad 1: Net-(J11-Pin_5) -> Net-(J8-Pin_20)
- R71 pad 2: +24V -> Net-(F11-Pad2)
- R72 pad 1: Net-(J11-Pin_7) -> Net-(J8-Pin_18)
- R72 pad 2: +24V -> Net-(F12-Pad2)
- R73 pad 1: Net-(J11-Pin_9) -> Net-(J8-Pin_16)
- R73 pad 2: +24V -> Net-(F13-Pad2)
- R74 pad 1: Net-(J11-Pin_11) -> Net-(J8-Pin_14)
- R74 pad 2: +24V -> Net-(F14-Pad2)
- R75 pad 1: Net-(J11-Pin_13) -> Net-(J8-Pin_12)
- R75 pad 2: +24V -> Net-(F15-Pad2)
- R76 pad 1: Net-(J11-Pin_15) -> Net-(J8-Pin_10)
- R76 pad 2: +24V -> Net-(F16-Pad2)
- R77 pad 1: Net-(J11-Pin_17) -> Net-(J8-Pin_8)
- R77 pad 2: +24V -> Net-(F17-Pad2)
- R78 pad 1: Net-(J11-Pin_19) -> Net-(J8-Pin_6)
- R78 pad 2: +24V -> Net-(F18-Pad2)
- R79 pad 1: Net-(J11-Pin_21) -> Net-(J8-Pin_4)
- R79 pad 2: +24V -> Net-(F19-Pad2)
- R80 pad 1: Net-(J11-Pin_23) -> Net-(J8-Pin_2)
- R80 pad 2: +24V -> Net-(F20-Pad2)
- R81 pad 1: Net-(J11-Pin_25) -> Net-(J8-Pin_39)
- R81 pad 2: +24V -> /vcu mcu/current loop sensors/current loop 1/CL_LOOP
- R82 pad 1: Net-(J11-Pin_27) -> Net-(J8-Pin_37)
- R82 pad 2: +24V -> /vcu mcu/current loop sensors/current loop 2/CL_LOOP
- R83 pad 1: Net-(J11-Pin_29) -> Net-(J8-Pin_35)
- R83 pad 2: +24V -> /vcu mcu/current loop sensors/current loop 3/CL_LOOP
- R97 pad 1: Net-(D29-K) -> Net-(J8-Pin_7)
- R97 pad 2: GND -> /vcu mcu/current loop sensors/current loop 17/CL_LOOP
- R98 pad 1: Net-(Q3-G) (its old number) -> Net-(J8-Pin_5)
- R98 pad 2: /vcu mcu/RTD light gate -> /vcu mcu/current loop sensors/current loop 18/CL_LOOP
- R99 pad 1: GND -> Net-(J8-Pin_3)
- R99 pad 2: Net-(Q3-G) (its old number) -> /vcu mcu/current loop sensors/current loop 19/CL_LOOP
- SW1 pad 1: GND -> /computer/compute module/PWR_BTN
- SW1 pad 2: /computer/compute module/PWR_BTN -> GND
- SW2 pad 2: /vcu mcu/NRST -> /stlink/DEBUG.RST
- U10 pad 1: +5V -> /CAN 2/CAN.TX
- U10 pad 10: /vcu mcu/SPI4_LEDPWM_5VTTL -> /computer/40P.GPIO21
- U10 pad 11: GND -> /computer/40P.GPIO20
- U10 pad 12: GND -> /computer/40P.GPIO19
- U10 pad 13: GND -> /computer/40P.GPIO18
- U10 pad 14: /vcu mcu/SPI4_LEDPWM -> +3V3
- U10 pad 2: GND -> /CAN 2/CAN.RX
- U10 pad 4: /vcu mcu/SPI4_SCK_5VTTL -> /computer/40P.GPIO13
- U10 pad 5: /vcu mcu/SPI4_CS_5VTTL -> Net-(U10-OSC2)
- U10 pad 6: /vcu mcu/SPI4_MISO_5VTTL -> Net-(U10-OSC1)
- U10 pad 7: /vcu mcu/SPI4_MOSI_5VTTL -> GND
- U12 pad 1: /vcu mcu/SPI4_SCK -> unconnected-(U12-PE2-Pad1)
- U12 pad 10: /vcu mcu/I2C2_SDA -> unconnected-(U12-PF0-Pad10)
- U12 pad 103: /DFP1.D- -> /vcu mcu/USBDN
- U12 pad 104: /DFP1.D+ -> /vcu mcu/USBDP
- U12 pad 11: /vcu mcu/I2C2_SCL -> unconnected-(U12-PF1-Pad11)
- U12 pad 115: /vcu mcu/button4 -> unconnected-(U12-PD1-Pad115)
- U12 pad 118: /vcu mcu/button3 -> unconnected-(U12-PD4-Pad118)
- U12 pad 119: /vcu mcu/button2 -> unconnected-(U12-PD5-Pad119)
- U12 pad 12: /vcu mcu/buzzer_gate -> unconnected-(U12-PF2-Pad12)
- U12 pad 122: /vcu mcu/LCD_CS -> unconnected-(U12-PD6-Pad122)
- U12 pad 123: /vcu mcu/LCD_MOSI -> unconnected-(U12-PD7-Pad123)
- U12 pad 124: /vcu mcu/LCD_MISO -> unconnected-(U12-PG9-Pad124)
- U12 pad 125: /vcu mcu/LCD_DC -> unconnected-(U12-PG10-Pad125)
- U12 pad 126: /vcu mcu/LCD_SCK -> unconnected-(U12-PG11-Pad126)
- U12 pad 127: /vcu mcu/BL_PWM -> unconnected-(U12-PG12-Pad127)
- U12 pad 129: /vcu mcu/TP_MOSI -> unconnected-(U12-PG14-Pad129)
- U12 pad 13: /vcu mcu/current loop sensors/CL_CH1 -> /vcu mcu/CL_CH1
- U12 pad 132: /vcu mcu/TP_CS -> unconnected-(U12-PG15-Pad132)
- U12 pad 133: /vcu mcu/TP_SCK -> unconnected-(U12-PB3-Pad133)
- U12 pad 134: /vcu mcu/TP_MISO -> unconnected-(U12-PB4-Pad134)
- U12 pad 135: /CAN 2/CAN.RX -> /CAN 4/CAN.RX
- U12 pad 136: /CAN 2/CAN.TX -> /CAN 4/CAN.TX
- U12 pad 137: /vcu mcu/SPI4_LEDPWM -> unconnected-(U12-PB7-Pad137)
- U12 pad 139: /CAN 1/CAN.RX -> /CAN 3/CAN.RX
- U12 pad 14: /vcu mcu/current loop sensors/CL_CH2 -> /vcu mcu/CL_CH2
- U12 pad 140: /CAN 1/CAN.TX -> /CAN 3/CAN.TX
- U12 pad 141: /vcu mcu/TP_IRQ -> unconnected-(U12-PE0-Pad141)
- U12 pad 15: /vcu mcu/current loop sensors/CL_CH3 -> /vcu mcu/CL_CH3
- U12 pad 18: /vcu mcu/current loop sensors/CL_CH4 -> /vcu mcu/CL_CH4
- U12 pad 19: /vcu mcu/current loop sensors/CL_CH5 -> /vcu mcu/CL_CH5
- U12 pad 20: /vcu mcu/current loop sensors/CL_CH6 -> /vcu mcu/CL_CH6
- U12 pad 21: /vcu mcu/current loop sensors/CL_CH7 -> /power/24V_SENSE
- U12 pad 22: /vcu mcu/current loop sensors/CL_CH8 -> unconnected-(U12-PF10-Pad22)
- U12 pad 3: /vcu mcu/SPI4_CS -> unconnected-(U12-PE4-Pad3)
- U12 pad 32: /vcu mcu/VDDA_MCU -> Net-(U11-OUT)
- U12 pad 34: /vcu mcu/current loop sensors/CL_CH13 -> unconnected-(U12-PA0-Pad34)
- U12 pad 35: /vcu mcu/current loop sensors/CL_CH14 -> unconnected-(U12-PA1-Pad35)
- U12 pad 36: /vcu mcu/current loop sensors/CL_CH15 -> /vcu mcu/CL_CH7
- U12 pad 37: unconnected-(U11-PA3-Pad37) -> /vcu mcu/CL_CH8
- U12 pad 4: /vcu mcu/SPI4_MISO -> unconnected-(U12-PE5-Pad4)
- U12 pad 40: unconnected-(U11-PA4-Pad40) -> /vcu mcu/CL_CH9
- U12 pad 41: unconnected-(U11-PA5-Pad41) -> /vcu mcu/CL_CH10
- U12 pad 42: unconnected-(U11-PA6-Pad42) -> /vcu mcu/CL_CH11
- U12 pad 43: unconnected-(U11-PA7-Pad43) -> /vcu mcu/CL_CH12
- U12 pad 44: unconnected-(U11-PC4-Pad44) -> /vcu mcu/CL_CH13
- U12 pad 45: unconnected-(U11-PC5-Pad45) -> /vcu mcu/CL_CH14
- U12 pad 46: unconnected-(U11-PB0-Pad46) -> /vcu mcu/CL_CH15
- U12 pad 47: unconnected-(U11-PB1-Pad47) -> /vcu mcu/CL_CH16
- U12 pad 49: /vcu mcu/current loop sensors/CL_CH9 -> /vcu mcu/CL_CH17
- U12 pad 5: /vcu mcu/SPI4_MOSI -> unconnected-(U12-PE6-Pad5)
- U12 pad 50: /vcu mcu/current loop sensors/CL_CH10 -> /vcu mcu/CL_CH18
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Routing:
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- added copper zone on B.Cu, net /computer/compute module/RPI_5V_in
- added copper zone on In1.Cu, net GND
- added copper zone on In2.Cu, net GND
Other:
- board size 102 x 85 mm -> 100 x 90 mm
- copper layers 6 -> 4
- board text added: "100x90mm (screws: M3 92x82mm) Stackup: 6 layer 1.2mm 3313 Via: min 0.3mm drill/Epoxy filled and capped Connector: P2.0 pin header, centered, 2mm from bottom"
- board text removed: "102x85mm (screws: M3 94x77mm) Stackup: 6 layer 1.2mm 3313 Via: min 0.3mm drill/Epoxy filled and capped Connector: P2.0 pin header, centered, 2mm from bottom"
