File: Electrical_Group/VCU_CM5/VCU_CM5.kicad_pcb (KiCad board)
At the start: 4 copper layers, 100 x 90 mm, 426 parts, among them J1 USB3_A, J10 MSD-4-A, J11 STDC14, J2 UPS_CAP, J3 S_SWD, J4 JST_SH, J5 MIPI_CAM_22P, J6 MIPI_DISP_15P, J7 MSD-4-A, J8 Conn_01x30_Socket, J9 Conn_02x15_Odd_Even, Q1 AO3400A, Q2 MMBT3904, Q3 2N7002, SW1 RPI_PWR, SW2 RESET, SW3 BOOT0, U1 LM66100DCK, U10 MCP2518FD, U11 REF3133AIDBZR, U12 STM32H743ZITx, U13 TPS5430DDA, U14 TCAN1042VDRQ1, U15 USB2514B_Bi, U17 TCAN1042VDRQ1, U19 TCAN1042VDRQ1, U2 TLV75733PDRV, U3 TPS5430DDA, U4 TCAN1042VDRQ1, U5 STM32F103CBT6, U6 TLV75733PDRV, U7 TLV75733PDRV, U8 TLV75733PDRV, U9 MCP2518FD, Y1 8MHz X50328MSB2GI, Y2 40Mhz XTM32040000DT00351001, Y3 40Mhz XTM32040000DT00351001, Y4 40Mhz XTM32040000DT00351001, Y5 32.768kHz Q13FC13500004, Y6 24Mhz X322524MOB4SI

Commit message: [VCU_CM5] update to V1.2
Parts:
- removed J11: STDC14, nturt_kicad_lib_EP7:box_header_14P_pitch1.27_smd
- removed R133: 100R, Resistor_SMD:R_0603_1608Metric
- removed R134: 0R, Resistor_SMD:R_0603_1608Metric
- added J24: USB_C_stm32, Connector_USB:USB_C_Receptacle_GCT_USB4105-xx-A_16P_TopMnt_Horizontal, B.Cu at (295.3, 85.2)
- added TP15: S_DIO, TestPoint:TestPoint_Pad_D1.0mm, B.Cu at (260.5, 125.5)
- added TP16: S_CLK, TestPoint:TestPoint_Pad_D1.0mm, B.Cu at (261.9, 124.1)
- added TP17: S_GND, TestPoint:TestPoint_Pad_D1.0mm, B.Cu at (263.3, 122.7)
- BT1: footprint nturt_kicad_lib_EP6:BAT_1056 -> nturt_kicad_lib_EP7:BAT_1056
- D13: value YELLOW led -> GREEN led
- J3: value S_SWD -> RPI_RST; footprint Connector_PinHeader_2.00mm:PinHeader_1x03_P2.00mm_Vertical -> Connector_PinHeader_2.00mm:PinHeader_1x02_P2.00mm_Horizontal
- Module1: footprint CM5IO:Raspberry-Pi-5-Compute-Module -> nturt_kicad_lib_EP7:Raspberry-Pi-5-Compute-Module
- R48, R49: moved to F.Cu
- moved J3 48.1 mm to (206.0, 111.9), turned to 180 degrees
- moved J10 24.5 mm to (255.4, 145.9), turned to 180 degrees
- moved R43 22.3 mm to (267.4, 124.8), turned to 135 degrees
- moved R37 22.0 mm to (266.0, 123.5), turned to -45 degrees
- moved C36 21.6 mm to (260.7, 118.2), turned to -45 degrees
- moved R32 21.6 mm to (262.3, 119.8), turned to -45 degrees
- moved R44 21.3 mm to (265.3, 124.2), turned to 135 degrees
- moved Q2 21.1 mm to (266.6, 127.4), turned to -45 degrees
- moved R31 21.0 mm to (258.7, 117.6), turned to 135 degrees
- moved C35 21.0 mm to (264.2, 123.3), turned to 45 degrees
- moved C37 20.5 mm to (264.6, 124.9), turned to -45 degrees
- moved R30 20.3 mm to (257.6, 117.9), turned to 135 degrees
- moved R45 19.4 mm to (263.9, 126.7), turned to -135 degrees
- moved C32 19.1 mm to (255.7, 118.6), turned to 45 degrees
- moved Y1 18.9 mm to (253.1, 117.4), turned to -135 degrees
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Connections:
- net /CAN 1/CAN.RX renamed /RPI CAN0/CAN.RX
- net /CAN 1/CAN.TX renamed /RPI CAN0/CAN.TX
- net /CAN 1/CAN_H renamed /RPI CAN0/CAN_H
- net /CAN 1/CAN_L renamed /RPI CAN0/CAN_L
- net /CAN 2/CAN.RX renamed /RPI CAN1/CAN.RX
- net /CAN 2/CAN.TX renamed /RPI CAN1/CAN.TX
- net /CAN 2/CAN_H renamed /RPI CAN1/CAN_H
- net /CAN 2/CAN_L renamed /RPI CAN1/CAN_L
- net /CAN 3/CAN.RX renamed /STM32 CAN1/CAN.RX
- net /CAN 3/CAN.TX renamed /STM32 CAN1/CAN.TX
- net /CAN 3/CAN_H renamed /STM32 CAN1/CAN_H
- net /CAN 3/CAN_L renamed /STM32 CAN1/CAN_L
- net /CAN 4/CAN.RX renamed /STM32 CAN2/CAN.RX
- net /CAN 4/CAN.TX renamed /STM32 CAN2/CAN.TX
- net /CAN 4/CAN_H renamed /STM32 CAN2/CAN_H
- net /CAN 4/CAN_L renamed /STM32 CAN2/CAN_L
- net /computer/compute module/USB.D+ renamed /computer/compute module/USB2.D+
- net /computer/compute module/USB.D- renamed /computer/compute module/USB2.D-
- net /computer/compute module/USB.OTG renamed /computer/compute module/USB2.OTG
- C41 pad 1: +5V_CPN -> +5V_CM
- D13 pad 1: /stlink/LED_STLINK -> Net-(D13-K)
- D13 pad 2: Net-(D13-A) -> +3V3
- D14 pad 1: Net-(D14-K) -> GND
- D14 pad 2: /stlink/LED_STLINK -> Net-(D14-A)
- J10 pad G1: unconnected-(J10-GND_1-PadG1) -> GND
- J10 pad G2: unconnected-(J10-GND_2-PadG2) -> GND
- J10 pad G3: unconnected-(J10-GND_3-PadG3) -> GND
- J10 pad G4: unconnected-(J10-GND_4-PadG4) -> GND
- J3 pad 2: /stlink/S_CLK -> /computer/compute module/PWR_BTN
- J4 pad 1: +5V_CPN -> +5V_CM
- J9 pad 10: /vcu mcu/EXTI3 -> /vcu mcu/EXTI5
- J9 pad 11: /vcu mcu/EXTI2 -> /vcu mcu/EXTI4
- J9 pad 12: /vcu mcu/EXTI15 -> /vcu mcu/EXTI3
- J9 pad 13: /vcu mcu/EXTI14 -> /vcu mcu/EXTI2
- J9 pad 14: /vcu mcu/EXTI11 -> /vcu mcu/EXTI15
- J9 pad 15: /vcu mcu/EXTI10 -> /vcu mcu/EXTI14
- J9 pad 16: /vcu mcu/EXTI9 -> /vcu mcu/EXTI11
- J9 pad 17: unconnected-(J9-Pin_17-Pad17) -> /vcu mcu/EXTI10
- J9 pad 18: unconnected-(J9-Pin_18-Pad18) -> /vcu mcu/EXTI9
- J9 pad 23: /vcu mcu/SPI4_CS2 -> /vcu mcu/SPI4_CS1
- J9 pad 24: /vcu mcu/SPI4_CS1 -> /vcu mcu/SPI4_CS0
- J9 pad 7: /vcu mcu/EXTI6 -> /stlink/DEBUG.RST
- J9 pad 8: /vcu mcu/EXTI5 -> /vcu mcu/EXTI7
- J9 pad 9: /vcu mcu/EXTI4 -> /vcu mcu/EXTI6
- Q1 pad 3: /vcu mcu/EXTI7 -> /vcu mcu/EXTI8
- R142 pad 2: /vcu mcu/buzzer/buzzer_s -> /vcu mcu/buzzer_gate
- R35 pad 1: +3V3 -> Net-(D13-K)
- R35 pad 2: Net-(D13-A) -> /stlink/LED_STLINK
- R36 pad 1: Net-(D14-K) -> /stlink/LED_STLINK
- R36 pad 2: GND -> Net-(D14-A)
- R7 pad 2: /vcu mcu/EXTI7 -> /vcu mcu/EXTI8
- U12 pad 117: unconnected-(U12-PD3-Pad117) -> /vcu mcu/buzzer_gate
- U12 pad 63: /vcu mcu/SPI4_CS1 -> /vcu mcu/SPI4_CS0
- U12 pad 64: /vcu mcu/SPI4_CS2 -> /vcu mcu/SPI4_CS1
Routing:
- net /vcu mcu/buzzer_gate: track 0.00 -> 52.6 mm, vias 0 -> 4
- net /vcu mcu/EXTI8: track 0.00 -> 41.7 mm, vias 0 -> 4
- net /stlink/VCP_MCU_UART.RX: track 42.1 -> 3.84 mm, vias 2 -> 1
- net /stlink/DEBUG.CLK: track 35.1 -> 2.37 mm, vias 2 -> 1
- net /stlink/VCP_MCU_UART.TX: track 36.3 -> 4.67 mm, vias 2 -> 1
- net /stlink/DEBUG.DIO: track 32.8 -> 2.59 mm
- net +5V: track 157.5 -> 132.3 mm, vias 8 -> 6
- net /stlink/USB_DP: track 28.8 -> 50.9 mm
- net /stlink/USB_DN: track 27.4 -> 49.0 mm
- net Net-(D15-K): track 1.85 -> 22.9 mm, vias 0 -> 1
- net /vcu mcu/CL_CH8: track 33.4 -> 13.2 mm
- net /computer/compute module/nACT_LED: track 39.6 -> 19.6 mm, vias 2 -> 1
- net /vcu mcu/CL_CH9: track 33.9 -> 14.2 mm
- net Net-(D16-K): track 1.81 -> 21.5 mm, vias 0 -> 1
- net /computer/compute module/nPWR_LED: track 25.2 -> 5.85 mm, vias 0 -> 1
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Other:
- board text added: "+"
- board text added: "+ -"
- board text added: "+3V3"
- board text added: "+5V"
- board text added: "-"
- board text added: "- +"
- board text added: "100x90mm (screws: M3 92x82mm) Stackup: 6 layer 1.2mm 3313 Via: min 0.3mm drill/Epoxy filled and capped Connector: P2.0 pin header, centered, 4mm from bottom"
- board text added: "4-20 mA"
- board text added: "BUZZER"
- board text added: "CAN"
- board text added: "CLK"
- board text added: "CM5 FUSE"
- board text added: "DIO"
- board text added: "GND"
- board text added: "H"
- board text added: "Jack Kuo Jerrymk"
- board text added: "L"
- board text added: "PWRIN"
- board text added: "RPI CAN0"
- board text added: "RPI CAN1"
- board text added: "RPI FAN"
- board text added: "RPI LED"
- board text added: "RPI PWRSW"
- board text added: "RPI SD"
- board text added: "RPI USB3_1"
- board text added: "RPI_5V FUSE"
- board text added: "RST"
- board text added: "RX"
- board text added: "SENSE"
- board text added: "STLINK"
- board text added: "STM CAN1"
- board text added: "STM CAN2"
- board text added: "S_DIO S_CLK GND"
- board text added: "S_RST"
- board text added: "TX"
- board text added: "UPS CAP"
- board text added: "VCU BOOT0"
- board text added: "VCU RESET"
- board text added: "VCU VREF"
- board text added: "VCU_5V FUSE"
- board text added: "VCU_CM5 V1.2"
- board text removed: "100x90mm (screws: M3 92x82mm) Stackup: 6 layer 1.2mm 3313 Via: min 0.3mm drill/Epoxy filled and capped Connector: P2.0 pin header, centered, 2mm from bottom"
- board text removed: "24V IN"
- board text removed: "24V OUT"
- board text removed: "5V OUT"
- board text removed: "BUZ"
- board text removed: "CAN H/L"
- board text removed: "PI Ch0"
- board text removed: "PI Ch1"
- board text removed: "ST Ch0"
- board text removed: "ST Ch1"
- board text removed: "VCU_CM5 V1.0"
- board text removed: "jerrymk 202510xx"

Commit message: Embed fonts, update components
Other:
- board text added: "Jack Kuo"
- board text added: "jerrymk"
- board text removed: "Jack Kuo Jerrymk"
