File: Electrical_Group/VCU_CM5/buzzer.kicad_sch (KiCad schematic)
At the start: 6 parts, among them J15 buzzer, Q4 2N7002

Commit message: [VCU_CM5] update to V1.0
still needs many modifications
Parts:
- removed J15: buzzer, Connector_JST:JST_XH_B2B-XH-A_1x02_P2.50mm_Vertical, symbol Connector_Generic:Conn_01x02
- added TP13: BUZZER_P, nturt_kicad_lib_EP7:edge_pad_1.4mm_0.7mm, symbol Connector:TestPoint_Small
- added TP14: BUZZER_N, nturt_kicad_lib_EP7:edge_pad_1.4mm_0.7mm, symbol Connector:TestPoint_Small
- renumbered D35 to D32, Q4 to Q3, R129 to R142, R130 to R143, R131 to R144
Connections:
- net +24V: now also TP13.1
- net buzzer_outbox: now also TP14.1
Other:
- company: (none) -> NTURacing Team
- title: (none) -> VCU_CM5
Changed lines of the file:
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@@
 	(generator_version "9.0")
 	(paper "A4")
+	(title_block
+		(title "VCU_CM5")
+		(date "2026-02-25")
+		(rev "1.1")
+		(company "NTURacing Team")
+		(comment 1 "Jack Kuo")
+		(comment 2 "Jerry mk")
+	)
 	(junction
 		(at 138.43 99.06)
@@
 	(wire
 		(pts
-			(xy 138.43 88.9) (xy 138.43 99.06)
+			(xy 138.43 90.17) (xy 138.43 99.06)
 		)
 		(stroke
@@
 	(wire
 		(pts
-			(xy 138.43 82.55) (xy 138.43 86.36)
+			(xy 138.43 82.55) (xy 138.43 83.82)
 		)
 		(stroke
@@
 		(pts
 			(xy 127 109.22) (xy 127 106.68)
+		)
+		(stroke
+			(width 0)
+			(type default)
+		)
+	)
+	(wire
+		(pts
+			(xy 149.86 83.82) (xy 138.43 83.82)
+		)
+		(stroke
+			(width 0)
+			(type default)
+		)
+	)
+	(wire
+		(pts
+			(xy 138.43 90.17) (xy 149.86 90.17)
 		)
 		(stroke
@@
 	)
 	(symbol
+		(lib_id "Connector:TestPoint_Small")
+		(at 149.86 90.17 0)
+		(unit 1)
+		(exclude_from_sim no)
+		(in_bom yes)
+		(on_board yes)
+		(dnp no)
+		(property "Reference" "TP14"
+			(at 151.13 88.8999 0)
+			(effects
+				(font
+					(size 1.27 1.27)
+				)
+				(justify left)
+			)
+		)
+		(property "Value" "BUZZER_N"
+			(at 151.13 91.4399 0)
+			(effects
+				(font
+					(size 1.27 1.27)
+				)
+				(justify left)
+			)
+		)
+		(property "Footprint" "nturt_kicad_lib_EP7:edge_pad_1.4mm_0.7mm"
+			(at 154.94 90.17 0)
+			(effects
+				(font
+					(size 1.27 1.27)
+				)
+				(hide yes)
+			)
+		)
+		(property "Datasheet" "~"
+			(at 154.94 90.17 0)
+			(effects
+				(font
+					(size 1.27 1.27)
+				)
+				(hide yes)
+			)
+		)
+		(property "Description" "test point"
+			(at 149.86 90.17 0)
+			(effects
+				(font
+					(size 1.27 1.27)
+				)
+				(hide yes)
+			)
+		)
+		(pin "1"
+		)
+		(instances
+			(project "VCU_CM5"
+				(path "/eb296f24-894e-4ea0-b0cd-3ba211155378/59ca343a-7d66-4d76-8c27-2a427ae9c4b3/a66a3f29-f441-43fa-9af8-e97ffe62ede3"
+					(reference "TP14")
+					(unit 1)
+				)
+			)
+		)
+	)
+	(symbol
 		(lib_id "Device:R_Small")
 		(at 121.92 106.68 270)
@@
 		(dnp no)
 		(fields_autoplaced yes)
-		(property "Reference" "R129"
+		(property "Reference" "R142"
 			(at 121.92 101.6 90)
 			(effects
@@
 			(project "VCU"
 				(path "/eb296f24-894e-4ea0-b0cd-3ba211155378/59ca343a-7d66-4d76-8c27-2a427ae9c4b3/a66a3f29-f441-43fa-9af8-e97ffe62ede3"
-					(reference "R129")
+					(reference "R142")
 					(unit 1)
 				)
@@
 		(dnp no)
 		(fields_autoplaced yes)
-		(property "Reference" "R130"
+		(property "Reference" "R143"
 			(at 129.54 110.49 0)
 			(effects
@@
 			(project "VCU"
 				(path "/eb296f24-894e-4ea0-b0cd-3ba211155378/59ca343a-7d66-4d76-8c27-2a427ae9c4b3/a66a3f29-f441-43fa-9af8-e97ffe62ede3"
-					(reference "R130")
+					(reference "R143")
 					(unit 1)
 				)
@@
 		(dnp no)
 		(fields_autoplaced yes)
-		(property "Reference" "#PWR0202"
+		(property "Reference" "#PWR0188"
 			(at 127 120.65 0)
 			(effects
@@
 			(project "VCU"
 				(path "/eb296f24-894e-4ea0-b0cd-3ba211155378/59ca343a-7d66-4d76-8c27-2a427ae9c4b3/a66a3f29-f441-43fa-9af8-e97ffe62ede3"
-					(reference "#PWR0202")
-					(unit 1)
-				)
-			)
-		)
-	)
-	(symbol
-		(lib_id "Connector_Generic:Conn_01x02")
-		(at 143.51 88.9 0)
-		(mirror x)
-		(unit 1)
-		(exclude_from_sim no)
-		(in_bom yes)
-		(on_board yes)
-		(dnp no)
-		(property "Reference" "J15"
-			(at 146.05 88.9 0)
-			(effects
-				(font
-					(size 1.27 1.27)
-				)
-				(justify left)
-			)
-		)
-		(property "Value" "buzzer"
-			(at 146.05 86.36 0)
-			(effects
-				(font
-					(size 1.27 1.27)
-				)
-				(justify left)
-			)
-		)
-		(property "Footprint" "Connector_JST:JST_XH_B2B-XH-A_1x02_P2.50mm_Vertical"
-			(at 143.51 88.9 0)
-			(effects
-				(font
-					(size 1.27 1.27)
-				)
-				(hide yes)
-			)
-		)
-		(property "Datasheet" "~"
-			(at 143.51 88.9 0)
-			(effects
-				(font
-					(size 1.27 1.27)
-				)
-				(hide yes)
-			)
-		)
-		(property "Description" "Generic connector, single row, 01x02, script generated (kicad-library-utils/schlib/autogen/connector/)"
-			(at 143.51 88.9 0)
-			(effects
-				(font
-					(size 1.27 1.27)
-				)
-				(hide yes)
-			)
-		)
-		(pin "1"
-		)
-		(pin "2"
-		)
-		(instances
-			(project "VCU"
-				(path "/eb296f24-894e-4ea0-b0cd-3ba211155378/59ca343a-7d66-4d76-8c27-2a427ae9c4b3/a66a3f29-f441-43fa-9af8-e97ffe62ede3"
-					(reference "J15")
+					(reference "#PWR0188")
 					(unit 1)
 				)
@@
 		(dnp no)
 		(fields_autoplaced yes)
-		(property "Reference" "Q4"
+		(property "Reference" "Q3"
 			(at 142.24 104.1399 0)
 			(effects
@@
 			(project "VCU"
 				(path "/eb296f24-894e-4ea0-b0cd-3ba211155378/59ca343a-7d66-4d76-8c27-2a427ae9c4b3/a66a3f29-f441-43fa-9af8-e97ffe62ede3"
-					(reference "Q4")
+					(reference "Q3")
 					(unit 1)
 				)
@@
 		(on_board yes)
 		(dnp no)
-		(property "Reference" "D35"
+		(property "Reference" "D32"
 			(at 128.016 83.566 90)
 			(effects
@@
 			(project "VCU"
 				(path "/eb296f24-894e-4ea0-b0cd-3ba211155378/59ca343a-7d66-4d76-8c27-2a427ae9c4b3/a66a3f29-f441-43fa-9af8-e97ffe62ede3"
-					(reference "D35")
+					(reference "D32")
 					(unit 1)
 				)
@@
 		(dnp no)
 		(fields_autoplaced yes)
-		(property "Reference" "#PWR0204"
+		(property "Reference" "#PWR0190"
 			(at 138.43 121.92 0)
 			(effects
@@
 			(project "VCU"
 				(path "/eb296f24-894e-4ea0-b0cd-3ba211155378/59ca343a-7d66-4d76-8c27-2a427ae9c4b3/a66a3f29-f441-43fa-9af8-e97ffe62ede3"
-					(reference "#PWR0204")
+					(reference "#PWR0190")
+					(unit 1)
+				)
+			)
+		)
+	)
+	(symbol
+		(lib_id "Connector:TestPoint_Small")
+		(at 149.86 83.82 0)
+		(unit 1)
+		(exclude_from_sim no)
+		(in_bom yes)
+		(on_board yes)
+		(dnp no)
+		(property "Reference" "TP13"
+			(at 151.13 82.5499 0)
+			(effects
+				(font
+					(size 1.27 1.27)
+				)
+				(justify left)
+			)
+		)
+		(property "Value" "BUZZER_P"
+			(at 151.13 85.0899 0)
+			(effects
+				(font
+					(size 1.27 1.27)
+				)
+				(justify left)
+			)
+		)
+		(property "Footprint" "nturt_kicad_lib_EP7:edge_pad_1.4mm_0.7mm"
+			(at 154.94 83.82 0)
+			(effects
+				(font
+					(size 1.27 1.27)
+				)
+				(hide yes)
+			)
+		)
+		(property "Datasheet" "~"
+			(at 154.94 83.82 0)
+			(effects
+				(font
+					(size 1.27 1.27)
+				)
+				(hide yes)
+			)
+		)
+		(property "Description" "test point"
+			(at 149.86 83.82 0)
+			(effects
+				(font
+					(size 1.27 1.27)
+				)
+				(hide yes)
+			)
+		)
+		(pin "1"
+		)
+		(instances
+			(project "VCU_CM5"
+				(path "/eb296f24-894e-4ea0-b0cd-3ba211155378/59ca343a-7d66-4d76-8c27-2a427ae9c4b3/a66a3f29-f441-43fa-9af8-e97ffe62ede3"
+					(reference "TP13")
 					(unit 1)
 				)
@@
 		(dnp no)
 		(fields_autoplaced yes)
-		(property "Reference" "#PWR0203"
+		(property "Reference" "#PWR0189"
 			(at 138.43 85.09 0)
 			(effects
@@
 			(project "VCU"
 				(path "/eb296f24-894e-4ea0-b0cd-3ba211155378/59ca343a-7d66-4d76-8c27-2a427ae9c4b3/a66a3f29-f441-43fa-9af8-e97ffe62ede3"
-					(reference "#PWR0203")
+					(reference "#PWR0189")
 					(unit 1)
 				)
@@
 		(dnp no)
 		(fields_autoplaced yes)
-		(property "Reference" "R131"
+		(property "Reference" "R144"
 			(at 133.35 91.44 0)
 			(effects
@@
 			(project "VCU"
 				(path "/eb296f24-894e-4ea0-b0cd-3ba211155378/59ca343a-7d66-4d76-8c27-2a427ae9c4b3/a66a3f29-f441-43fa-9af8-e97ffe62ede3"
-					(reference "R131")
-					(unit 1)
-				)
+					(reference "R144")
+					(unit 1)
+				)
