File: Electrical_Group/VCU_CM5/compute module.kicad_sch (KiCad schematic)
At the start: 5 parts

Commit message: [VCU_CM5] update to V1.0
still needs many modifications
Parts:
- added D17: SMBJ5.0A, Diode_SMD:D_SMB, symbol PCM_Diode_TVS_AKL:SMBJ5.0A
- added F4: RPI_FUSE_5A, Fuse:Fuse_1206_3216Metric_Pad1.42x1.75mm_HandSolder, symbol Device:Fuse_Small
- added NT1: NetTie, NetTie:NetTie-2_SMD_Pad0.5mm, symbol Device:NetTie_2
- renumbered R65 to R57, R66 to R58, R67 to R59, R68 to R60
Connections:
- net 5V_IN: now also F4.1; no longer Module1.77 (+5v_(Input)), Module1.79 (+5v_(Input)), Module1.81 (+5v_(Input)), Module1.83 (+5v_(Input)), Module1.85 (+5v_(Input)), Module1.87 (+5v_(Input))
- net GND: now also D17.2 (A)
- net GPIO_VREF: now also NT1.1; no longer Module1.78 (GPIO_VREF(1.8v/3.3v_Input))
- net USB_D+ renamed USB2.D+
- net USB_D- renamed USB2.D-
- net USB_OTG renamed USB2.OTG
- new net: Module1.78 (GPIO_VREF(1.8v/3.3v_Input)), NT1.2
- new net RPI_5V_in: D17.1 (K), F4.2, Module1.77 (+5v_(Input)), Module1.79 (+5v_(Input)), Module1.81 (+5v_(Input)), Module1.83 (+5v_(Input)), Module1.85 (+5v_(Input)), Module1.87 (+5v_(Input))
Other:
- company: (none) -> NTURacing Team
- title: (none) -> VCU_CM5
