File: Electrical_Group/VCU_CM5/computer.kicad_sch (KiCad schematic)
At the start: 39 parts, among them J10 MSD-4-A, J7 MIPI_CAM_22P, J8 JST_SH, J9 MIPI_DISP_15P, SW1 POWER_BTN, U19 MCP2515-xST, U6 TLV75733PDRV, U7 TLV75733PDRV, U8 TLV75733PDRV, U9 MCP2515-xST, Y2 12MHz 830105420809, Y6 12MHz 830105420809

Commit message: [VCU_CM5] update to V1.0
still needs many modifications
Parts:
- removed C54: 30p, Capacitor_SMD:C_0402_1005Metric, symbol Device:C_Small
- removed J7: MIPI_CAM_22P, dd-fmu:Amphenol_SFV22R-2STE1HLF_1x22-1MP_P0.50mm_Horizontal_TopContact, symbol Connector_Generic_MountingPin:Conn_01x22_MountingPin
- removed R150, R64: 10k, Resistor_SMD:R_0402_1005Metric, symbol Device:R_Small
- removed U19, U9: MCP2515-xST, Package_SO:TSSOP-20_4.4x6.5mm_P0.65mm, symbol Interface_CAN_LIN:MCP2515-xST
- removed Y2: 12MHz 830105420809, Crystal:Crystal_SMD_3225-4Pin_3.2x2.5mm, symbol Device:Crystal_GND24
- added C51: 30p, Capacitor_SMD:C_0402_1005Metric, symbol Device:C_Small
- added D15: GREEN_LED, LED_SMD:LED_0603_1608Metric, symbol Device:LED_Small
- added J5: MIPI_CAM_22P, Connector_FFC-FPC:Hirose_FH12-22S-0.5SH_1x22-1MP_P0.50mm_Horizontal, symbol Connector_Generic_MountingPin:Conn_01x22_MountingPin
- added R48: 680R, Resistor_SMD:R_0402_1005Metric, symbol Device:R_Small
- added U10, U9: MCP2518FD, Package_SO:SOIC-14_3.9x8.7mm_P1.27mm, symbol Interface_CAN_LIN:MCP2517FD-xSL
- added Y3: 40Mhz XTM32040000DT00351001, Crystal:Crystal_SMD_3225-4Pin_3.2x2.5mm, symbol Device:Crystal_GND24
- D16: renamed from D15; value RED -> RED_LED
- J4: renamed from J8; footprint Connector_JST:JST_SH_BM04B-SRSS-TB_1x04-1MP_P1.00mm_Vertical -> Connector_JST:JST_SH_SM04B-SRSS-TB_1x04-1MP_P1.00mm_Horizontal
- J7: renamed from J10; footprint SamacSys_Parts_EP6:MSD4A -> nturt_kicad_lib_EP7:MSD4A; symbol SamacSys_Parts:MSD-4-A -> nturt_kicad_lib_EP7:MSD-4-A
- SW1: value POWER_BTN -> RPI_PWR; footprint Button_Switch_SMD:SW_SPST_PTS810 -> Button_Switch_SMD:SW_Tactile_SPST_NO_Straight_CK_PTS636Sx25SMTRLFS
- Y2: renamed from Y6; value 12MHz 830105420809 -> 40Mhz XTM32040000DT00351001
- renumbered C43 to C40, C44 to C41, C45 to C42, C46 to C43, C47 to C44, C48 to C45, C49 to C46, C50 to C47, C51 to C48, C52 to C49, C144 to C50, C145 to C52, C146 to C54, J9 to J6, R56 to R49, R57 to R50, R58 to R51, R59 to R52, R60 to R53, R61 to R54, R62 to R55, R63 to R56
Connections:
- net +5V_CPN is gone; now on net +5V_CM: C41.1, J4.1 (Pin_1)
- net +3V3: now also U10.14 (VDD), U9.14 (VDD)
- net +3V3_CMOUT: now also D16.2 (A), D15.2 (A); no longer R49.1
- net 40P.GPIO13: now also U10.4 (~{INT})
- net 40P.GPIO17: now also U9.13 (~{CS})
- net 40P.GPIO18: now also U10.13 (~{CS})
- net 40P.GPIO19: now also U10.12 (SDO), U9.12 (SDO)
- net 40P.GPIO20: now also U10.11 (SDI), U9.11 (SDI)
- net 40P.GPIO21: now also U10.10 (SCK), U9.10 (SCK)
- net 40P.GPIO22: now also U9.4 (~{INT})
- net CAN0.RX: now also U9.2 (RXCAN)
- net CAN0.TX: now also U9.1 (TXCAN)
- net CAN1.RX: now also U10.2 (RXCAN)
- net CAN1.TX: now also U10.1 (TXCAN)
- net GND: now also SW1.2, C51.2, J5.10 (Pin_10), J5.13 (Pin_13), J5.16 (Pin_16), J5.19 (Pin_19), J5.22 (Pin_22), J5.4 (Pin_4), J5.7 (Pin_7), J5.MP (MountPin), U10.7 (VSS), U9.7 (VSS), Y3.2, Y3.4; no longer J4.MP (MountPin), J6.MP (MountPin), J7.G1 (GND_1), J7.G2 (GND_2), J7.G3 (GND_3), J7.G4 (GND_4), SW1.1
- net MIPI0.C_N: now also J5.15 (Pin_15)
- net MIPI0.C_P: now also J5.14 (Pin_14)
- net MIPI0.D0_N: now also J5.21 (Pin_21)
- net MIPI0.D0_P: now also J5.20 (Pin_20)
- net MIPI0.D1_N: now also J5.18 (Pin_18)
- net MIPI0.D1_P: now also J5.17 (Pin_17)
- net MIPI0.D2_N: now also J5.12 (Pin_12)
- net MIPI0.D2_P: now also J5.11 (Pin_11)
- net MIPI0.D3_N: now also J5.9 (Pin_9)
- net MIPI0.D3_P: now also J5.8 (Pin_8)
- net MIPI0.GPIO0: now also J5.6 (Pin_6)
- net MIPI0.GPIO1: now also J5.5 (Pin_5)
- net MIPI0.SCL: now also J5.3 (Pin_3)
- net MIPI0.SDA: now also J5.2 (Pin_2)
- net compute module/PWR_BTN: now also SW1.1; no longer SW1.2
- net compute module/nACT_LED: now also R49.2; no longer D16.1 (K)
- net compute module/nPWR_LED: now also R48.2
- net at C53.1: now also U10.6 (OSC1), Y3.1
- net at C50.1, Y2.3: now also U9.5 (OSC2)
- net at C52.1, Y2.1: now also U9.6 (OSC1)
- net 3V3_HUB renamed 3V3_CAM
- net 3V3_CAM: now also J5.1 (Pin_1)
- new net: C51.1, U10.5 (OSC2), Y3.3
- new net: D16.1 (K), R49.1
- new net: D15.1 (K), R48.1
- no-connect marks 18 -> 23
Other:
- sheet compute module ports: added USB2{D+ D- OTG}; removed USB_D+, USB_D-, USB_OTG
- company: (none) -> NTURacing Team
- title: (none) -> VCU_CM5
- moved on the sheet: C41, C43, C44, C45, C46, C47, C48, C49, C50, C52, C54, D16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
