File: Electrical_Group/VCU_CM5/computer.kicad_sch (KiCad schematic)
At the start: 39 parts, among them J4 JST_SH, J5 MIPI_CAM_22P, J6 MIPI_DISP_15P, J7 MSD-4-A, SW1 RPI_PWR, U10 MCP2518FD, U6 TLV75733PDRV, U7 TLV75733PDRV, U8 TLV75733PDRV, U9 MCP2518FD, Y2 40Mhz XTM32040000DT00351001, Y3 40Mhz XTM32040000DT00351001

Commit message: [VCU_CM5] update to V1.2
Parts:
- added J3: RPI_RST, Connector_PinHeader_2.00mm:PinHeader_1x02_P2.00mm_Horizontal, symbol Connector_Generic:Conn_01x02
Connections:
- net GND: now also J3.1 (Pin_1)
- net compute module/PWR_BTN: now also J3.2 (Pin_2)
Other:
- moved on the sheet: C40, C41, C42, C43, C44, C45, C46, C47, C48, C49, C50, C51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
