File: Electrical_Group/VCU_CM5/current loop.kicad_sch (KiCad schematic)
At the start: 4 parts

Commit message: [VCU_CM5] update to V1.0
still needs many modifications
Parts:
- added R19: 100R, Resistor_SMD:R_0603_1608Metric, symbol Device:R_Small
- C20: renamed from C33; value 1n -> 1u
- D7: renamed from D12; footprint Diode_SMD:D_SOD-523 -> Diode_SMD:D_SOD-323
- renumbered C34 to C21, R38 to R18
Connections:
- net CL_LOOP: now also R19.1; no longer C21.1, D7.1 (K)
- new net CL_SIG: C21.1, D7.1 (K), R19.2
Other:
- company: (none) -> NTURacing Team
- title: (none) -> VCU_CM5
