File: Electrical_Group/VCU_CM5/m2.kicad_sch (KiCad schematic)
At the start: 18 parts, among them J17 Bus_M.2_Socket_M, U15 AP3441SHE-7B, U16 ASEK-32.768KHZ-L-R-T

Commit message: [VCU_CM5] update to V1.0
still needs many modifications
Parts:
- renumbered C131 to C132, C132 to C133, C133 to C134, C134 to C135, C135 to C138, C136 to C139, C137 to C140, C138 to C141, C139 to C142, D39 to D37, J17 to J12, L5 to L4, R140 to R153, R141 to R154, R142 to R157, R143 to R159, U15 to U16, U16 to U18
Other:
- company: (none) -> NTURacing Team
- title: (none) -> VCU_CM5
