File: Electrical_Group/VCU_CM5/usb_hub.kicad_sch (KiCad schematic)
At the start: 15 parts, among them U14 USB2514B_Bi, Y5 24MHz

Commit message: [VCU_CM5] update to V1.0
still needs many modifications
Parts:
- removed Y5: 24MHz, Crystal:Crystal_SMD_5032-2Pin_5.0x3.2mm, symbol Device:Crystal
- added Y6: 24Mhz X322524MOB4SI, Crystal:Crystal_SMD_3225-4Pin_3.2x2.5mm, symbol Device:Crystal_GND24
- renumbered C121 to C122, C122 to C123, C123 to C124, C124 to C125, C125 to C126, C126 to C127, C127 to C128, C128 to C129, C129 to C130, C130 to C131, R137 to R150, R138 to R151, R139 to R152, U14 to U15
Connections:
- net GND: now also Y6.2, Y6.4
- net at C123.1, U15.32 (XTALOUT): now also Y6.3
- net at C122.1, U15.33 (XTALIN/CLKIN): now also Y6.1
Other:
- company: (none) -> NTURacing Team
- title: (none) -> VCU_CM5
- moved on the sheet: C122, C123
