File: Powertrain_Group/DIY_MGJ6/DIY_MGJ6.kicad_pcb (KiCad board)
At the start: 2 copper layers, 39.3 x 28.1 mm, 33 parts, among them J1 INPUT, J2 OUTPUT, T1 FC-STR0809-4.5V-5.0V-5.0W, U1 SN6507DGQ, U17 AMS1117-3.3, U2 TPS5430DDAR

Commit message: [DIY_MGJ6] V1.1 minor change
Parts:
- T1: footprint Transformer_SMD_Wurth:T_Wurth_WE-PPTI-1308 -> nturt_kicad_lib_EP7:T_Wurth_WE-PPTI-1308
- moved J1 9.96 mm to (114.3, 86.4)
- moved J2 9.96 mm to (147.3, 86.4)
- moved C1 9.87 mm to (115.7, 89.5)
- moved C11 9.87 mm to (140.0, 104.6)
- moved C12 9.87 mm to (134.6, 95.1)
- moved C2 9.87 mm to (134.4, 103.8)
- moved C3 9.87 mm to (142.1, 86.2)
- moved C4 9.87 mm to (143.0, 82.7)
- moved C5 9.87 mm to (130.8, 82.7)
- moved C6 9.87 mm to (147.6, 91.1)
- moved C7 9.87 mm to (116.8, 98.0)
- moved D2 9.87 mm to (130.3, 100.7)
- moved D5 9.87 mm to (144.0, 101.7)
- moved L3 9.87 mm to (148.4, 100.3)
- moved R2 9.87 mm to (113.4, 91.7)
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Routing:
- net Net-(D5-K): track 4.77 -> 14.1 mm, vias 2 -> 0
- net /ISO_VEE: track 16.2 -> 14.8 mm, vias 12 -> 15
- removed copper zone on F.Cu, net Net-(D5-K)
Other:
- board text added: "EP7 DIY_MGJ6 V1.1 26/03/06 Shinkansen942 Jack Kuo"
