File: Powertrain_Group/DIY_MGJ6/DIY_MGJ6.kicad_sch (KiCad schematic)
At the start: 33 parts, among them J1 INPUT, J2 OUTPUT, T1 FC-STR0809-4.5V-5.0V-5.0W, U1 SN6507DGQ, U17 AMS1117-3.3, U2 TPS5430DDAR

Commit message: [DIY_MGJ6] V1.1 minor change
Parts:
- T1: footprint Transformer_SMD_Wurth:T_Wurth_WE-PPTI-1308 -> nturt_kicad_lib_EP7:T_Wurth_WE-PPTI-1308; symbol Transformer_Wurth_WE-PPTI:1308_750319697 -> nturt_kicad_lib_EP7:Transformer_Wurth_1308_750319697
- U2: symbol nturt_kicad_lib_EP6:TPS5430DDAR -> nturt_kicad_lib_EP7:TPS5430DDAR
Other:
- note added: "V1.0 init by Shinkansen942 V1.1 modify by Jack Kuo"
- company: (none) -> NTURacing
- title: (none) -> DIY_MGJ6
