File: Powertrain_Group/INV_Boost_Power/INV_Boost_Power.kicad_pcb (KiCad board)
At the start: 2 copper layers, 187 x 55 mm, 60 parts, among them J1 Conn_01x08, Q1 ADR014B12MC, Q2 ADR014B12MC, U1 CKSR_75-NP, U2 1ED3122MC12HXUMA1, U3 MGJ6D241505SC, U4 1ED3122MC12HXUMA1, U5 MGJ6D241505SC, U6 AMC3302

Commit message: [INV_Boost_Iso] V1.1
Parts:
- C15, C16, C17, C18: footprint Personal:C_8060_Murata_DK1 -> nturt_kicad_lib_EP7:C_8060_Murata_DK1
- C3: footprint Personal:CeraLink_FA3 -> nturt_kicad_lib_EP7:TKD_CeraLink_FA3
- L1: footprint Inductor_THT_Wurth_New:L_Wurth_WE-HCFT-3635_74437636352702 -> nturt_kicad_lib_EP7:L_Wurth_WE-HCFT-3635_74437636352702
- MP1, MP2, MP3, MP4: footprint REDCUBE_THT_Wurth:MP_Wurth_WP-THRSH_74651175R -> nturt_kicad_lib_EP7:MP_Wurth_WP-THRSH_74651175R
- Q1, Q2: footprint Personal:TO-247-4_Horizontal_TabUp_NoHole -> nturt_kicad_lib_EP7:TO-247-4_Horizontal_TabUp_NoHole
- U2, U4: footprint Snapeda:PG-DSO-8-66-L -> Package_SO:Infineon_PG-DSO-8-59_7.5x6.3mm
- U3, U5: footprint Snapeda:PMPN -> nturt_kicad_lib_EP7:Murata_PMPN
- moved U5 1.09 mm to (155.3, 126.8)
- moved R1 0.81 mm to (180.2, 100.8)
- moved R3 0.80 mm to (180.2, 98.8)
- moved R6 0.80 mm to (180.2, 120.4)
- moved R8 0.80 mm to (180.2, 118.5)
- moved C5 0.50 mm to (178.3, 103.3)
- moved U2 0.41 mm to (172.6, 99.8)
- moved C8 0.40 mm to (178.3, 123.1)
- moved U4 0.40 mm to (172.6, 119.5)
- moved C7 0.39 mm to (164.5, 97.9)
- moved C9 0.10 mm to (168.4, 123.9)
- moved D2 0.10 mm to (159.9, 124.9)
- moved R7 0.10 mm to (165.1, 123.5)
- moved R9 0.10 mm to (159.6, 121.5)
Routing:
- net /HV_IN-: track 26.1 -> 0.00 mm, vias 100 -> 105
- net Net-(U2-VCC2): track 36.2 -> 30.0 mm
- net /LS: track 31.0 -> 33.2 mm
- net /ISO_24V: track 63.4 -> 61.8 mm
- net Net-(U4-VCC2): track 18.7 -> 20.1 mm
- net /HS: track 39.2 -> 37.9 mm
- net Net-(U4-VEE2): track 33.7 -> 34.9 mm
- net /ISO_GND: track 247.0 -> 247.7 mm
- net Net-(U4-IN+): track 1.33 -> 2.03 mm
- net Net-(U4-IN-): track 1.36 -> 2.06 mm
- net /INN: track 101.4 -> 102.0 mm
- net Net-(U2-VEE2): track 40.9 -> 40.3 mm
- net /INP: track 101.8 -> 102.4 mm
