File: Powertrain_Group/INV_Boost_Power/INV_Boost_Power.kicad_sch (KiCad schematic)
At the start: 55 parts, among them J1 Conn_01x08, Q1 ADR014B12MC, Q2 ADR014B12MC, U1 CKSR_75-NP, U2 1ED3122MC12HXUMA1, U3 MGJ6D241505SC, U4 1ED3122MC12HXUMA1, U5 MGJ6D241505SC

Commit message: [INV_Boost_Iso] V1.1
Parts:
- C15, C16, C17, C18: footprint Personal:C_8060_Murata_DK1 -> nturt_kicad_lib_EP7:C_8060_Murata_DK1
- C3: footprint Personal:CeraLink_FA3 -> nturt_kicad_lib_EP7:TKD_CeraLink_FA3
- L1: footprint Inductor_THT_Wurth_New:L_Wurth_WE-HCFT-3635_74437636352702 -> nturt_kicad_lib_EP7:L_Wurth_WE-HCFT-3635_74437636352702
- MP1, MP2, MP3, MP4: footprint REDCUBE_THT_Wurth:MP_Wurth_WP-THRSH_74651175R -> nturt_kicad_lib_EP7:MP_Wurth_WP-THRSH_74651175R; symbol REDCUBE_Wurth_WP-THRSH:74651175R -> nturt_kicad_lib_EP7:Mounting_Screw_74651175R
- Q1, Q2: footprint Personal:TO-247-4_Horizontal_TabUp_NoHole -> nturt_kicad_lib_EP7:TO-247-4_Horizontal_TabUp_NoHole
- U2, U4: footprint Snapeda:PG-DSO-8-66-L -> Package_SO:Infineon_PG-DSO-8-59_7.5x6.3mm; symbol Snapeda:1ED3122MC12HXUMA1 -> nturt_kicad_lib_EP7:1ED3122MC12HXUMA1
- U3, U5: footprint Snapeda:PMPN -> nturt_kicad_lib_EP7:Murata_PMPN; symbol Snapeda:MGJ6D241505SC -> nturt_kicad_lib_EP7:MGJ6D241505SC
Other:
- note added: "V1.0 init by Shinkansen942 V1.1 minor modification by Jack Kuo"
- company: (none) -> NTURacing
- title: (none) -> INV_Boost_Power
Changed lines of the file:
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@@
 	(generator_version "9.0")
 	(paper "A4")
+	(title_block
+		(title "INV_Boost_Power")
+		(date "2026-03-06")
+		(rev "1.1")
+		(company "NTURacing")
+		(comment 1 "Shinkansen942")
+		(comment 2 "Jack Kuo")
+	)
+	(text "V1.0 init by Shinkansen942\nV1.1 minor modification by Jack Kuo"
+		(exclude_from_sim no)
+		(at 153.416 85.344 0)
+		(effects
+			(font
+				(size 1.27 1.27)
+			)
+			(justify left top)
+		)
+	)
 	(junction
 		(at 113.03 64.77)
@@
 	)
 	(junction
-		(at 246.38 140.97)
-		(diameter 0)
-		(color 0 0 0 0)
-	)
-	(junction
 		(at 154.94 125.73)
 		(diameter 0)
@@
 	)
 	(junction
-		(at 246.38 115.57)
-		(diameter 0)
-		(color 0 0 0 0)
-	)
-	(junction
 		(at 127 48.26)
 		(diameter 0)
@@
 	(wire
 		(pts
-			(xy 36.5199 96.52) (xy 36.83 96.52)
-		)
-		(stroke
-			(width 0)
-			(type default)
-		)
-	)
-	(wire
-		(pts
 			(xy 93.98 115.57) (xy 93.98 125.73)
 		)
@@
 	)
 	(label "ISO_24V"
-		(at 36.5199 96.52 0)
+		(at 36.83 96.52 0)
 		(effects
 			(font
@@
 	)
 	(symbol
-		(lib_id "Snapeda:MGJ6D241505SC")
+		(lib_id "nturt_kicad_lib_EP7:MGJ6D241505SC")
 		(at 236.22 125.73 0)
 		(mirror y)
@@
 			)
 		)
-		(property "Footprint" "Snapeda:PMPN"
+		(property "Footprint" "nturt_kicad_lib_EP7:Murata_PMPN"
 			(at 236.22 125.73 0)
 			(effects
@@
 			)
 		)
-		(property "Footprint" "Inductor_THT_Wurth_New:L_Wurth_WE-HCFT-3635_74437636352702"
+		(property "Footprint" "nturt_kicad_lib_EP7:L_Wurth_WE-HCFT-3635_74437636352702"
 			(at 151.13 69.85 0)
 			(effects
@@
 	)
 	(symbol
-		(lib_id "Snapeda:1ED3122MC12HXUMA1")
+		(lib_id "nturt_kicad_lib_EP7:1ED3122MC12HXUMA1")
 		(at 120.65 144.78 0)
 		(unit 1)
@@
 			)
 		)
-		(property "Footprint" "Snapeda:PG-DSO-8-66-L"
+		(property "Footprint" "Package_SO:Infineon_PG-DSO-8-59_7.5x6.3mm"
 			(at 100.33 140.97 0)
 			(effects
@@
 			)
 		)
-		(property "Footprint" "Personal:TO-247-4_Horizontal_TabUp_NoHole"
+		(property "Footprint" "nturt_kicad_lib_EP7:TO-247-4_Horizontal_TabUp_NoHole"
 			(at 180.34 56.515 0)
 			(effects
@@
 	)
 	(symbol
-		(lib_id "REDCUBE_Wurth_WP-THRSH:74651175R")
+		(lib_id "nturt_kicad_lib_EP7:Mounting_Screw_74651175R")
 		(at 83.82 64.77 0)
 		(unit 1)
@@
 			)
 		)
-		(property "Footprint" "REDCUBE_THT_Wurth:MP_Wurth_WP-THRSH_74651175R"
+		(property "Footprint" "nturt_kicad_lib_EP7:MP_Wurth_WP-THRSH_74651175R"
 			(at 96.52 44.45 0)
 			(effects
@@
 			)
 		)
-		(property "Footprint" "Personal:C_8060_Murata_DK1"
+		(property "Footprint" "nturt_kicad_lib_EP7:C_8060_Murata_DK1"
 			(at 64.4652 85.09 0)
 			(effects
@@
 	)
 	(symbol
-		(lib_id "REDCUBE_Wurth_WP-THRSH:74651175R")
+		(lib_id "nturt_kicad_lib_EP7:Mounting_Screw_74651175R")
 		(at 83.82 82.55 180)
 		(unit 1)
@@
 			)
 		)
-		(property "Footprint" "REDCUBE_THT_Wurth:MP_Wurth_WP-THRSH_74651175R"
+		(property "Footprint" "nturt_kicad_lib_EP7:MP_Wurth_WP-THRSH_74651175R"
 			(at 71.12 102.87 0)
 			(effects
@@
 	)
 	(symbol
-		(lib_id "Snapeda:1ED3122MC12HXUMA1")
+		(lib_id "nturt_kicad_lib_EP7:1ED3122MC12HXUMA1")
 		(at 120.65 119.38 0)
 		(unit 1)
@@
 			)
 		)
-		(property "Footprint" "Snapeda:PG-DSO-8-66-L"
+		(property "Footprint" "Package_SO:Infineon_PG-DSO-8-59_7.5x6.3mm"
 			(at 100.33 115.57 0)
 			(effects
@@
 	)
 	(symbol
-		(lib_id "REDCUBE_Wurth_WP-THRSH:74651175R")
+		(lib_id "nturt_kicad_lib_EP7:Mounting_Screw_74651175R")
 		(at 203.2 52.07 180)
 		(unit 1)
@@
 			)
 		)
-		(property "Footprint" "REDCUBE_THT_Wurth:MP_Wurth_WP-THRSH_74651175R"
+		(property "Footprint" "nturt_kicad_lib_EP7:MP_Wurth_WP-THRSH_74651175R"
 			(at 190.5 72.39 0)
 			(effects
@@
 			)
 		)
-		(property "Footprint" "Personal:C_8060_Murata_DK1"
+		(property "Footprint" "nturt_kicad_lib_EP7:C_8060_Murata_DK1"
 			(at 214.3252 39.37 0)
 			(effects
@@
 			)
 		)
-		(property "Footprint" "Personal:CeraLink_FA3"
+		(property "Footprint" "nturt_kicad_lib_EP7:TKD_CeraLink_FA3"
 			(at 100.0252 77.47 0)
 			(effects
@@
 	)
 	(symbol
-		(lib_id "REDCUBE_Wurth_WP-THRSH:74651175R")
+		(lib_id "nturt_kicad_lib_EP7:Mounting_Screw_74651175R")
 		(at 203.2 34.29 0)
 		(unit 1)
@@
 			)
 		)
-		(property "Footprint" "REDCUBE_THT_Wurth:MP_Wurth_WP-THRSH_74651175R"
+		(property "Footprint" "nturt_kicad_lib_EP7:MP_Wurth_WP-THRSH_74651175R"
 			(at 215.9 13.97 0)
 			(effects
@@
 			)
 		)
-		(property "Footprint" "Personal:C_8060_Murata_DK1"
+		(property "Footprint" "nturt_kicad_lib_EP7:C_8060_Murata_DK1"
 			(at 214.3252 46.99 0)
 			(effects
@@
 			)
 		)
-		(property "Footprint" "Personal:TO-247-4_Horizontal_TabUp_NoHole"
+		(property "Footprint" "nturt_kicad_lib_EP7:TO-247-4_Horizontal_TabUp_NoHole"
 			(at 180.34 46.355 0)
 			(effects
@@
 	)
 	(symbol
-		(lib_id "Snapeda:MGJ6D241505SC")
+		(lib_id "nturt_kicad_lib_EP7:MGJ6D241505SC")
 		(at 236.22 151.13 0)
 		(mirror y)
@@
 			)
 		)
-		(property "Footprint" "Snapeda:PMPN"
+		(property "Footprint" "nturt_kicad_lib_EP7:Murata_PMPN"
 			(at 236.22 151.13 0)
 			(effects
@@
 			)
 		)
-		(property "Footprint" "Personal:C_8060_Murata_DK1"
+		(property "Footprint" "nturt_kicad_lib_EP7:C_8060_Murata_DK1"
 			(at 64.4652 69.85 0)
 			(effects
@@
 		)
 		(instances
-			(project "1_phase_15kW_boost_power_stage"
+			(project "INV_Boost_Power"
 				(path "/7625315e-1f21-4ac3-9514-464edd9d9f80"
 					(page "2")
