File: Powertrain_Group/INV_Boost_Power/ISO_CS.kicad_sch (KiCad schematic)
At the start: 5 parts, among them U6 AMC3302

Commit message: [INV_Boost_Iso] V1.1
Other:
- company: (none) -> NTURacing
- title: (none) -> INV_Boost_Power
Changed lines of the file:
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@@
 	(generator_version "9.0")
 	(paper "A4")
+	(title_block
+		(title "INV_Boost_Power")
+		(date "2026-03-06")
+		(rev "1.1")
+		(company "NTURacing")
+		(comment 1 "Shinkansen942")
+		(comment 2 "Jack Kuo")
+	)
 	(junction
 		(at 114.3 104.14)
