File: Powertrain_Group/INV_Boost_Controller/OCPnode.kicad_sch (KiCad schematic)
At the start: 7 parts, among them U14 LM393

Commit message: [INV_Boost_Controller] V1.1
Other:
- company: (none) -> NTURacing
- title: (none) -> INV_Boost_Controller
Changed lines of the file:
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@@
 	(generator_version "9.0")
 	(paper "A4")
+	(title_block
+		(title "INV_Boost_Controller")
+		(date "2026-03-09")
+		(rev "1.1")
+		(company "NTURacing")
+		(comment 1 "Shinkansen942")
+		(comment 2 "Jack Kuo")
+	)
 	(junction
 		(at 166.37 104.14)
