File: Powertrain_Group/INV_Boost_Controller/difftosinglegnd.kicad_sch (KiCad schematic)
At the start: 8 parts, among them U6 INA333AIDGK

Commit message: [INV_Boost_Controller] V1.1
Parts:
- U6: footprint PCM_Package_SO_AKL:MSOP-8_3x3mm_P0.65mm -> Package_SO:VSSOP-8_3x3mm_P0.65mm; symbol PCM_Amplifier_Instrumentation_AKL:INA333AIDGK -> Amplifier_Instrumentation:INA333xxDGK
Other:
- company: (none) -> NTURacing
- title: (none) -> INV_Boost_Controller
- moved on the sheet: R16, R18
