File: Powertrain_Group/INV_Boost_Controller/INV_Boost_Controller.kicad_pcb (KiCad board)
At the start: 4 copper layers, 100 x 100 mm, 262 parts, among them J1 CAN, J10 TEMP, J11 TEMP, J12 TEMP, J13 TEMP, J14 MSD-4-A, J2 CAN, J3 CAN, J4 CAN, J5 15120682601000, J6 LVBattery, J7 LVBattery, J8 USB_C_Receptacle_USB2.0_16P, J9 STDC14, SW1 SW_DIP_x01, SW2 TS-1187A-B-A-B, SW3 TS-1187A-B-A-B, U1 INA333AIDGK, U10 TCAN1042VDRQ1, U11 TCAN1042VDRQ1, U12 SRV05-4, U13 STM32G474VETx, U14 LM393, U15 LM393, U16 INA333AIDGK, U17 INA333AIDGK, U18 LM393, U19 LM393, U2 INA333AIDGK, U20 LM393, U21 LM393, U3 INA333AIDGK, U4 INA333AIDGK, U5 INA333AIDGK, U6 INA333AIDGK, U7 TPS5430DDAR, U8 AMS1117-3.3, U9 REF2033, Y1 48MHz YF4048M00033T8188103

Commit message: [INV_Boost_Controller] V1.1
Parts:
- C1, C2, C3, C4: footprint Personal:C_8060_Murata_DK1 -> nturt_kicad_lib_EP7:C_8060_Murata_DK1
- FL1: footprint Samacsys:ACM70V7012PLTL00 -> nturt_kicad_lib_EP7:Common_Mode_Choke_4A_ACM70V7012PLTL00
- FL2, FL3: footprint Samacsys:EXCX4CE900U -> nturt_kicad_lib_EP7:EXCX4CE900U
- J14: footprint EasyEDA:TF-SMD_HX-TF-CARD-H1.8-SY -> nturt_kicad_lib_EP7:MSD4A
- J5: footprint Samacsys:15120682601000 -> nturt_kicad_lib_EP7:Harting 15120682601000
- J9: footprint Personal:box_header_14P_pitch127 -> nturt_kicad_lib_EP7:box_header_14P_pitch1.27
- L1: footprint PCM_Inductor_SMD_AKL:L_Wuerth_MAPI-3015 -> Inductor_SMD:L_Wuerth_MAPI-3015
- U1, U16, U17, U2, U3, U4, U5, U6: footprint PCM_Package_SO_AKL:MSOP-8_3x3mm_P0.65mm -> Package_SO:VSSOP-8_3x3mm_P0.65mm
- moved J14 1.71 mm to (89.2, 36.0)
Routing:
- net /Diff To Single GNDREF 2/Vout: vias 3 -> 2
- net +3V3: vias 19 -> 18
Other:
- outline, holes or cut-outs redrawn
- board text added: "+ -"
- board text added: "24V"
- board text added: "5V"
- board text added: "B12"
- board text added: "B13"
- board text added: "B14"
- board text added: "B15"
- board text added: "D10"
- board text added: "D11"
- board text added: "D8"
- board text added: "D9"
- board text added: "EP7 INV_Boost_Controller V1.1 26/03/09 Shinkansen Jack Kuo"
- board text added: "H L"
- board text added: "TEMP1"
- board text added: "TEMP2"
- board text added: "TEMP3"
- board text added: "TEMP4"
- board text added: "VBUS"

Commit message: [INV_Boost_Controller] V1.1 again
minor update for jlc
Parts:
- D6: value RED 5V -> WHITE 5V
- D7: value RED 3V3 -> WHITE 3V3
- R20: value 47k 1% -> 47k
- R21: value 15k 1% -> 15k
- Y1: value 48MHz YF4048M00033T8188103 -> X322516MLB4SI (16MHz)
Changed lines of the file:
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@@
 			)
 		)
-		(property "Value" "RED 5V"
+		(property "Value" "WHITE 5V"
 			(at 0 1.43 90)
 			(layer "F.Fab")
@@
 			)
 		)
-		(property "Value" "RED 3V3"
+		(property "Value" "WHITE 3V3"
 			(at 0 1.43 90)
 			(layer "F.Fab")
@@
 			)
 		)
-		(property "Value" "15k 1%"
+		(property "Value" "15k"
 			(at 0 1.43 90)
 			(layer "F.Fab")
@@
 			)
 		)
-		(property "Value" "48MHz YF4048M00033T8188103"
+		(property "Value" "X322516MLB4SI (16MHz)"
 			(at 0 2.95 0)
 			(layer "F.Fab")
@@
 			)
 		)
-		(property "Value" "47k 1%"
+		(property "Value" "47k"
 			(at 0 1.43 90)
 			(layer "F.Fab")
