File: Powertrain_Group/INV_Boost_Controller/mcu.kicad_sch (KiCad schematic)
At the start: 54 parts, among them J10 TEMP, J11 TEMP, J12 TEMP, J13 TEMP, J14 MSD-4-A, J9 STDC14, SW2 TS-1187A-B-A-B, SW3 TS-1187A-B-A-B, U13 STM32G474VETx, Y1 48MHz YF4048M00033T8188103

Commit message: [INV_Boost_Controller] V1.1
Parts:
- J14: footprint EasyEDA:TF-SMD_HX-TF-CARD-H1.8-SY -> nturt_kicad_lib_EP7:MSD4A; symbol SamacSys_Parts_EP6:MSD-4-A -> nturt_kicad_lib_EP7:MSD-4-A; Manufacturer_Name Same Sky -> CUI Devices; Mouser Price/Stock https://www.mouser.co.uk/ProductDetail/Same-Sky/MSD-4-A?qs=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 -> https://www.mouser.co.uk/ProductDetail/CUI-Devices/MSD-4-A?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
- J9: footprint Personal:box_header_14P_pitch127 -> nturt_kicad_lib_EP7:box_header_14P_pitch1.27
Other:
- company: (none) -> NTURacing
- title: (none) -> INV_Boost_Controller
Changed lines of the file:
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@@
 	(generator_version "9.0")
 	(paper "A3")
+	(title_block
+		(title "INV_Boost_Controller")
+		(date "2026-03-09")
+		(rev "1.1")
+		(company "NTURacing")
+		(comment 1 "Shinkansen942")
+		(comment 2 "Jack Kuo")
+	)
 	(rectangle
 		(start 322.58 184.15)
@@
 			)
 		)
+		(property "Sim.Pins" "1=K 2=A"
+			(at 53.34 201.93 0)
+			(effects
+				(font
+					(size 1.27 1.27)
+				)
+				(hide yes)
+			)
+		)
 		(pin "1"
 		)
@@
 			)
 		)
+		(property "Sim.Pins" "1=K 2=A"
+			(at 53.34 226.06 0)
+			(effects
+				(font
+					(size 1.27 1.27)
+				)
+				(hide yes)
+			)
+		)
 		(pin "1"
 		)
@@
 			)
 		)
+		(property "Sim.Pins" "1=K 2=A"
+			(at 43.18 201.93 0)
+			(effects
+				(font
+					(size 1.27 1.27)
+				)
+				(hide yes)
+			)
+		)
 		(pin "1"
 		)
@@
 	)
 	(symbol
-		(lib_id "SamacSys_Parts_EP6:MSD-4-A")
+		(lib_id "nturt_kicad_lib_EP7:MSD-4-A")
 		(at 349.25 194.31 0)
 		(unit 1)
@@
 			)
 		)
-		(property "Footprint" "EasyEDA:TF-SMD_HX-TF-CARD-H1.8-SY"
+		(property "Footprint" "nturt_kicad_lib_EP7:MSD4A"
 			(at 378.46 289.23 0)
 			(effects
@@
 			)
 		)
-		(property "Datasheet" "https://www.sameskydevices.com/product/resource/supplyframepdf/msd-4-a.pdf"
+		(property "Datasheet" "https://www.cuidevices.com/product/resource/pdf/msd-4-a.pdf"
 			(at 378.46 389.23 0)
 			(effects
@@
 			)
 		)
-		(property "Description" "Micro SD Card Connector, 9 Positions, Connector and Ejector, Push In, Auto Eject Out, Surface Mount, 1.8 mm Height Above Board, Gold Flash"
+		(property "Description" "Memory Card Connectors 9 Positions, Push In, Auto Eject Out, SMT, 1.8 mm Height Above Board,"
 			(at 349.25 194.31 0)
 			(effects
@@
 			)
 		)
-		(property "Mouser Price/Stock" "https://www.mouser.co.uk/ProductDetail/Same-Sky/MSD-4-A?qs=Z%252BL2brAPG1Jll%252BQTi%252Btupg%3D%3D"
+		(property "Mouser Price/Stock" "https://www.mouser.co.uk/ProductDetail/CUI-Devices/MSD-4-A?qs=Z%252BL2brAPG1Jll%252BQTi%252Btupg%3D%3D"
 			(at 378.46 789.23 0)
 			(effects
@@
 			)
 		)
-		(property "Manufacturer_Name" "Same Sky"
+		(property "Manufacturer_Name" "CUI Devices"
 			(at 378.46 889.23 0)
 			(effects
@@
 			)
 		)
-		(property "Footprint" "Personal:box_header_14P_pitch127"
+		(property "Footprint" "nturt_kicad_lib_EP7:box_header_14P_pitch1.27"
 			(at 370.84 166.37 0)
 			(effects
@@
 			)
 		)
+		(property "Sim.Pins" "1=K 2=A"
+			(at 33.02 226.06 0)
+			(effects
+				(font
+					(size 1.27 1.27)
+				)
+				(hide yes)
+			)
+		)
 		(pin "1"
 		)
@@
 			)
 		)
+		(property "Sim.Pins" "1=K 2=A"
+			(at 43.18 226.06 0)
+			(effects
+				(font
+					(size 1.27 1.27)
+				)
+				(hide yes)
+			)
+		)
 		(pin "1"
 		)
@@
 			)
 		)
+		(property "Sim.Pins" "1=K 2=A"
+			(at 22.86 201.93 0)
+			(effects
+				(font
+					(size 1.27 1.27)
+				)
+				(hide yes)
+			)
+		)
 		(pin "1"
 		)
@@
 			)
 		)
+		(property "Sim.Pins" "1=K 2=A"
+			(at 22.86 226.06 0)
+			(effects
+				(font
+					(size 1.27 1.27)
+				)
+				(hide yes)
+			)
+		)
 		(pin "1"
 		)
@@
 			(at 33.02 201.93 0)
 			(effects
+				(font
+					(size 1.27 1.27)
+				)
+				(hide yes)
+			)
+		)
+		(property "Sim.Pins" "1=K 2=A"
+			(at 33.02 201.93 0)
+			(effects

Commit message: [INV_Boost_Controller] V1.1 again
minor update for jlc
Parts:
- Y1: value 48MHz YF4048M00033T8188103 -> X322516MLB4SI (16MHz)
Changed lines of the file:
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@@
 			)
 		)
-		(property "Value" "48MHz YF4048M00033T8188103"
+		(property "Value" "X322516MLB4SI (16MHz)"
 			(at 146.05 81.28 90)
 			(effects
