File: Powertrain_Group/INV_Boost_Controller/pwr.kicad_sch (KiCad schematic)
At the start: 46 parts, among them J6 LVBattery, J7 LVBattery, U7 TPS5430DDAR, U8 AMS1117-3.3, U9 REF2033

Commit message: [INV_Boost_Controller] V1.1
Parts:
- D1, D4: symbol PCM_Diode_Schottky_AKL:SS54 -> Device:D_Schottky_Small_Filled
- FL1: footprint Samacsys:ACM70V7012PLTL00 -> nturt_kicad_lib_EP7:Common_Mode_Choke_4A_ACM70V7012PLTL00; symbol SamacSys_Parts_EP6:ACM70V-701-2PL-TL00 -> nturt_kicad_lib_EP7:ACM70V-701-2PL-TL00
- L1: footprint PCM_Inductor_SMD_AKL:L_Wuerth_MAPI-3015 -> Inductor_SMD:L_Wuerth_MAPI-3015
- U7: symbol nturt_kicad_lib_EP6:TPS5430DDAR -> nturt_kicad_lib_EP7:TPS5430DDAR
Other:
- company: (none) -> NTURacing
- title: (none) -> INV_Boost_Controller
- moved on the sheet: D1, D4
Changed lines of the file:
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@@
 	(generator_version "9.0")
 	(paper "A4")
+	(title_block
+		(title "INV_Boost_Controller")
+		(date "2026-03-09")
+		(rev "1.1")
+		(company "NTURacing")
+		(comment 1 "Shinkansen942")
+		(comment 2 "Jack Kuo")
+	)
 	(rectangle
 		(start 201.93 19.05)
@@
 	(wire
 		(pts
-			(xy 229.87 30.48) (xy 236.22 30.48)
-		)
-		(stroke
-			(width 0)
-			(type default)
-		)
-	)
-	(wire
-		(pts
 			(xy 161.29 99.06) (xy 161.29 97.79)
 		)
@@
 	(wire
 		(pts
+			(xy 123.19 87.63) (xy 123.19 90.17)
+		)
+		(stroke
+			(width 0)
+			(type default)
+		)
+	)
+	(wire
+		(pts
 			(xy 177.8 44.45) (xy 177.8 43.18)
 		)
@@
 	(wire
 		(pts
-			(xy 123.19 81.28) (xy 123.19 80.01)
+			(xy 123.19 82.55) (xy 123.19 80.01)
 		)
 		(stroke
@@
 	(wire
 		(pts
-			(xy 107.95 44.45) (xy 119.38 44.45)
+			(xy 228.6 30.48) (xy 236.22 30.48)
 		)
 		(stroke
@@
 	(wire
 		(pts
-			(xy 261.62 30.48) (xy 261.62 34.29)
+			(xy 107.95 44.45) (xy 119.38 44.45)
 		)
 		(stroke
@@
 	(wire
 		(pts
-			(xy 87.63 36.83) (xy 87.63 46.99)
+			(xy 261.62 30.48) (xy 261.62 34.29)
 		)
 		(stroke
@@
 	(wire
 		(pts
-			(xy 187.96 130.81) (xy 196.85 130.81)
+			(xy 87.63 36.83) (xy 87.63 46.99)
 		)
 		(stroke
@@
 	(wire
 		(pts
-			(xy 123.19 90.17) (xy 123.19 88.9)
+			(xy 187.96 130.81) (xy 196.85 130.81)
 		)
 		(stroke
@@
 	(wire
 		(pts
-			(xy 220.98 30.48) (xy 222.25 30.48)
+			(xy 220.98 30.48) (xy 223.52 30.48)
 		)
 		(stroke
@@
 	)
 	(symbol
-		(lib_id "PCM_Diode_Schottky_AKL:SS54")
-		(at 123.19 85.09 90)
+		(lib_id "Device:D_Schottky_Small_Filled")
+		(at 123.19 85.09 270)
 		(unit 1)
 		(exclude_from_sim no)
@@
 		(fields_autoplaced yes)
 		(property "Reference" "D4"
-			(at 125.73 83.5024 90)
+			(at 125.73 83.5659 90)
 			(effects
 				(font
 					(size 1.27 1.27)
 				)
-				(justify right)
+				(justify left)
 			)
 		)
 		(property "Value" "SS54"
-			(at 125.73 86.0424 90)
+			(at 125.73 86.1059 90)
 			(effects
 				(font
 					(size 1.27 1.27)
 				)
-				(justify right)
+				(justify left)
 			)
 		)
 		(property "Footprint" "Diode_SMD:D_SMA"
-			(at 123.19 85.09 0)
+			(at 123.19 85.09 90)
 			(effects
 				(font
@@
 			)
 		)
-		(property "Datasheet" "https://www.laro.com.pl/pdf/ss56.pdf"
-			(at 123.19 85.09 0)
+		(property "Datasheet" "~"
+			(at 123.19 85.09 90)
 			(effects
 				(font
@@
 			)
 		)
-		(property "Description" "SMC Schottky diode, 40V, 5A, Alternate KiCAD Library"
+		(property "Description" "Schottky diode, small symbol, filled shape"
 			(at 123.19 85.09 0)
 			(effects
@@
 	)
 	(symbol
-		(lib_id "nturt_kicad_lib_EP6:TPS5430DDAR")
+		(lib_id "nturt_kicad_lib_EP7:TPS5430DDAR")
 		(at 85.09 85.09 0)
 		(unit 1)
@@
 			)
 		)
+		(property "Sim.Pins" "1=K 2=A"
+			(at 201.93 88.9 0)
+			(effects
+				(font
+					(size 1.27 1.27)
+				)
+				(hide yes)
+			)
+		)
 		(pin "1"
 		)
@@
 	)
 	(symbol
-		(lib_id "SamacSys_Parts_EP6:ACM70V-701-2PL-TL00")
+		(lib_id "nturt_kicad_lib_EP7:ACM70V-701-2PL-TL00")
 		(at 63.5 46.99 0)
 		(unit 1)
@@
 			)
 		)
-		(property "Footprint" "Samacsys:ACM70V7012PLTL00"
+		(property "Footprint" "nturt_kicad_lib_EP7:Common_Mode_Choke_4A_ACM70V7012PLTL00"
 			(at 80.01 141.91 0)
 			(effects
@@
 			)
 		)
+		(property "Sim.Pins" "1=K 2=A"
+			(at 229.87 133.35 0)
+			(effects
+				(font
+					(size 1.27 1.27)
+				)
+				(hide yes)
+			)
+		)
 		(pin "1"
 		)
@@
 			)
 		)
-		(property "Footprint" "PCM_Inductor_SMD_AKL:L_Wuerth_MAPI-3015"
+		(property "Footprint" "Inductor_SMD:L_Wuerth_MAPI-3015"
 			(at 129.54 36.83 0)
 			(effects
@@
 	)
 	(symbol
-		(lib_id "PCM_Diode_Schottky_AKL:SS54")
-		(at 226.06 30.48 0)
+		(lib_id "Device:D_Schottky_Small_Filled")
+		(at 226.06 30.48 180)
 		(unit 1)
 		(exclude_from_sim no)
@@
 		(fields_autoplaced yes)
 		(property "Reference" "D1"
-			(at 226.3775 24.13 0)
+			(at 226.314 24.13 0)
 			(effects
 				(font
@@
 		)
 		(property "Value" "SS54"
-			(at 226.3775 26.67 0)
+			(at 226.314 26.67 0)
 			(effects
 				(font
@@
 		)
 		(property "Footprint" "Diode_SMD:D_SMA"
-			(at 226.06 30.48 0)
+			(at 226.06 30.48 90)
 			(effects
 				(font
@@
 			)
 		)
-		(property "Datasheet" "https://www.laro.com.pl/pdf/ss56.pdf"
-			(at 226.06 30.48 0)
+		(property "Datasheet" "~"
+			(at 226.06 30.48 90)
 			(effects
 				(font
@@
 			)
 		)
-		(property "Description" "SMC Schottky diode, 40V, 5A, Alternate KiCAD Library"
+		(property "Description" "Schottky diode, small symbol, filled shape"
 			(at 226.06 30.48 0)
 			(effects
@@
 			(at 261.62 38.1 0)
 			(effects
+				(font
+					(size 1.27 1.27)
+				)
+				(hide yes)
+			)
+		)
+		(property "Sim.Pins" "1=K 2=A"
+			(at 261.62 38.1 0)
+			(effects

Commit message: [INV_Boost_Controller] V1.1 again
minor update for jlc
Parts:
- D6: value RED 5V -> WHITE 5V
- D7: value RED 3V3 -> WHITE 3V3
- R20: value 47k 1% -> 47k
- R21: value 15k 1% -> 15k
Changed lines of the file:
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@@
 			)
 		)
-		(property "Value" "47k 1%"
+		(property "Value" "47k"
 			(at 111.76 88.9 0)
 			(effects
@@
 			)
 		)
-		(property "Value" "RED 5V"
+		(property "Value" "WHITE 5V"
 			(at 205.74 91.7574 90)
 			(effects
@@
 		(fields_autoplaced yes)
 		(property "Reference" "D7"
-			(at 233.68 133.6675 90)
+			(at 233.68 133.6674 90)
 			(effects
 				(font
@@
 			)
 		)
-		(property "Value" "RED 3V3"
-			(at 233.68 136.2075 90)
+		(property "Value" "WHITE 3V3"
+			(at 233.68 136.2074 90)
 			(effects
 				(font
@@
 			)
 		)
-		(property "Value" "15k 1%"
+		(property "Value" "15k"
 			(at 111.76 99.06 0)
 			(effects
