File: Powertrain_Group/INV_Boost_Iso/PBI.kicad_sch (KiCad schematic)
At the start: 11 parts, among them J2 Conn_01x08, U1 ISO7720FDWV, U2 TEC2-2411WI, U3 TEL12-2415, U4 AMC1350DWV

Commit message: [INV_Bost_Isense] V1.1
Parts:
- C3: footprint Personal:C_8060_Murata_DK1 -> nturt_kicad_lib_EP7:C_8060_Murata_DK1
- U2: footprint Personal:Converter_DCDC_Meanwell_xPx0xW8-xx_THT -> nturt_kicad_lib_EP7:Converter_DCDC_Meanwell_xPx0xW8-xx_THT
- U3: footprint Converter_DCDC:Converter_DCDC_TRACO_TEL12-xxxx_THT -> nturt_kicad_lib_EP7:Converter_DCDC_TRACO_TEL12-xxxx_THT
Other:
- company: (none) -> NTURacing
- title: (none) -> INV_Boost_Iso
Changed lines of the file:
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@@
 	(generator_version "9.0")
 	(paper "A4")
+	(title_block
+		(title "INV_Boost_Iso")
+		(date "2026-03-06")
+		(rev "1.1")
+		(company "NTURacing")
+		(comment 1 "Shinkansen942")
+		(comment 2 "Jack Kuo")
+	)
 	(junction
 		(at 111.76 58.42)
@@
 		)
 	)
-	(wire
-		(pts
-			(xy 45.4099 57.15) (xy 45.72 57.15)
-		)
-		(stroke
-			(width 0)
-			(type default)
-		)
-	)
 	(label "ISO_GND"
 		(at 83.82 63.5 180)
@@
 	)
 	(label "ISO_24V"
-		(at 45.4099 57.15 0)
+		(at 45.72 57.15 0)
 		(effects
 			(font
@@
 			)
 		)
-		(property "Footprint" "Personal:Converter_DCDC_Meanwell_xPx0xW8-xx_THT"
+		(property "Footprint" "nturt_kicad_lib_EP7:Converter_DCDC_Meanwell_xPx0xW8-xx_THT"
 			(at 93.98 67.564 0)
 			(effects
@@
 			)
 		)
-		(property "Footprint" "Converter_DCDC:Converter_DCDC_TRACO_TEL12-xxxx_THT"
+		(property "Footprint" "nturt_kicad_lib_EP7:Converter_DCDC_TRACO_TEL12-xxxx_THT"
 			(at 93.98 90.805 0)
 			(effects
@@
 			)
 		)
-		(property "Footprint" "Personal:C_8060_Murata_DK1"
+		(property "Footprint" "nturt_kicad_lib_EP7:C_8060_Murata_DK1"
 			(at 97.79 44.7548 0)
 			(effects

Commit message: [INV_Boost_Iso] V1.2
swap 0402 with 0603
Parts:
- C1, C2, C4, C5: footprint Capacitor_SMD:C_0402_1005Metric -> Capacitor_SMD:C_0603_1608Metric
Changed lines of the file:
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@@
 	(title_block
 		(title "INV_Boost_Iso")
-		(date "2026-03-06")
-		(rev "1.1")
+		(date "2026-03-09")
+		(rev "1.2")
 		(company "NTURacing")
 		(comment 1 "Shinkansen942")
@@
 			)
 		)
-		(property "Footprint" "Capacitor_SMD:C_0402_1005Metric"
+		(property "Footprint" "Capacitor_SMD:C_0603_1608Metric"
 			(at 112.7252 33.02 0)
 			(effects
@@
 			)
 		)
-		(property "Footprint" "Capacitor_SMD:C_0402_1005Metric"
+		(property "Footprint" "Capacitor_SMD:C_0603_1608Metric"
 			(at 147.32 95.25 0)
 			(effects
@@
 			)
 		)
-		(property "Footprint" "Capacitor_SMD:C_0402_1005Metric"
+		(property "Footprint" "Capacitor_SMD:C_0603_1608Metric"
 			(at 82.2452 124.46 0)
 			(effects
@@
 			)
 		)
-		(property "Footprint" "Capacitor_SMD:C_0402_1005Metric"
+		(property "Footprint" "Capacitor_SMD:C_0603_1608Metric"
 			(at 68.2752 33.02 0)
 			(effects
