File: Powertrain_Group/INV_Discrete_Power/gate_drive.kicad_sch (KiCad schematic)
At the start: 23 parts, among them U3 1ED3122MC12HXUMA1, U4 1ED3122MC12HXUMA1

Commit message: [INV_Discrete_Power] V1.1 by Jack Kuo
Parts:
- C501: renamed from C6; symbol Device:C -> Device:C_Small
- C504: renamed from C7; symbol Device:C -> Device:C_Small
- renumbered C8 to C502, C9 to C503, C10 to C505, C11 to C506, D8 to D501, D3 to D502, D1 to D503, D2 to D504, R66 to R501, R1 to R502, R5 to R503, R2 to R504, R6 to R505, R9 to R506, R3 to R507, R7 to R508, R4 to R509, R8 to R510, R10 to R511, U3 to U501, U4 to U502
Connections:
- net +5VA renamed +5V_in
- net GND1 renamed GND_in
Other:
- company: (none) -> NTURacing
- title: (none) -> INV_Discrete_Power
- moved on the sheet: C504, D502

Commit message: [INV_Discrete_Power] V1.2
Parts:
- R501: value 1k -> 10k
- R503, R505, R508, R510: value 1 -> 1R
- U501, U502: symbol Snapeda:1ED3122MC12HXUMA1 -> nturt_kicad_lib_EP7:1ED3122MC12HXUMA1
Other:
- moved on the sheet: R505
Changed lines of the file:
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@@
 		(title "INV_Discrete_Power")
 		(date "2026-03-13")
-		(rev "1.1")
+		(rev "1.2")
 		(company "NTURacing")
 		(comment 1 "LY Chen")
@@
 	)
 	(junction
+		(at 162.56 67.31)
+		(diameter 0)
+		(color 0 0 0 0)
+	)
+	(junction
 		(at 168.91 90.17)
 		(diameter 0)
@@
 	)
 	(junction
-		(at 162.56 66.04)
-		(diameter 0)
-		(color 0 0 0 0)
-	)
-	(junction
 		(at 59.69 58.42)
 		(diameter 0)
@@
 	(wire
 		(pts
-			(xy 162.56 66.04) (xy 162.56 68.58)
-		)
-		(stroke
-			(width 0)
-			(type default)
-		)
-	)
-	(wire
-		(pts
 			(xy 144.78 82.55) (xy 177.8 82.55)
 		)
@@
 	(wire
 		(pts
-			(xy 158.75 66.04) (xy 162.56 66.04)
-		)
-		(stroke
-			(width 0)
-			(type default)
-		)
-	)
-	(wire
-		(pts
-			(xy 148.59 68.58) (xy 148.59 60.96)
+			(xy 158.75 67.31) (xy 162.56 67.31)
+		)
+		(stroke
+			(width 0)
+			(type default)
+		)
+	)
+	(wire
+		(pts
+			(xy 148.59 69.85) (xy 148.59 60.96)
 		)
 		(stroke
@@
 	(wire
 		(pts
-			(xy 162.56 66.04) (xy 162.56 63.5)
-		)
-		(stroke
-			(width 0)
-			(type default)
-		)
-	)
-	(wire
-		(pts
 			(xy 91.44 31.75) (xy 31.75 31.75)
 		)
@@
 	(wire
 		(pts
+			(xy 162.56 63.5) (xy 162.56 67.31)
+		)
+		(stroke
+			(width 0)
+			(type default)
+		)
+	)
+	(wire
+		(pts
 			(xy 95.25 66.04) (xy 105.41 66.04)
 		)
@@
 	(wire
 		(pts
+			(xy 162.56 67.31) (xy 162.56 69.85)
+		)
+		(stroke
+			(width 0)
+			(type default)
+		)
+	)
+	(wire
+		(pts
 			(xy 58.42 58.42) (xy 59.69 58.42)
 		)
@@
 	(wire
 		(pts
-			(xy 162.56 68.58) (xy 148.59 68.58)
+			(xy 162.56 69.85) (xy 148.59 69.85)
 		)
 		(stroke
@@
 	(wire
 		(pts
-			(xy 151.13 58.42) (xy 151.13 66.04)
+			(xy 151.13 58.42) (xy 151.13 67.31)
 		)
 		(stroke
@@
 	)
 	(symbol
-		(lib_id "Snapeda:1ED3122MC12HXUMA1")
+		(lib_id "nturt_kicad_lib_EP7:1ED3122MC12HXUMA1")
 		(at 128.27 86.36 0)
 		(unit 1)
@@
 	(symbol
 		(lib_id "Device:R")
-		(at 154.94 66.04 90)
+		(at 154.94 67.31 90)
 		(unit 1)
 		(exclude_from_sim no)
@@
 		(fields_autoplaced yes)
 		(property "Reference" "R505"
-			(at 154.94 69.85 90)
-			(effects
-				(font
-					(size 1.27 1.27)
-				)
-			)
-		)
-		(property "Value" "1"
-			(at 154.94 72.39 90)
+			(at 154.94 60.96 90)
+			(effects
+				(font
+					(size 1.27 1.27)
+				)
+			)
+		)
+		(property "Value" "1R"
+			(at 154.94 63.5 90)
 			(effects
 				(font
@@
 		)
 		(property "Footprint" "Resistor_SMD:R_1206_3216Metric"
-			(at 154.94 67.818 90)
+			(at 154.94 69.088 90)
 			(effects
 				(font
@@
 		)
 		(property "Datasheet" "~"
-			(at 154.94 66.04 0)
+			(at 154.94 67.31 0)
 			(effects
 				(font
@@
 		)
 		(property "Description" "Resistor"
-			(at 154.94 66.04 0)
+			(at 154.94 67.31 0)
 			(effects
 				(font
@@
 			)
 		)
-		(property "Value" "1k"
+		(property "Value" "10k"
 			(at 34.29 48.2599 0)
 			(effects
@@
 	)
 	(symbol
-		(lib_id "Snapeda:1ED3122MC12HXUMA1")
+		(lib_id "nturt_kicad_lib_EP7:1ED3122MC12HXUMA1")
 		(at 128.27 59.69 0)
 		(unit 1)
@@
 			)
 		)
+		(property "Sim.Pins" "1=K 2=A"
+			(at 31.75 36.83 0)
+			(effects
+				(font
+					(size 1.27 1.27)
+				)
+				(hide yes)
+			)
+		)
 		(pin "1"
 		)
@@
 			)
 		)
-		(property "Value" "1"
+		(property "Value" "1R"
 			(at 154.94 80.01 90)
 			(effects
@@
 			)
 		)
-		(property "Value" "1"
+		(property "Value" "1R"
 			(at 154.94 54.61 90)
 			(effects
@@
 			)
 		)
-		(property "Value" "1"
+		(property "Value" "1R"
 			(at 154.94 90.17 90)
 			(effects
