File: Powertrain_Group/INV_Discrete_Power/phase.kicad_sch (KiCad schematic)
At the start: 13 parts, among them J201 ISO_PWR_H, J202 PHASE_OUT, J203 PWM, J204 I_sig, J205 ISO_PWR_L, Q201 ADR014B12MC, Q202 ADR014B12MC

Commit message: [INV_Discrete_Power] V1.2
Parts:
- C202: footprint SamacSys_Parts_EP6:B58035U5106M001 -> nturt_kicad_lib_EP7:TDK_Ceralink_FA10
- Q201, Q202: footprint Package_TO_SOT_THT:TO-247-4_Vertical -> nturt_kicad_lib_EP7:TO-247-4_Horizontal_TabUp_NoHole
Other:
- moved on the sheet: J201, J203, J204, J205
