File: Electrical_Group/PCAN_PRO/PCAN_PRO.kicad_pcb (KiCad board)
At the start: 2 copper layers, 80 x 23 mm, 92 parts, among them IC1 UCC33420QRAQRQ1, IC2 UCC33420QRAQRQ1, J1 STDC14, J2 CAN, J3 CAN, J4 CAN, J5 CAN, J6 USB_C_stm32, SW1 SW_DIP_x01, SW2 SW_DIP_x01, SW3 RESET, SW4 BOOT0, U1 ISO7721DWV, U2 ISO7721DWV, U3 TCAN1042VDRQ1, U4 TCAN1042VDRQ1, U5 STM32F405RGTx, U7 SRV05-4, U8 AMS1117-3.3, Y1 8MHz X50328MSB2GI

Commit message: [PCAN_PRO] V1.1
Parts:
- removed FB1: GZ2012D601TF, Inductor_SMD:L_0805_2012Metric
- added R28: 0R, Resistor_SMD:R_0402_1005Metric, F.Cu at (158.4, 109.4)
- added R29: 0R, Resistor_SMD:R_0402_1005Metric, F.Cu at (158.2, 115.9)
- FL1, FL2: footprint Samacsys:EXCX4CE900U -> nturt_kicad_lib_EP7:EXCX4CE900U
- IC1, IC2: footprint Samacsys:UCC33020QRAQRQ1 -> nturt_kicad_lib_EP7:UCC33020
- J1: footprint Personal:box_header_14P_pitch127 -> nturt_kicad_lib_EP7:box_header_14P_pitch1.27
- moved R18 2.96 mm to (133.8, 102.8)
- moved R16 2.93 mm to (133.8, 101.8)
- moved D4 2.08 mm to (136.3, 101.6)
- moved D6 2.08 mm to (136.3, 103.1)
- moved D10 1.35 mm to (110.7, 119.6)
- moved D3 1.35 mm to (110.7, 118.1)
- moved R12 1.35 mm to (106.9, 119.5), turned to 0 degrees
- moved R27 1.21 mm to (108.6, 119.4), turned to 90 degrees
- moved R15 0.84 mm to (108.6, 117.5), turned to 90 degrees
- moved F1 0.56 mm to (109.9, 115.3)
- moved R6 0.11 mm to (158.3, 105.6)
- moved FL1 0.10 mm to (158.4, 107.5)
- moved FL2 0.10 mm to (158.4, 114.0)
Connections:
- net /CAN1N renamed /CAN1L
- net /CAN1P renamed /CAN1H
- net /CAN2N renamed /CAN2L
- net /CAN2P renamed /CAN2H
- C28 pad 1: /3V3_REF -> +3V3
- C29 pad 1: /3V3_REF -> +3V3
- D4 pad 1: Net-(D4-K) -> GND
- D4 pad 2: /PA4 -> Net-(D4-A)
- D6 pad 1: Net-(D6-K) -> GND
- D6 pad 2: /PA5 -> Net-(D6-A)
- R16 pad 1: Net-(D4-K) -> /PA4
- R16 pad 2: GND -> Net-(D4-A)
- R18 pad 1: Net-(D6-K) -> /PA5
- R18 pad 2: GND -> Net-(D6-A)
- U3 pad 5: +5V_ISO1 -> Net-(U3-VIO)
- U4 pad 5: +5V_ISO2 -> Net-(U4-VIO)
- U5 pad 13: /3V3_REF -> +3V3
Routing:
- net GND2: track 19.8 -> 9.55 mm, vias 3 -> 6
- net GND1: track 19.8 -> 9.90 mm
- net GND: track 7.12 -> 16.7 mm, vias 138 -> 42
- net /CAN2H: track 30.3 -> 23.5 mm, vias 0 -> 2
- net +3V3: track 124.8 -> 130.4 mm
- net /3V3_REF: track 4.98 -> 0.00 mm
- net +5V: track 68.4 -> 73.1 mm
- net /CAN2L: track 38.5 -> 34.0 mm
- net /VBUS: track 16.3 -> 20.4 mm, vias 3 -> 2
- net +5V_ISO1: track 15.3 -> 19.0 mm
- net +5V_ISO2: track 15.3 -> 18.7 mm
- net /BOOT0: track 35.1 -> 33.2 mm
- net Net-(U3-VIO): track 0.00 -> 1.91 mm
- net Net-(U4-VIO): track 0.00 -> 1.72 mm
- net /SWD_NRST: track 50.4 -> 51.9 mm
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- added copper zone on B.Cu, net GND1
- added copper zone on B.Cu, net GND2
Other:
- board text added: "EP7 PCAN_PRO V1.1 26/03/04 Shinkansen942 Jack Kuo"
- board text added: "FUSE"
- board text added: "TX RX"
- board text removed: "CAN2 TX RX"

Commit message: [PCAN_PRO] V1.1 again
minor update for jlc
Parts:
- C17, C19: value 2.2u 10V -> 2u2
- R10, R11: value 120R -> 122R
- R13, R14, R2, R3, R4, R5: value 20R -> 22R
Other:
- outline, holes or cut-outs redrawn
- board text added: "EP7 PCAN_PRO V1.1 26/03/16 Shinkansen942 Jack Kuo"
- board text removed: "EP7 PCAN_PRO V1.1 26/03/04 Shinkansen942 Jack Kuo"
Changed lines of the file:
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@@
 	(title_block
 		(title "PCAN_PRO")
-		(date "2026-03-04")
+		(date "2026-03-16")
 		(rev "1.1")
 		(company "NTURacing")
@@
 			)
 		)
-		(property "Value" "2.2u 10V"
+		(property "Value" "2u2"
 			(at 0 1.16 0)
 			(layer "F.Fab")
@@
 			)
 		)
-		(property "Value" "20R"
+		(property "Value" "22R"
 			(at 0 1.17 0)
 			(layer "F.Fab")
@@
 			)
 		)
-		(property "Value" "20R"
+		(property "Value" "22R"
 			(at 0 1.17 0)
 			(layer "F.Fab")
@@
 			)
 		)
-		(property "Value" "120R"
+		(property "Value" "122R"
 			(at 0 1.65 0)
 			(layer "F.Fab")
@@
 			)
 		)
-		(property "Value" "20R"
+		(property "Value" "22R"
 			(at 0 1.17 0)
 			(layer "F.Fab")
@@
 			)
 		)
-		(property "Value" "2.2u 10V"
+		(property "Value" "2u2"
 			(at 0 1.16 90)
 			(layer "F.Fab")
@@
 			)
 		)
-		(property "Value" "20R"
+		(property "Value" "22R"
 			(at 0 1.17 0)
 			(layer "F.Fab")
@@
 			)
 		)
-		(property "Value" "20R"
+		(property "Value" "22R"
 			(at 0 1.17 0)
 			(layer "F.Fab")
@@
 			)
 		)
-		(property "Value" "120R"
+		(property "Value" "122R"
 			(at 0 1.65 0)
 			(layer "F.Fab")
@@
 			)
 		)
-		(property "Value" "20R"
+		(property "Value" "22R"
 			(at 0 1.17 0)
 			(layer "F.Fab")
@@
 		(layer "B.SilkS")
 	)
-	(gr_rect
-		(start 97.475 99.25)
-		(end 177.475 122.25)
+	(gr_line
+		(start 97.475 118.25)
+		(end 97.475 103.25)
+		(stroke
+			(width 0.05)
+			(type default)
+		)
+		(layer "Edge.Cuts")
+	)
+	(gr_line
+		(start 101.475 99.25)
+		(end 173.475 99.25)
+		(stroke
+			(width 0.05)
+			(type default)
+		)
+		(layer "Edge.Cuts")
+	)
+	(gr_arc
+		(start 97.475 103.25)
+		(mid 98.646573 100.421573)
+		(end 101.475 99.25)
+		(stroke
+			(width 0.05)
+			(type default)
+		)
+		(layer "Edge.Cuts")
+	)
+	(gr_arc
+		(start 173.475 99.25)
+		(mid 176.303427 100.421573)
+		(end 177.475 103.25)
+		(stroke
+			(width 0.05)
+			(type default)
+		)
+		(layer "Edge.Cuts")
+	)
+	(gr_arc
+		(start 177.475 118.25)
+		(mid 176.303427 121.078427)
+		(end 173.475 122.25)
+		(stroke
+			(width 0.05)
+			(type default)
+		)
+		(layer "Edge.Cuts")
+	)
+	(gr_line
+		(start 173.475 122.25)
+		(end 101.475 122.25)
+		(stroke
+			(width 0.05)
+			(type default)
+		)
+		(layer "Edge.Cuts")
+	)
+	(gr_arc
+		(start 101.475 122.25)
+		(mid 98.646573 121.078427)
+		(end 97.475 118.25)
+		(stroke
+			(width 0.05)
+			(type default)
+		)
+		(layer "Edge.Cuts")
+	)
+	(gr_line
+		(start 177.475 103.25)
+		(end 177.475 118.25)
 		(stroke
 			(width 0.05)
 			(type default)
 		)
-		(fill no)
 		(layer "Edge.Cuts")
 	)
@@
 		)
 	)
-	(gr_text "EP7\nPCAN_PRO\nV1.1 26/03/04\nShinkansen942\nJack Kuo"
+	(gr_text "EP7\nPCAN_PRO\nV1.1 26/03/16\nShinkansen942\nJack Kuo"
 		(at 122.595853 111.659941 0)
 		(layer "B.SilkS")
