File: Electrical_Group/Tire_Temp/Tire_Temp.kicad_sch (KiCad schematic)
At the start: 13 parts, among them IC1 MLX90640ESF-BAA-000-SP

Commit message: [Tire_Temp] V1.0 again
minor update for jlc
Other:
- note added: "V1.0 init 3/16 change res for buck fb note: remember to add logo next time add meassure angle indication next time maybe can have more led in the future"
- note removed: "V1.0 init"
Changed lines of the file:
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@@
 		(comment 2 "Jack Kuo 郭哲明")
 	)
-	(text "V1.0 init"
+	(text "V1.0 init\n     3/16 change res for buck fb\n\n\nnote: remember to add logo next time\n      add meassure angle indication next time\n      maybe can have more led in the future"
 		(exclude_from_sim no)
 		(at 59.436 43.942 0)
