File: Electrical_Group/Tire_Temp/power.kicad_sch (KiCad schematic)
At the start: 19 parts, among them U1 XC6206P332MR-G, U4 LMR50410

Commit message: [Tire_Temp] V1.0 again
minor update for jlc
Parts:
- R3: value 9k1 -> 75k
- R4: value 2k2 -> 18k
Other:
- note added: "LMR50410 is 700k replace with LMR5140 for 1.1Mhz"
Changed lines of the file:
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@@
+		)
+	)
+	(text "LMR50410 is 700k\nreplace with LMR5140 for 1.1Mhz"
+		(exclude_from_sim no)
+		(at 68.834 69.088 0)
+		(effects
+			(font
+				(size 1.27 1.27)
+			)
 		)
 	)
@@
 			)
 		)
-		(property "Value" "2k2"
+		(property "Value" "18k"
 			(at 125.73 109.22 0)
 			(effects
@@
 			)
 		)
-		(property "Value" "9k1"
+		(property "Value" "75k"
 			(at 125.73 99.06 0)
 			(effects
