File: Powertrain_Group/INV_CONN1/INV_CONN1.kicad_pcb (KiCad board)
At the start: 2 copper layers, 59 x 23 mm, 11 parts, among them J1 24V, J10 24V, J2 CAN, J3 CAN0, J4 CAN1, J5 24V_CAN_4P, J6 24V_CAN_4P, J8 CAN

Commit message: [INV_CONN1] V1.1
Parts:
- JP2: moved to F.Cu
- moved JP2 4.38 mm to (129.5, 70.0)
- moved JP1 3.60 mm to (129.5, 70.0)
- turned J5 to 90 degrees
Routing:
- net GNDPWR: track 68.3 -> 0.00 mm
- net +24V: track 58.5 -> 0.00 mm
- net /CAN1_L: track 43.3 -> 31.0 mm
- net /CAN1_H: track 41.9 -> 31.3 mm
- net /CAN0_L: track 28.8 -> 31.9 mm
- net /CAN0_H: track 31.4 -> 33.8 mm, vias 1 -> 0
- added copper zone on F.Cu, net +24V
- added copper zone on B.Cu, net /SH
- added copper zone on B.Cu, net GNDPWR
Other:
- board text added: "24V"
- board text added: "4"
- board text added: "CAN"
- board text added: "H"
- board text added: "L"
- board text added: "SH"
- board text added: "V1.1 26/03/16 Jack Kuo"
- board text removed: "SH L H"
- board text removed: "V1.0 26/03/04 Jack Kuo"
