File: Powertrain_Group/INV_CONN1/INV_CONN1.kicad_sch (KiCad schematic)
At the start: 11 parts, among them J1 24V, J10 24V, J2 CAN, J3 CAN0, J4 CAN1, J5 24V_CAN_4P, J6 24V_CAN_4P, J8 CAN

Commit message: [INV_CONN1] V1.1
Other:
- note added: "V1.0 init V1.1 modify layout"
- note removed: "V1.0 init"
Changed lines of the file:
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@@
 	(title_block
 		(title "INV_CONN1")
-		(date "2026-03-04")
-		(rev "1.0")
+		(date "2026-03-16")
+		(rev "1.1")
 		(company "NTURacing")
 		(comment 1 "Jack Kuo")
@@
 		)
 	)
-	(text "V1.0 init"
+	(text "V1.0 init\nV1.1 modify layout"
 		(exclude_from_sim no)
 		(at 111.76 111.506 0)
