File: Powertrain_Group/INV_CONN2/INV_CONN2.kicad_pcb (KiCad board)
At the start: 2 copper layers, 52 x 20 mm, 7 parts, among them J1 encoder, J12 Encoder, J13 motorTemp, J3 Conn_02x05_Odd_Even_MountingP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

Commit message: [INV_CONN2] V1.1
Parts:
- removed J12: Encoder, Connector_JST:JST_PH_B6B-PH-K_1x06_P2.00mm_Vertical
- removed J13: motorTemp, Connector_JST:JST_PH_B4B-PH-K_1x04_P2.00mm_Vertical
- removed JP1, JP2: SolderJumper_2_Bridged, Jumper:SolderJumper-2_P1.3mm_Bridged_Pad1.0x1.5mm
- moved H1 39.0 mm to (164.0, 106.0)
- turned J1 to 0 degrees
Routing:
- net /shielding: track 72.5 -> 34.0 mm
- net GND: track 32.7 -> 7.46 mm, vias 1 -> 0
- net /cos-: track 23.9 -> 6.06 mm, vias 1 -> 0
- net /encoderPWR: track 31.6 -> 15.7 mm
- net /temp-: track 40.0 -> 27.1 mm, vias 1 -> 0
- net /tempPWR: track 10.9 -> 0.00 mm
- net /sin-: track 22.3 -> 14.5 mm, vias 1 -> 0
- net /cos+: track 23.2 -> 17.6 mm
- net /tempGND: track 4.32 -> 0.00 mm
- net /sin+: track 23.6 -> 27.2 mm
- net /temp+: track 39.8 -> 40.4 mm
Other:
- board size 52 x 20 mm -> 38 x 20 mm
- board text added: "EP7 INV_CONN2"
- board text added: "Jack Kuo V1.1 26/03/16"
- board text added: "c"
- board text added: "pwr"
- board text added: "sin"
- board text added: "temp"
- board text removed: "+5V"
- board text removed: "GND"
- board text removed: "GND PWR C- C+ S- S+"
- board text removed: "GND T- T+ +5V"
- board text removed: "NTUR EP7 INV_CONN2 Jack Kuo V1.0 26/03/04"
