File: Powertrain_Group/INV_CONN2/INV_CONN2.kicad_sch (KiCad schematic)
At the start: 7 parts, among them J1 encoder, J12 Encoder, J13 motorTemp, J3 Conn_02x05_Odd_Even_MountingP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

Commit message: [INV_CONN2] V1.1
Parts:
- removed J12: Encoder, Connector_JST:JST_PH_B6B-PH-K_1x06_P2.00mm_Vertical, symbol Connector_Generic:Conn_01x06
- removed J13: motorTemp, Connector_JST:JST_PH_B4B-PH-K_1x04_P2.00mm_Vertical, symbol Connector_Generic:Conn_01x04
- removed JP1, JP2: SolderJumper_2_Bridged, Jumper:SolderJumper-2_P1.3mm_Bridged_Pad1.0x1.5mm, symbol Jumper:SolderJumper_2_Bridged
Other:
- note added: "V1.0 init V1.1 remove 2.0 connector"
- note removed: "V1.0"
- moved on the sheet: J1
