File: Powertrain_Group/INV_Discrete_Controller/DifToSingle.kicad_sch (KiCad schematic)
At the start: 8 parts, among them U13 INA333AIDGK

Commit message: [INV_Discrete_Controller] V1.1
Parts:
- removed R70: ${Res2}, Resistor_SMD:R_0402_1005Metric, symbol Device:R_Small
- added C20: ${Cap}, Capacitor_SMD:C_0402_1005Metric, symbol Device:C_Small
- R71: value ${Res3} -> ${Res2}
- U13: footprint Package_SO:MSOP-8_3x3mm_P0.65mm -> Package_SO:VSSOP-8_3x3mm_P0.65mm; symbol PCM_Amplifier_Instrumentation_AKL:INA333AIDGK -> Amplifier_Instrumentation:INA333xxDGK
Connections:
- net at R68.2, U13.2 (-): now also C20.2
- net at R69.2, U13.3 (+): now also C20.1
Other:
- company: (none) -> NTURacing
- title: (none) -> INV_Discrete_Controller
- moved on the sheet: C81, R68, R69

Commit message: [INV_Discrete_Controller] V1.2
Other:
- note added: "R1 : ${Res1} R2 : ${Res2} gain = 1+100k/${Res2} = 1.2325"
- note added: "Vout = (1+100k/${Res2}))* Vin = 1.1"
- note removed: "R1 : ${Res1} R2 : ${Res2} R3 : ${Res3} gain = 1+100k/${Res3} = 1.2325"
- note removed: "Vout = (2R2/(2R1 + R2))* Vin"
Changed lines of the file:
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@@
 	(title_block
 		(title "INV_Discrete_Controller")
-		(date "2026-03-15")
-		(rev "1.1")
+		(date "2026-03-17")
+		(rev "1.2")
 		(company "NTURacing")
 		(comment 1 "LY Chen")
 		(comment 2 "Jack Kuo")
 	)
-	(text "Vout = (2R2/(2R1 + R2))* Vin"
+	(text "Vout = (1+100k/${Res2}))* Vin = 1.1"
 		(exclude_from_sim no)
-		(at 87.63 59.69 0)
+		(at 114.554 66.802 0)
 		(effects
 			(font
@@
 		)
 	)
-	(text "R1 : ${Res1} \nR2 : ${Res2}\nR3 : ${Res3}\ngain = 1+100k/${Res3} = 1.2325"
+	(text "R1 : ${Res1} \nR2 : ${Res2}\ngain = 1+100k/${Res2} = 1.2325"
 		(exclude_from_sim no)
 		(at 157.988 85.852 0)
