File: Powertrain_Group/INV_Discrete_Controller/DifToSingle2.kicad_sch (KiCad schematic)
At the start: 8 parts, among them U12 INA333AIDGK

Commit message: [INV_Discrete_Controller] V1.1
Parts:
- U12: footprint Package_SO:MSOP-8_3x3mm_P0.65mm -> Package_SO:VSSOP-8_3x3mm_P0.65mm; symbol PCM_Amplifier_Instrumentation_AKL:INA333AIDGK -> Amplifier_Instrumentation:INA333xxDGK
Other:
- company: (none) -> NTURacing
- title: (none) -> INV_Discrete_Controller
- moved on the sheet: C79, R65, R66
