File: Powertrain_Group/INV_Discrete_Controller/Isense_OCP.kicad_sch (KiCad schematic)
At the start: 35 parts, among them J13 motorTemp, J14 current_DC, J15 Conn_01x02, J16 Conn_01x02, J17 Conn_01x02, U11 LM393

Commit message: [INV_Discrete_Controller] V1.1
Parts:
- removed J13: motorTemp, Connector_JST:JST_XH_B4B-XH-A_1x04_P2.50mm_Vertical, symbol Connector_Generic:Conn_01x04
- added J601: current_DC, Connector_JST:JST_PH_B4B-PH-K_1x04_P2.00mm_Vertical, symbol Connector_Generic:Conn_01x04
- J14: symbol PCM_4ms_Connector:Conn_01x04 -> Connector_Generic:Conn_01x04
- R63, R64: symbol Device:R -> Device:R_Small
- RV1, RV2: footprint nturt_kicad_lib_EP6:Throughhole Potentiometer 3296W -> nturt_kicad_lib_EP7:Potentiometer_Bourns_3296W_Horizontal
- TP14: value I_DC+ -> threshold
- TP15: value I_DC- -> threshold
Connections:
- net +5V: now also J601.4 (Pin_4)
- net GND: now also J601.1 (Pin_1)
- net DCVsenseNode/IN+: now also J601.3 (Pin_3); no longer TP14.1
- net DCVsenseNode/IN-: now also J601.2 (Pin_2); no longer TP15.1
- net OT_ref: now also TP15.1
- net at RV1.2, U11.5 (+): now also TP14.1
- net MotTempNode/IN+ renamed mot_T+
- net MotTempNode/IN- renamed mot_T-
Other:
- sheet IsenseNode renamed DCVsenseNode
- note added: "should be updated OCP res should be recalculated"
- note removed: "NOTE: differential pin reversed"
- company: (none) -> NTURacing
- title: (none) -> INV_Discrete_Controller

Commit message: [INV_Discrete_Controller] V1.2
Parts:
- added R601, R602, R603, R604, R605: 0R, Resistor_SMD:R_0402_1005Metric, symbol Device:R_Small
Connections:
- net OC&OT_Falut: now also R601.2, R602.1, R603.1, R604.1, R605.2; no longer U11.1, U11.7
- new net: R605.1, U11.1, U11.7
- new net OCPnode1/GateEnablePull: R601.1
- new net OTPnode/GateEnablePull: R602.2
- new net OTPnode1/GateEnablePull: R603.2
- new net OTPnode2/GateEnablePull: R604.2
Other:
- note added: "per phase current sensor: LEM CKSR 75-NP 6.25 mV/A 5V supply Vout: Vref +- 1.125 V Vref: 2.495 ~ 2.505 V diff gain = 2*1.1 = 2.2 => 13.75 mV/A OCP voltage set : 100A => 1.65+-1.375 = 3.025, 0.275 OCP voltage actual: 3.109, 0.191 gain 2 at Isense board gain 1.1 at controller board"
- note removed: "per phase current sensor: LEM LZSR 80-P 7.813 mV/A 5V supply Vout: 0.25 ~ 4.75 V Vref: 2.485 ~ 2.515 V diff gain = 1 => 15.626 mV/A OCP voltage set : 100A => 1.65+-0.7813 = 2.431,0.868 OCP voltage actual: 2.431, 0.868"
- note removed: "should be updated OCP res should be recalculated"
