File: Powertrain_Group/INV_Discrete_Controller/MCU.kicad_sch (KiCad schematic)
At the start: 74 parts, among them J11 MSD-4-A, J12 STDC14, SW1 TS-1187A-B-A-B, SW2 TS-1187A-B-A-B, SW4 TS-1187A-B-A-B, U10 STM32H743ZITx, U9 REF2033, Y1 X322516MLB4SI (16MHz), Y2 32.768kHz Q13FC13500004

Commit message: [INV_Discrete_Controller] V1.1
Parts:
- BT1: footprint nturt_kicad_lib_EP6:BAT_1056 -> nturt_kicad_lib_EP7:BAT_1056; symbol nturt_kicad_lib_EP6:1056 -> nturt_kicad_lib_EP7:BAT_1056
- C38, C39, C40, C60, C67: value 0u1 -> 100n
- J11: footprint SamacSys_Parts_EP6:MSD4A -> nturt_kicad_lib_EP7:MSD4A; symbol SamacSys_Parts_EP6:MSD-4-A -> nturt_kicad_lib_EP7:MSD-4-A; Manufacturer_Name Same Sky -> CUI Devices; Mouser Price/Stock https://www.mouser.co.uk/ProductDetail/Same-Sky/MSD-4-A?qs=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 -> https://www.mouser.co.uk/ProductDetail/CUI-Devices/MSD-4-A?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
- J12: footprint nturt_kicad_lib_EP6:box_header_14P_pitch127 -> nturt_kicad_lib_EP7:box_header_14P_pitch1.27
- R37, R47, R49, R50, R51, R52, R53: symbol Device:R -> Device:R_Small
Connections:
- net Vref_1.65 renamed Vref_1.65V
- no-connect marks 66 -> 67
Other:
- company: (none) -> NTURacing
- title: (none) -> INV_Discrete_Controller
- moved on the sheet: C38, C39, C67, C68, C69, C70, C71, FB1, R37, R38, R47, SW1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
