File: Powertrain_Group/INV_Discrete_Controller/OCPnode.kicad_sch (KiCad schematic)
At the start: 7 parts, among them U17 LM393

Commit message: [INV_Discrete_Controller] V1.1
Parts:
- R81, R82, R83, R84: symbol Device:R -> Device:R_Small
Other:
- company: (none) -> NTURacing
- title: (none) -> INV_Discrete_Controller
Changed lines of the file:
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@@
 	(generator_version "9.0")
 	(paper "A4")
+	(title_block
+		(title "INV_Discrete_Controller")
+		(date "2026-03-15")
+		(rev "1.1")
+		(company "NTURacing")
+		(comment 1 "LY Chen")
+		(comment 2 "Jack Kuo")
+	)
 	(text "1 if V < 2.66\n0 if V > 2.66"
 		(exclude_from_sim no)
@@
 	(wire
 		(pts
+			(xy 105.41 127) (xy 105.41 129.54)
+		)
+		(stroke
+			(width 0)
+			(type default)
+		)
+	)
+	(wire
+		(pts
 			(xy 133.35 45.72) (xy 125.73 45.72)
 		)
@@
 	(wire
 		(pts
-			(xy 105.41 120.65) (xy 105.41 111.76)
+			(xy 106.68 77.47) (xy 106.68 78.74)
 		)
 		(stroke
@@
 	(wire
 		(pts
-			(xy 105.41 128.27) (xy 105.41 129.54)
-		)
-		(stroke
-			(width 0)
-			(type default)
-		)
-	)
-	(wire
-		(pts
 			(xy 119.38 74.93) (xy 113.03 74.93)
 		)
@@
 	(wire
 		(pts
+			(xy 105.41 111.76) (xy 105.41 121.92)
+		)
+		(stroke
+			(width 0)
+			(type default)
+		)
+	)
+	(wire
+		(pts
 			(xy 113.03 100.33) (xy 113.03 124.46)
 		)
@@
 	(wire
 		(pts
-			(xy 106.68 58.42) (xy 106.68 60.96)
+			(xy 106.68 58.42) (xy 106.68 62.23)
 		)
 		(stroke
@@
 	(wire
 		(pts
-			(xy 106.68 69.85) (xy 106.68 71.12)
+			(xy 106.68 69.85) (xy 106.68 72.39)
 		)
 		(stroke
@@
 	(wire
 		(pts
-			(xy 106.68 68.58) (xy 106.68 69.85)
-		)
-		(stroke
-			(width 0)
-			(type default)
-		)
-	)
-	(wire
-		(pts
-			(xy 105.41 129.54) (xy 105.41 130.81)
+			(xy 106.68 67.31) (xy 106.68 69.85)
+		)
+		(stroke
+			(width 0)
+			(type default)
+		)
+	)
+	(wire
+		(pts
+			(xy 105.41 129.54) (xy 105.41 132.08)
 		)
 		(stroke
@@
 		(pts
 			(xy 113.03 74.93) (xy 113.03 100.33)
+		)
+		(stroke
+			(width 0)
+			(type default)
+		)
+	)
+	(wire
+		(pts
+			(xy 105.41 137.16) (xy 105.41 138.43)
 		)
 		(stroke
@@
 	)
 	(symbol
-		(lib_id "Device:R")
+		(lib_id "Device:R_Small")
 		(at 105.41 124.46 0)
 		(mirror y)
@@
 		)
 		(property "Footprint" "Resistor_SMD:R_0402_1005Metric"
-			(at 107.188 124.46 90)
+			(at 105.41 124.46 0)
 			(effects
 				(font
@@
 			)
 		)
-		(property "Description" "Resistor"
+		(property "Description" "Resistor, small symbol"
 			(at 105.41 124.46 0)
 			(effects
@@
 	)
 	(symbol
-		(lib_id "Device:R")
+		(lib_id "Device:R_Small")
 		(at 106.68 74.93 0)
 		(mirror y)
@@
 		)
 		(property "Footprint" "Resistor_SMD:R_0402_1005Metric"
-			(at 108.458 74.93 90)
+			(at 106.68 74.93 0)
 			(effects
 				(font
@@
 			)
 		)
-		(property "Description" "Resistor"
+		(property "Description" "Resistor, small symbol"
 			(at 106.68 74.93 0)
 			(effects
@@
 	)
 	(symbol
-		(lib_id "Device:R")
+		(lib_id "Device:R_Small")
 		(at 105.41 134.62 0)
 		(mirror y)
@@
 		)
 		(property "Footprint" "Resistor_SMD:R_0402_1005Metric"
-			(at 107.188 134.62 90)
+			(at 105.41 134.62 0)
 			(effects
 				(font
@@
 			)
 		)
-		(property "Description" "Resistor"
+		(property "Description" "Resistor, small symbol"
 			(at 105.41 134.62 0)
 			(effects
@@
 	)
 	(symbol
-		(lib_id "Device:R")
+		(lib_id "Device:R_Small")
 		(at 106.68 64.77 0)
 		(mirror y)
@@
 		)
 		(property "Footprint" "Resistor_SMD:R_0402_1005Metric"
-			(at 108.458 64.77 90)
+			(at 106.68 64.77 0)
 			(effects
 				(font
@@
 			)
 		)
-		(property "Description" "Resistor"
+		(property "Description" "Resistor, small symbol"
 			(at 106.68 64.77 0)
 			(effects

Commit message: [INV_Discrete_Controller] V1.2
Other:
- note added: "3.3v * ${Res1} / ${Res1}+${Res2} = 0.191V"
- note added: "3.3v * ${Res2} / ${Res1}+${Res2} =3.109V"
- note removed: "3.3v * ${Res2} / ${Res1}+${Res2} = 2.66V"
- note removed: "3.3v * 2.4 / 12.4 = 0.638v"
Changed lines of the file:
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@@
 	(title_block
 		(title "INV_Discrete_Controller")
-		(date "2026-03-15")
-		(rev "1.1")
+		(date "2026-03-17")
+		(rev "1.2")
 		(company "NTURacing")
 		(comment 1 "LY Chen")
@@
 		)
 	)
-	(text "3.3v * ${Res2} / ${Res1}+${Res2} = 2.66V"
+	(text "3.3v * ${Res1} / ${Res1}+${Res2} = 0.191V"
 		(exclude_from_sim no)
-		(at 86.106 70.358 0)
+		(at 81.28 130.302 0)
 		(effects
 			(font
@@
 		)
 	)
-	(text "3.3v * 2.4 / 12.4 = 0.638v\n"
+	(text "3.3v * ${Res2} / ${Res1}+${Res2} =3.109V"
 		(exclude_from_sim no)
-		(at 86.614 130.302 0)
+		(at 86.106 70.358 0)
 		(effects
 			(font
