File: Powertrain_Group/INV_Discrete_Controller/PWM_Enable.kicad_sch (KiCad schematic)
At the start: 2 parts, among them Q2 2N7002

Commit message: [INV_Discrete_Controller] V1.1
Parts:
- R94: renamed from R80; symbol Device:R -> Device:R_Small
- renumbered Q2 to Q4
Other:
- company: (none) -> NTURacing
- title: (none) -> INV_Discrete_Controller
Changed lines of the file:
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@@
 	(generator_version "9.0")
 	(paper "A4")
+	(title_block
+		(title "INV_Discrete_Controller")
+		(date "2026-03-15")
+		(rev "1.1")
+		(company "NTURacing")
+		(comment 1 "LY Chen")
+		(comment 2 "Jack Kuo")
+	)
 	(junction
 		(at 110.49 73.66)
@@
 	(wire
 		(pts
-			(xy 97.79 73.66) (xy 100.33 73.66)
+			(xy 97.79 73.66) (xy 101.6 73.66)
 		)
 		(stroke
@@
 	(wire
 		(pts
-			(xy 107.95 73.66) (xy 110.49 73.66)
+			(xy 106.68 73.66) (xy 110.49 73.66)
 		)
 		(stroke
@@
 		(dnp no)
 		(fields_autoplaced yes)
-		(property "Reference" "Q2"
+		(property "Reference" "Q4"
 			(at 114.3 86.3599 0)
 			(effects
@@
 	)
 	(symbol
-		(lib_id "Device:R")
+		(lib_id "Device:R_Small")
 		(at 104.14 73.66 270)
 		(unit 1)
@@
 		(dnp no)
 		(fields_autoplaced yes)
-		(property "Reference" "R80"
-			(at 104.14 67.31 90)
+		(property "Reference" "R94"
+			(at 104.14 68.58 90)
 			(effects
 				(font
@@
 		)
 		(property "Value" "510R"
-			(at 104.14 69.85 90)
+			(at 104.14 71.12 90)
 			(effects
 				(font
@@
 		)
 		(property "Footprint" "Resistor_SMD:R_0603_1608Metric"
-			(at 104.14 71.882 90)
+			(at 104.14 73.66 0)
 			(effects
 				(font
@@
 			)
 		)
-		(property "Description" "Resistor"
+		(property "Description" "Resistor, small symbol"
 			(at 104.14 73.66 0)
 			(effects
@@
 		(dnp no)
 		(fields_autoplaced yes)
-		(property "Reference" "#PWR0159"
+		(property "Reference" "#PWR0186"
 			(at 110.49 100.33 0)
 			(effects
