File: Powertrain_Group/INV_Discrete_Controller/Peripherals.kicad_sch (KiCad schematic)
At the start: 42 parts, among them J10 USB_C_stm32, U4 SRV05-4, U5 TCAN1042VDRQ1, U6 TCAN1042VDRQ1, U7 SN74LVC2G14DBV, U8 74LVC1G06

Commit message: [INV_Discrete_Controller] V1.1
Parts:
- C27, C28, C29, C30: value 0u1 -> 100n
- D10, D13, D14: symbol Device:LED -> Device:LED_Small_Filled
- FL2, FL3: footprint SamacSys_Parts_EP6:EXCX4CE900U -> nturt_kicad_lib_EP7:EXCX4CE900U; symbol SamacSys_Parts_EP6:EXC-X4CE900U -> nturt_kicad_lib_EP7:EXC-X4CE900U
- R19, R24, R29, R30, R33, R34: symbol Device:R -> Device:R_Small
- U5, U6: symbol nturt_kicad_lib_EP6:TCAN1042VDRQ1 -> nturt_kicad_lib_EP7:TCAN1042VDRQ1
Other:
- company: (none) -> NTURacing
- title: (none) -> INV_Discrete_Controller
