File: Powertrain_Group/INV_Discrete_Controller/SR_Latch.kicad_sch (KiCad schematic)
At the start: 3 parts, among them U21 74AUP1G00, U22 74AUP1G00, U23 74AUP1G07

Commit message: [INV_Discrete_Controller] V1.1
Other:
- company: (none) -> NTURacing
- title: (none) -> INV_Discrete_Controller
Changed lines of the file:
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@@
 	(generator_version "9.0")
 	(paper "A4")
+	(title_block
+		(title "INV_Discrete_Controller")
+		(date "2026-03-15")
+		(rev "1.1")
+		(company "NTURacing")
+		(comment 1 "LY Chen")
+		(comment 2 "Jack Kuo")
+	)
 	(text "S R Q Q!\n-----\n1 1 Q Q!\n0 1 1 0 \n1 0 0 1\n0 0 1 1"
 		(exclude_from_sim no)
