File: Powertrain_Group/INV_Discrete_Controller/TsenseNode.kicad_sch (KiCad schematic)
At the start: 4 parts

Commit message: [INV_Discrete_Controller] V1.1
Parts:
- R104, R105: symbol Device:R -> Device:R_Small
Other:
- company: (none) -> NTURacing
- title: (none) -> INV_Discrete_Controller
Changed lines of the file:
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@@
 	(generator_version "9.0")
 	(paper "A4")
+	(title_block
+		(title "INV_Discrete_Controller")
+		(date "2026-03-15")
+		(rev "1.1")
+		(company "NTURacing")
+		(comment 1 "LY Chen")
+		(comment 2 "Jack Kuo")
+	)
 	(text "Vout = NTC/(R+NTC)*3V3"
 		(exclude_from_sim no)
@@
 	(wire
 		(pts
-			(xy 105.41 92.71) (xy 114.3 92.71)
+			(xy 105.41 92.71) (xy 115.57 92.71)
 		)
 		(stroke
@@
 	(wire
 		(pts
-			(xy 105.41 91.44) (xy 105.41 92.71)
-		)
-		(stroke
-			(width 0)
-			(type default)
-		)
-	)
-	(wire
-		(pts
-			(xy 105.41 83.82) (xy 105.41 82.55)
+			(xy 105.41 90.17) (xy 105.41 92.71)
+		)
+		(stroke
+			(width 0)
+			(type default)
+		)
+	)
+	(wire
+		(pts
+			(xy 120.65 92.71) (xy 123.19 92.71)
+		)
+		(stroke
+			(width 0)
+			(type default)
+		)
+	)
+	(wire
+		(pts
+			(xy 105.41 82.55) (xy 105.41 85.09)
 		)
 		(stroke
@@
 		(pts
 			(xy 123.19 92.71) (xy 123.19 95.25)
-		)
-		(stroke
-			(width 0)
-			(type default)
-		)
-	)
-	(wire
-		(pts
-			(xy 123.19 92.71) (xy 121.92 92.71)
 		)
 		(stroke
@@
 	)
 	(symbol
-		(lib_id "Device:R")
+		(lib_id "Device:R_Small")
 		(at 118.11 92.71 90)
 		(unit 1)
@@
 		(fields_autoplaced yes)
 		(property "Reference" "R105"
-			(at 118.11 86.36 90)
+			(at 118.11 87.63 90)
 			(effects
 				(font
@@
 		)
 		(property "Value" "1K"
-			(at 118.11 88.9 90)
+			(at 118.11 90.17 90)
 			(effects
 				(font
@@
 		)
 		(property "Footprint" "Resistor_SMD:R_0603_1608Metric"
-			(at 118.11 94.488 90)
+			(at 118.11 92.71 0)
 			(effects
 				(font
@@
 			)
 		)
-		(property "Description" "Resistor"
+		(property "Description" "Resistor, small symbol"
 			(at 118.11 92.71 0)
 			(effects
@@
 	)
 	(symbol
-		(lib_id "Device:R")
+		(lib_id "Device:R_Small")
 		(at 105.41 87.63 0)
 		(unit 1)
@@
 		)
 		(property "Footprint" "Resistor_SMD:R_0603_1608Metric"
-			(at 103.632 87.63 90)
+			(at 105.41 87.63 0)
 			(effects
 				(font
@@
 			)
 		)
-		(property "Description" "Resistor"
+		(property "Description" "Resistor, small symbol"
 			(at 105.41 87.63 0)
 			(effects

Commit message: [INV_Discrete_Controller] V1.2
Parts:
- C95, C96: value 1uF -> 1u
Changed lines of the file:
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@@
 	(title_block
 		(title "INV_Discrete_Controller")
-		(date "2026-03-15")
-		(rev "1.1")
+		(date "2026-03-17")
+		(rev "1.2")
 		(company "NTURacing")
 		(comment 1 "LY Chen")
@@
 			)
 		)
-		(property "Value" "1uF"
+		(property "Value" "1u"
 			(at 125.73 99.0662 0)
 			(effects
@@
 			)
 		)
-		(property "Value" "1uF"
+		(property "Value" "1u"
 			(at 107.95 96.5262 0)
 			(effects
