File: Powertrain_Group/INV_Discrete_Controller/power.kicad_sch (KiCad schematic)
At the start: 45 parts, among them J8 LVBattery, J9 LVBattery, U1 TPS5430DDAR, U2 AMS1117-3.3

Commit message: [INV_Discrete_Controller] V1.1
Parts:
- removed C20: 100uF 27V, Capacitor_THT:CP_Radial_D10.0mm_P5.00mm, symbol Device:C_Polarized_Small
- removed D6: SS54, Diode_SMD:D_SMA, symbol PCM_Diode_Schottky_AKL:SS54
- C3: value 0u1 -> 100n
- D3: symbol PCM_Diode_Schottky_AKL:SS54 -> Device:D_Schottky_Small_Filled
- D4, D8, D9: symbol Device:LED -> Device:LED_Small_Filled
- FL1: footprint SamacSys_Parts_EP6:ACM70V7012PLTL00 -> nturt_kicad_lib_EP7:Common_Mode_Choke_4A_ACM70V7012PLTL00; symbol SamacSys_Parts_EP6:ACM70V-701-2PL-TL00 -> nturt_kicad_lib_EP7:ACM70V-701-2PL-TL00
- L2: footprint SamacSys_Parts_EP6:SRR1260A220M -> Inductor_SMD:L_Bourns_SRR1260
- R10: value 510R -> 10k; symbol Device:R -> Device:R_Small
- R6: value 47k 1% -> 47k; symbol Device:R -> Device:R_Small
- R7: value 15k 1% -> 15k; symbol Device:R -> Device:R_Small
- R8: value 1k -> 10k; symbol Device:R -> Device:R_Small
- R9: value 10k -> 47k; symbol Device:R -> Device:R_Small
- U1: symbol nturt_kicad_lib_EP6:TPS5430DDAR -> nturt_kicad_lib_EP7:TPS5430DDAR
Connections:
- net +24V: now also F2.2
Other:
- note removed: "49.9k & 5.9k = 9.5x attenuation w/ input impedance of 5.25k"
- company: (none) -> NTURacing
- title: (none) -> INV_Discrete_Controller
- moved on the sheet: D3, D7, R9

Commit message: [INV_Discrete_Controller] V1.2
Parts:
- added D201, D202, D203, D204: WHITE LED, LED_SMD:LED_0603_1608Metric, symbol Device:LED_Small_Filled
Connections:
- net +5V: now also D4.2 (A), D201.2 (A), D202.2 (A), D203.2 (A), D204.2 (A)
- net 5V_buck: no longer D4.2 (A)
- net at D4.1 (K), R8.1: now also D201.1 (K), D202.1 (K), D203.1 (K), D204.1 (K)
Other:
- moved on the sheet: C108, C37, D4, D5, F1, R8, TP1
