File: Electrical_Group/VCU_CM4/CAN.kicad_sch (KiCad schematic)
At the start: 8 parts, among them U17 TCAN1042VDRQ1

Commit message: [VCU_CM4] V1.1
Other:
- note added: "can replace with TCAN1057AV (note only the "AV" version has VDDIO for 3.3V the "A" version does not support VDDIO)"
Changed lines of the file:
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@@
 	(title_block
 		(title "VCU_CM4")
-		(date "2026-05-22")
-		(rev "1.0")
+		(date "2026-05-23")
+		(rev "1.1")
 		(company "NTURacing Team")
 		(comment 1 "Jack Kuo")
 		(comment 2 "Jerry mk")
 	)
+	(text "can replace with TCAN1057AV\n(note only the \"AV\" version has VDDIO for 3.3V\nthe \"A\" version does not support VDDIO)"
+		(exclude_from_sim no)
+		(at 115.824 105.664 0)
+		(effects
+			(font
+				(size 1.27 1.27)
+			)
+			(justify left top)
+		)
+	)
 	(junction
