File: Electrical_Group/VCU_CM4/VCU_CM4.kicad_sch (KiCad schematic)
At the start: 29 parts, among them J24 USB_C_stm32

Commit message: [VCU_CM4] V1.1
Parts:
- added R174, R175, R176: 0R, Resistor_SMD:R_0603_1608Metric_Pad0.98x0.95mm_HandSolder, symbol Device:R_Small
Connections:
- new net 24V_lowTrig: R176.1
- new net 40P.GPIO14: R175.1
- new net 40P.GPIO15: R174.1
- new net 40P.GPIO25: R176.2
- new net VCP_MCU_UART.RX: R175.2
- new net VCP_MCU_UART.TX: R174.2
Other:
- note added: "RPI_UART_RX"
- note added: "RPI_UART_TX"
- note added: "next time use a spare UART"
