File: Electrical_Group/VCU_CM4/computer.kicad_sch (KiCad schematic)
At the start: 46 parts, among them J4 MIPI_DSI_22P, J5 MIPI_CAM_22P, J7 MSD-4-A, Q4 AO3401A, SW1 RPI_CPU_RST, SW6 RPI_PWR, U10 MCP2518FD, U20 MCP7940N-xSN, U6 TLV75733PDRV, U7 TLV75733PDRV, U8 TLV75733PDRV, U9 MCP2518FD, Y2 40Mhz XTM32040000DT00351001, Y3 40Mhz XTM32040000DT00351001, Y7 32.768kHz Q13FC13500004

Commit message: [VCU_CM4] V1.1
Parts:
- U6, U7, U8: value TLV75733PDRV -> TLV75733; footprint Package_SON:WSON-6-1EP_2x2mm_P0.65mm_EP1x1.6mm -> Package_TO_SOT_SMD:SOT-23-5; symbol Regulator_Linear:TLV75733PDRV -> Regulator_Linear:TLV75733PDBV
Connections:
- net +5V_RPI: now also U6.1 (IN), U7.1 (IN), U8.1 (IN); no longer U6.6 (IN), U7.6 (IN), U8.6 (IN)
- net 3V3_CAM: now also U7.5 (OUT); no longer U7.1 (OUT)
- net 3V3_DISP: now also U8.5 (OUT); no longer U8.1 (OUT)
- net GND: now also U6.2 (GND), U7.2 (GND), U8.2 (GND); no longer U6.3 (GND), U6.7 (GND), U7.3 (GND), U7.7 (GND), U8.3 (GND), U8.7 (GND)
- net SD_PWR_ON: now also U6.3 (EN); no longer U6.4 (EN)
- net at R55.2: now also U7.3 (EN); no longer U7.4 (EN)
- net at C46.1, C49.1, J7.4 (VDD): now also U6.5 (OUT); no longer U6.1 (OUT)
- net at R56.2: now also U8.3 (EN); no longer U8.4 (EN)
Other:
- note added: "NOTE!!! remember to change the cs pins in future versions change to hardware cs pins for easier dtoverlay for cm4"
Changed lines of the file:
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@@
 	(title_block
 		(title "VCU_CM4")
-		(date "2026-05-22")
-		(rev "1.0")
+		(date "2026-05-23")
+		(rev "1.1")
 		(company "NTURacing Team")
 		(comment 1 "Jack Kuo")
@@
 		)
 	)
+	(text "NOTE!!!\nremember to change the cs pins in future versions\nchange to hardware cs pins for easier dtoverlay for cm4"
+		(exclude_from_sim no)
+		(at 175.006 155.194 0)
+		(effects
+			(font
+				(size 2.54 2.54)
+				(thickness 0.508)
+				(bold yes)
+				(color 255 0 0 1)
+			)
+			(justify left top)
+		)
+	)
 	(text "from CM4 IO board shcematic"
 		(exclude_from_sim no)
@@
 	)
 	(symbol
-		(lib_id "Regulator_Linear:TLV75733PDRV")
+		(lib_id "Regulator_Linear:TLV75733PDBV")
 		(at 163.83 34.29 0)
 		(unit 1)
@@
 			)
 		)
-		(property "Value" "TLV75733PDRV"
+		(property "Value" "TLV75733"
 			(at 163.83 27.94 0)
 			(effects
@@
 			)
 		)
-		(property "Footprint" "Package_SON:WSON-6-1EP_2x2mm_P0.65mm_EP1x1.6mm"
+		(property "Footprint" "Package_TO_SOT_SMD:SOT-23-5"
 			(at 163.83 26.035 0)
 			(effects
@@
 			)
 		)
-		(property "Description" "1A Low IQ Small Size Low Dropout Voltage Regulator, Fixed Output 3.3V, WSON6"
+		(property "Description" "1A Low IQ Small Size Low Dropout Voltage Regulator, Fixed Output 3.3V, SOT-23-5"
 			(at 163.83 34.29 0)
 			(effects
@@
 		(pin "3"
 		)
-		(pin "6"
-		)
 		(pin "4"
 		)
-		(pin "7"
-		)
 		(instances
 			(project "VCU_CM4"
@@
 	)
 	(symbol
-		(lib_id "Regulator_Linear:TLV75733PDRV")
+		(lib_id "Regulator_Linear:TLV75733PDBV")
 		(at 158.75 69.85 0)
 		(unit 1)
@@
 			)
 		)
-		(property "Value" "TLV75733PDRV"
+		(property "Value" "TLV75733"
 			(at 158.75 63.5 0)
 			(effects
@@
 			)
 		)
-		(property "Footprint" "Package_SON:WSON-6-1EP_2x2mm_P0.65mm_EP1x1.6mm"
+		(property "Footprint" "Package_TO_SOT_SMD:SOT-23-5"
 			(at 158.75 61.595 0)
 			(effects
@@
 			)
 		)
-		(property "Description" "1A Low IQ Small Size Low Dropout Voltage Regulator, Fixed Output 3.3V, WSON6"
+		(property "Description" "1A Low IQ Small Size Low Dropout Voltage Regulator, Fixed Output 3.3V, SOT-23-5"
 			(at 158.75 69.85 0)
 			(effects
@@
 		(pin "3"
 		)
-		(pin "6"
-		)
 		(pin "4"
 		)
-		(pin "7"
-		)
 		(instances
 			(project "VCU_CM4"
@@
 	)
 	(symbol
-		(lib_id "Regulator_Linear:TLV75733PDRV")
+		(lib_id "Regulator_Linear:TLV75733PDBV")
 		(at 158.75 101.6 0)
 		(unit 1)
@@
 			)
 		)
-		(property "Value" "TLV75733PDRV"
+		(property "Value" "TLV75733"
 			(at 158.75 95.25 0)
 			(effects
@@
 			)
 		)
-		(property "Footprint" "Package_SON:WSON-6-1EP_2x2mm_P0.65mm_EP1x1.6mm"
+		(property "Footprint" "Package_TO_SOT_SMD:SOT-23-5"
 			(at 158.75 93.345 0)
 			(effects
@@
 			)
 		)
-		(property "Description" "1A Low IQ Small Size Low Dropout Voltage Regulator, Fixed Output 3.3V, WSON6"
+		(property "Description" "1A Low IQ Small Size Low Dropout Voltage Regulator, Fixed Output 3.3V, SOT-23-5"
 			(at 158.75 101.6 0)
 			(effects
@@
 		(pin "3"
 		)
-		(pin "6"
-		)
 		(pin "4"
 		)
-		(pin "7"
-		)
 		(instances
