File: Electrical_Group/VCU_CM4/current_loop_sensors.kicad_sch (KiCad schematic)
At the start: 61 parts, among them J8 Conn_01x30_Socket

Commit message: [VCU_CM4] V1.1
Parts:
- added F26: 0.5A, Fuse:Fuse_1206_3216Metric, symbol Device:Fuse_Small
- J8: value Conn_01x30_Socket -> current_loops
Connections:
- net +24V: now also F26.1; no longer F10.1, F11.1, F12.1, F13.1, F14.1, F15.1, F16.1, F17.1, F18.1, F19.1, F20.1, F21.1, F22.1, F23.1, F24.1, F5.1, F6.1, F7.1, F8.1, F9.1
- new net: F10.1, F11.1, F12.1, F13.1, F14.1, F15.1, F16.1, F17.1, F18.1, F19.1, F20.1, F21.1, F22.1, F23.1, F24.1, F26.2, F5.1, F6.1, F7.1, F8.1, F9.1
Changed lines of the file:
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@@
 	(title_block
 		(title "VCU_CM4")
-		(date "2026-05-22")
-		(rev "1.0")
+		(date "2026-05-23")
+		(rev "1.1")
 		(company "NTURacing Team")
 		(comment 1 "Jack Kuo")
@@
 	(wire
 		(pts
-			(xy 129.54 33.02) (xy 129.54 39.37)
+			(xy 129.54 25.4) (xy 129.54 29.21)
 		)
 		(stroke
@@
 	(wire
 		(pts
+			(xy 129.54 34.29) (xy 129.54 39.37)
+		)
+		(stroke
+			(width 0)
+			(type default)
+		)
+	)
+	(wire
+		(pts
 			(xy 57.15 59.69) (xy 77.47 59.69)
 		)
@@
 	(symbol
 		(lib_id "Device:Fuse_Small")
+		(at 129.54 31.75 270)
+		(unit 1)
+		(exclude_from_sim no)
+		(in_bom yes)
+		(on_board yes)
+		(dnp no)
+		(fields_autoplaced yes)
+		(property "Reference" "F26"
+			(at 130.81 30.4799 90)
+			(effects
+				(font
+					(size 1.27 1.27)
+				)
+				(justify left)
+			)
+		)
+		(property "Value" "0.5A"
+			(at 130.81 33.0199 90)
+			(effects
+				(font
+					(size 1.27 1.27)
+				)
+				(justify left)
+			)
+		)
+		(property "Footprint" "Fuse:Fuse_1206_3216Metric"
+			(at 129.54 31.75 0)
+			(effects
+				(font
+					(size 1.27 1.27)
+				)
+				(hide yes)
+			)
+		)
+		(property "Datasheet" "~"
+			(at 129.54 31.75 0)
+			(effects
+				(font
+					(size 1.27 1.27)
+				)
+				(hide yes)
+			)
+		)
+		(property "Description" "Fuse, small symbol"
+			(at 129.54 31.75 0)
+			(effects
+				(font
+					(size 1.27 1.27)
+				)
+				(hide yes)
+			)
+		)
+		(pin "1"
+		)
+		(pin "2"
+		)
+		(instances
+			(project "VCU_CM4"
+				(path "/eb296f24-894e-4ea0-b0cd-3ba211155378/59ca343a-7d66-4d76-8c27-2a427ae9c4b3/553e4d5b-d7d4-4625-993b-7bf191101b33"
+					(reference "F26")
+					(unit 1)
+				)
+			)
+		)
+	)
+	(symbol
+		(lib_id "Device:Fuse_Small")
 		(at 95.25 64.77 180)
 		(unit 1)
@@
 	(symbol
 		(lib_id "power:+24V")
-		(at 129.54 33.02 0)
+		(at 129.54 25.4 0)
 		(unit 1)
 		(exclude_from_sim no)
@@
 		(fields_autoplaced yes)
 		(property "Reference" "#PWR0126"
-			(at 129.54 36.83 0)
+			(at 129.54 29.21 0)
 			(effects
 				(font
@@
 		)
 		(property "Value" "+24V"
-			(at 129.54 28.575 0)
+			(at 129.54 20.955 0)
 			(effects
 				(font
@@
 		)
 		(property "Footprint" ""
-			(at 129.54 33.02 0)
+			(at 129.54 25.4 0)
 			(effects
 				(font
@@
 		)
 		(property "Datasheet" ""
-			(at 129.54 33.02 0)
+			(at 129.54 25.4 0)
 			(effects
 				(font
@@
 		)
 		(property "Description" "Power symbol creates a global label with name \"+24V\""
-			(at 129.54 33.02 0)
+			(at 129.54 25.4 0)
 			(effects
 				(font
@@
 			)
 		)
-		(property "Value" "Conn_01x30_Socket"
+		(property "Value" "current_loops"
 			(at 52.07 87.6301 0)
 			(effects
