File: Electrical_Group/VCU_CM4/power.kicad_sch (KiCad schematic)
At the start: 34 parts, among them J1 RPI_UPS, J2 VCU_UPS, Q1 AO3400A, U1 LM66100DCK, U2 TLV75733PDRV

Commit message: [VCU_CM4] V1.1
Parts:
- F2: value 0.5A -> 1A
- U2: value TLV75733PDRV -> TLV75733; footprint Package_SON:WSON-6-1EP_2x2mm_P0.65mm_EP1x1.6mm -> Package_TO_SOT_SMD:SOT-23-5; symbol Regulator_Linear:TLV75733PDRV -> Regulator_Linear:TLV75733PDBV
Connections:
- net +3V3: now also U2.5 (OUT); no longer U2.1 (OUT)
- net 5V_proUPS: now also U2.1 (IN); no longer U2.6 (IN)
- net GND: now also U2.2 (GND); no longer U2.3 (GND), U2.7 (GND)
- net at R11.2: now also U2.3 (EN); no longer U2.4 (EN)
Changed lines of the file:
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@@
 	(title_block
 		(title "VCU_CM4")
-		(date "2026-05-22")
-		(rev "1.0")
+		(date "2026-05-23")
+		(rev "1.1")
 		(company "NTURacing Team")
 		(comment 1 "Jack Kuo")
@@
 			)
 		)
-		(property "Value" "0.5A"
+		(property "Value" "1A"
 			(at 134.62 34.29 0)
 			(effects
@@
 	)
 	(symbol
-		(lib_id "Regulator_Linear:TLV75733PDRV")
+		(lib_id "Regulator_Linear:TLV75733PDBV")
 		(at 212.09 76.2 0)
 		(unit 1)
@@
 			)
 		)
-		(property "Value" "TLV75733PDRV"
+		(property "Value" "TLV75733"
 			(at 212.09 69.85 0)
 			(effects
@@
 			)
 		)
-		(property "Footprint" "Package_SON:WSON-6-1EP_2x2mm_P0.65mm_EP1x1.6mm"
+		(property "Footprint" "Package_TO_SOT_SMD:SOT-23-5"
 			(at 212.09 67.945 0)
 			(effects
@@
 			)
 		)
-		(property "Description" "1A Low IQ Small Size Low Dropout Voltage Regulator, Fixed Output 3.3V, WSON6"
+		(property "Description" "1A Low IQ Small Size Low Dropout Voltage Regulator, Fixed Output 3.3V, SOT-23-5"
 			(at 212.09 76.2 0)
 			(effects
@@
 		(pin "3"
 		)
-		(pin "6"
-		)
 		(pin "4"
 		)
-		(pin "7"
-		)
 		(instances
