File: Electrical_Group/VCU_CM4/vcu_mcu.kicad_sch (KiCad schematic)
At the start: 48 parts, among them J10 MSD-4-A, J9 Conn_02x15_Odd_Even, SW2 RESET, SW3 BOOT0, U11 REF3133AIDBZR, U12 STM32H743ZITx, Y4 40Mhz XTM32040000DT00351001, Y5 32.768kHz Q13FC13500004

Commit message: [VCU_CM4] V1.1
Parts:
- added C132: 100n, Capacitor_SMD:C_0402_1005Metric, symbol Device:C_Small
- added R170, R171, R172, R173: 2k2, Resistor_SMD:R_0402_1005Metric, symbol Device:R_Small
- J9: value Conn_02x15_Odd_Even -> to_Dash_Screen
- Y4: value 40Mhz XTM32040000DT00351001 -> 8Mhz
Connections:
- net +3V3: now also R170.2, R171.2, R172.2, R173.2
- net BOOT0: now also C132.1
- net GND: now also C132.2
- net I2C2_SCL: now also R171.1
- net I2C2_SDA: now also R172.1
- net I2C4_SCL: now also R170.1
- net I2C4_SDA: now also R173.1
- net SPI2_CS: now reaches J9.19 (Pin_19)
- net SPI2_CS: now also U12.73 (PB12)
- net SPI2_SCK: now reaches J9.20 (Pin_20)
- net SPI2_SCK: now also U12.74 (PB13)
- net SPI2_MOSI: now reaches J9.21 (Pin_21)
- net SPI2_MOSI: now also U12.76 (PB15)
- net SPI2_MISO: now reaches J9.22 (Pin_22)
- net SPI2_MISO: now also U12.75 (PB14)
- no-connect marks 55 -> 47
Other:
- note added: "for WS2812b RGB"
