File: Electrical_Group/Dash_Screen/Dash_Screen.kicad_pcb (KiCad board)
At the start: 2 copper layers, 100 x 90 mm, 57 parts, among them J1 RTD_BUT_LIGHT, J2 RTD_BUT_LIGHT, J9 to Dash_Screen_under, Q1 2N7002, Q2 AO3400A, U11 74HC595, U12 74HC595, U14 AMS1117-3.3, U17 SN74LVC4245APWR

Commit message: [Dash_Screen] V2.0
Parts:
- turned J9 to 90 degrees
- turned R70 to 90 degrees
Connections:
- U12 pad 14: /Dash_Screen_ShiftRegs/SER -> /REG_for_Dash_Screen
- U17 pad 16: /REG_for_Dash_Screen -> /SPI4_CS0
- U17 pad 17: /SPI4_LEDPWM -> /SPI4_SCK
- U17 pad 18: /SPI4_CS0 -> /SPI4_LEDPWM
- U17 pad 19: /SPI4_SCK -> unconnected-(U17-B3-Pad19)
- U17 pad 5: /Dash_Screen_ShiftRegs/RCLK -> unconnected-(U17-A3-Pad5)
- U17 pad 6: /Dash_Screen_ShiftRegs/OE -> /Dash_Screen_ShiftRegs/SRCLK
- U17 pad 7: /Dash_Screen_ShiftRegs/SRCLK -> /Dash_Screen_ShiftRegs/RCLK
- U17 pad 8: /Dash_Screen_ShiftRegs/SER -> /Dash_Screen_ShiftRegs/OE
Routing:
- net /REG_for_Dash_Screen: track 7.68 -> 49.8 mm, vias 0 -> 2
- net /Dash_Screen_ShiftRegs/SER: track 39.1 -> 0.00 mm
- net +5V: track 215.3 -> 237.1 mm, vias 8 -> 4
- net /SPI4_LEDPWM: track 9.89 -> 30.9 mm
- net /SPI4_SCK: track 10.00 -> 30.2 mm
- net /SPI4_CS0: track 12.3 -> 27.7 mm
- net Net-(U11-SER): track 28.8 -> 41.0 mm, vias 2 -> 0
- net GND: track 18.7 -> 25.3 mm, vias 10 -> 17
- net /Dash_Screen_ShiftRegs/OE: track 60.1 -> 61.8 mm
- net Net-(U12-QA): track 10.2 -> 8.69 mm
- net /Dash_Screen_ShiftRegs/SRCLK: track 74.1 -> 75.5 mm
- net /Dash_Screen_ShiftRegs/RCLK: track 62.2 -> 63.5 mm
Other:
- outline, holes or cut-outs redrawn
- board text added: "Dash_Screen V2.0 26/06/10"
- board text removed: "Dash_Screen V1.0 26/05/23"
