File: Electrical_Group/Dash_Screen/Dash_Screen.kicad_sch (KiCad schematic)
At the start: 13 parts, among them J9 to Dash_Screen_under, U14 AMS1117-3.3, U17 SN74LVC4245APWR

Commit message: [Dash_Screen] V2.0
Connections:
- net Dash_Screen_ShiftRegs/SERin is gone; now on net Dash_Screen_ShiftRegs/OEin: U17.8 (A6)
- net Dash_Screen_ShiftRegs/OEin: no longer U17.6 (A4)
- net Dash_Screen_ShiftRegs/RCLKin: now also U17.7 (A5); no longer U17.5 (A3)
- net Dash_Screen_ShiftRegs/SRCLKin: now also U17.6 (A4); no longer U17.7 (A5)
- net REG_for_Dash_Screen: no longer U17.16 (B6)
- net SPI4_CS0: now also U17.16 (B6); no longer U17.18 (B4)
- net SPI4_LEDPWM: now also U17.18 (B4); no longer U17.17 (B5)
- net SPI4_SCK: now also U17.17 (B5); no longer U17.19 (B3)
Changed lines of the file:
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@@
 	(title_block
 		(title "Dash_Screen")
-		(date "2026-05-23")
-		(rev "1.0")
+		(date "2026-06-10")
+		(rev "2.0")
 		(company "NTURacing")
 		(comment 1 "郭哲明")
@@
 	(wire
 		(pts
-			(xy 48.26 74.93) (xy 69.85 74.93)
-		)
-		(stroke
-			(width 0)
-			(type default)
-		)
-	)
-	(wire
-		(pts
 			(xy 57.15 146.05) (xy 64.77 146.05)
 		)
@@
 	(wire
 		(pts
-			(xy 90.17 74.93) (xy 114.3 74.93)
+			(xy 77.47 146.05) (xy 88.9 146.05)
 		)
 		(stroke
@@
 	(wire
 		(pts
-			(xy 77.47 146.05) (xy 88.9 146.05)
+			(xy 35.56 74.93) (xy 69.85 74.93)
 		)
 		(stroke
@@
 	(wire
 		(pts
-			(xy 46.99 80.01) (xy 69.85 80.01)
-		)
-		(stroke
-			(width 0)
-			(type default)
-		)
-	)
-	(wire
-		(pts
 			(xy 34.29 171.45) (xy 64.77 171.45)
 		)
@@
 	(wire
 		(pts
-			(xy 90.17 69.85) (xy 114.3 69.85)
-		)
-		(stroke
-			(width 0)
-			(type default)
-		)
-	)
-	(wire
-		(pts
 			(xy 93.98 46.99) (xy 93.98 48.26)
 		)
@@
 	(wire
 		(pts
-			(xy 77.47 171.45) (xy 90.17 171.45)
+			(xy 100.33 64.77) (xy 121.92 64.77)
 		)
 		(stroke
@@
 	(wire
 		(pts
-			(xy 48.26 69.85) (xy 69.85 69.85)
+			(xy 77.47 171.45) (xy 90.17 171.45)
 		)
 		(stroke
@@
 	(wire
 		(pts
-			(xy 191.77 54.61) (xy 194.31 54.61)
+			(xy 90.17 69.85) (xy 121.92 69.85)
 		)
 		(stroke
@@
 	(wire
 		(pts
-			(xy 90.17 80.01) (xy 114.3 80.01)
+			(xy 191.77 54.61) (xy 194.31 54.61)
 		)
 		(stroke
@@
 	(wire
 		(pts
-			(xy 57.15 156.21) (xy 64.77 156.21)
+			(xy 90.17 74.93) (xy 121.92 74.93)
 		)
 		(stroke
@@
 	(wire
 		(pts
-			(xy 45.72 158.75) (xy 64.77 158.75)
+			(xy 57.15 156.21) (xy 64.77 156.21)
 		)
 		(stroke
@@
 	(wire
 		(pts
-			(xy 49.53 140.97) (xy 64.77 140.97)
+			(xy 45.72 158.75) (xy 64.77 158.75)
 		)
 		(stroke
@@
 	(wire
 		(pts
-			(xy 80.01 101.6) (xy 80.01 100.33)
+			(xy 49.53 140.97) (xy 64.77 140.97)
 		)
 		(stroke
@@
 	(wire
 		(pts
-			(xy 90.17 64.77) (xy 114.3 64.77)
+			(xy 80.01 101.6) (xy 80.01 100.33)
 		)
 		(stroke
@@
 	(wire
 		(pts
+			(xy 35.56 80.01) (xy 69.85 80.01)
+		)
+		(stroke
+			(width 0)
+			(type default)
+		)
+	)
+	(wire
+		(pts
 			(xy 49.53 138.43) (xy 64.77 138.43)
 		)
@@
 	(wire
 		(pts
+			(xy 90.17 80.01) (xy 121.92 80.01)
+		)
+		(stroke
+			(width 0)
+			(type default)
+		)
+	)
+	(wire
+		(pts
 			(xy 90.17 95.25) (xy 91.44 95.25)
 		)
@@
 	(wire
 		(pts
-			(xy 93.98 40.64) (xy 82.55 40.64)
+			(xy 35.56 69.85) (xy 69.85 69.85)
 		)
 		(stroke
@@
 	(wire
 		(pts
-			(xy 48.26 64.77) (xy 69.85 64.77)
+			(xy 93.98 40.64) (xy 82.55 40.64)
 		)
 		(stroke
@@
 		)
 	)
+	(label "REG_for_Dash_Screen"
+		(at 100.33 64.77 0)
+		(effects
+			(font
+				(size 1.27 1.27)
+			)
+			(justify left bottom)
+		)
+	)
 	(label "BUT4"
 		(at 88.9 146.05 180)
@@
 		)
 	)
+	(label "SPI4_LEDPWM"
+		(at 35.56 69.85 0)
+		(effects
+			(font
+				(size 1.27 1.27)
+			)
+			(justify left bottom)
+		)
+	)
 	(label "BUT5"
 		(at 57.15 148.59 0)
@@
 		)
 	)
-	(label "REG_for_Dash_Screen"
-		(at 46.99 80.01 0)
-		(effects
-			(font
-				(size 1.27 1.27)
-			)
-			(justify left bottom)
-		)
-	)
-	(label "SPI4_CS0"
-		(at 48.26 69.85 0)
-		(effects
-			(font
-				(size 1.27 1.27)
-			)
-			(justify left bottom)
-		)
-	)
 	(label "BUT6"
 		(at 88.9 148.59 180)
@@
 	)
 	(label "SPI4_SCK"
-		(at 48.26 64.77 0)
+		(at 35.56 74.93 0)
 		(effects
 			(font
@@
 		)
 	)
-	(label "BUT8"
-		(at 88.9 151.13 180)
+	(label "SPI4_CS0"
+		(at 35.56 80.01 0)
 		(effects
 			(font
 				(size 1.27 1.27)
 			)
-			(justify right bottom)
+			(justify left bottom)
 		)
 	)
-	(label "SPI2_MOSI"
-		(at 45.72 161.29 0)
+	(label "BUT8"
+		(at 88.9 151.13 180)
 		(effects
 			(font
 				(size 1.27 1.27)
 			)
-			(justify left bottom)
+			(justify right bottom)
 		)
 	)
-	(label "SPI4_LEDPWM"
-		(at 48.26 74.93 0)
+	(label "SPI2_MOSI"
+		(at 45.72 161.29 0)
 		(effects
 			(font
@@
 	)
 	(sheet
-		(at 114.3 43.18)
+		(at 121.92 43.18)
 		(size 12.7 55.88)
 		(exclude_from_sim no)
@@
 		)
 		(property "Sheetname" "Dash_Screen_ShiftRegs"
-			(at 114.3 42.4684 0)
+			(at 121.92 42.4684 0)
 			(effects
 				(font
@@
 		)
 		(property "Sheetfile" "Dash_Screen_ShiftRegs.kicad_sch"
-			(at 114.3 99.6446 0)
+			(at 121.92 99.6446 0)
 			(effects
 				(font
@@
 		)
 		(pin "RCLKin" input
-			(at 114.3 64.77 180)
+			(at 121.92 74.93 180)
 			(effects
 				(font
@@
 		)
 		(pin "SRCLKin" input
-			(at 114.3 74.93 180)
+			(at 121.92 69.85 180)
 			(effects
 				(font
@@
 		)
 		(pin "SERin" input
-			(at 114.3 80.01 180)
+			(at 121.92 64.77 180)
 			(effects
 				(font
@@
 		)
 		(pin "OEin" input
-			(at 114.3 69.85 180)
+			(at 121.92 80.01 180)
 			(effects
 				(font
