File: Electrical_Group/Dash_Screen_Under/Dash_Screen_Under.kicad_pcb (KiCad board)
At the start: 4 copper layers, 100 x 90 mm, 135 parts, among them J1 pedal1-1 RED, J2 pedal1-2 RED, J3 pedal2-1 GREEN, J4 pedal2-2 GREEN, J5 to upper Dash_Screen, J6 buttons, J7 12864, J9 to VCU_CM4, U1 Seg2 WHITE .56, U10 74HC595, U11 74HC595, U12 74HC595, U13 74HC595, U14 AMS1117-3.3, U17 SN74LVC4245APWR, U2 Seg1 GREEN .56, U3 Seg0 GREEN .56, U4 74HC595, U5 Seg3 WHITE .56, U6 74HC595, U7 74HC595, U8 74HC595, U9 74HC595

Commit message: [Dash_Screen_Under] V2.0
Parts:
- added H5: 12864 support, MountingHole:MountingHole_3.2mm_M3, F.Cu at (131.0, 114.2)
- added H6: 12864 support, MountingHole:MountingHole_3.2mm_M3, F.Cu at (156.8, 114.2)
- added Q1: 2N7002, Package_TO_SOT_SMD:SOT-23, B.Cu at (86.8, 121.9)
- added Q2: AO3400A, Package_TO_SOT_SMD:SOT-23, B.Cu at (86.8, 117.9)
- added R81: 0R, Resistor_SMD:R_0805_2012Metric_Pad1.20x1.40mm_HandSolder, B.Cu at (82.4, 121.9)
- added R82: 0R, Resistor_SMD:R_0805_2012Metric_Pad1.20x1.40mm_HandSolder, B.Cu at (82.5, 117.9)
- added R83: 0R, Resistor_SMD:R_0603_1608Metric, B.Cu at (91.0, 121.2)
- added R84: 0R, Resistor_SMD:R_0603_1608Metric, B.Cu at (91.0, 119.0)
- added TP5: AUX_P, nturt_kicad_lib_EP7:edge_pad_1.4mm_0.7mm, F.Cu at (63.0, 85.0)
- R75: value 1k -> 10k
- TP6: renamed from TP5; value AUX -> AUX_N
- moved C26 14.2 mm to (103.8, 106.7), turned to -90 degrees
- moved R75 11.7 mm to (115.7, 96.7), turned to -90 degrees
- moved D62 11.0 mm to (109.2, 94.2), turned to 180 degrees
- moved C58 10.8 mm to (112.6, 96.9), turned to 0 degrees
- moved U17 10.0 mm to (108.5, 109.9), turned to 180 degrees
- moved TP19 8.01 mm to (108.4, 96.0), turned to -90 degrees
- moved C57 6.03 mm to (116.5, 101.9), turned to 90 degrees
- moved U14 5.02 mm to (110.9, 101.8), turned to 180 degrees
- moved C27 3.63 mm to (113.4, 107.1), turned to -90 degrees
- moved J3 0.30 mm to (89.8, 95.2)
- moved J2 0.27 mm to (72.2, 72.4)
- turned J5 to -90 degrees
- turned J9 to 90 degrees
- renumbered R78 to R77, R77 to R78, R80 to R79, R79 to R80
Connections:
- J6 pad 1: /BUT1 -> /BUT12
- J6 pad 11: /BUT6 -> /BUT7
- J6 pad 13: /BUT7 -> /BUT6
- J6 pad 15: /BUT8 -> /BUT5
- J6 pad 17: /BUT9 -> /BUT4
- J6 pad 19: /BUT10 -> /BUT3
- J6 pad 21: /BUT11 -> /BUT2
- J6 pad 23: /BUT12 -> /BUT1
- J6 pad 3: /BUT2 -> /BUT11
- J6 pad 5: /BUT3 -> /BUT10
- J6 pad 7: /BUT4 -> /BUT9
- J6 pad 9: /BUT5 -> /BUT8
- R77 pad 2: /I2C2_SCL -> /I2C4_SCL
- R78 pad 2: /I2C4_SCL -> /I2C2_SCL
- R79 pad 2: /I2C2_SDA -> /I2C4_SDA
- R80 pad 2: /I2C4_SDA -> /I2C2_SDA
- TP6 pad 1: unconnected-(TP5-Pad1)_2 -> Net-(Q1-D)
- U17 pad 15: /SPI4_MOSI -> /SPI2_MOSI
- U17 pad 16: /SPI4_SCK -> /SPI4_CS0
- U17 pad 18: /SPI4_CS0 -> /SPI4_SCK
- U17 pad 19: /SPI2_MOSI -> /SPI4_MOSI
- U17 pad 5: /WS2812_Din -> /Dash_Screen_ShiftRegs/SER
- U17 pad 9: /Dash_Screen_ShiftRegs/SER -> /WS2812_Din
Routing:
- net Net-(Q2-S): track 0.00 -> 51.7 mm, vias 0 -> 3
- net /REG_for_Dash_Screen: track 131.9 -> 82.4 mm, vias 1 -> 3
- net Net-(Q1-D): track 0.00 -> 44.5 mm
- net +5V: track 445.8 -> 484.4 mm, vias 15 -> 20
- net /BUT2: track 41.9 -> 71.3 mm
- net /BUT1: track 42.6 -> 69.8 mm
- net /Dash_Screen_ShiftRegs/RCLK: track 262.2 -> 288.7 mm
- net /Dash_Screen_ShiftRegs/OE: track 251.6 -> 275.9 mm
- net /Dash_Screen_ShiftRegs/SRCLK: track 254.3 -> 276.2 mm
- net /BUT4: track 45.9 -> 66.9 mm
- net /SPI2_CS: track 0.00 -> 17.5 mm, vias 1 -> 2
- net /I2C4_SCL: track 49.6 -> 32.9 mm, vias 2 -> 1
- net /BUT3: track 48.7 -> 64.3 mm
- net /BUT11: track 63.9 -> 48.3 mm
- net GND: track 137.2 -> 151.8 mm, vias 64 -> 66
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- added copper zone on B.Cu, net GND
Other:
- board text added: "2_0"
- board text added: "4_1"
- board text added: "ACTIVE PULL HIGH"
- board text added: "ACTIVE PULL LOW"
- board text added: "AUX SOURCE"
- board text added: "AUX_MODE"
- board text added: "AUX_N"
- board text added: "AUX_P"
- board text added: "CHOOSE ONLY ONE!!"
- board text added: "Dash_Screen_Under V2.0 26/06/09"
- board text removed: "Dash_Screen_Under V1.1 26/05/23"
